Commit message: flipped laser scanner on turtlebot

File: robots/turtlebot.urdf.xacro (robot description, xacro)
@@ -12,5 +12,5 @@
   <sensor_kinect  parent="base_link"/>
   <xacro:rplidar name="rplidar" parent="base_link" ros_topic="scan" update_rate="5" ray_count="1040" min_angle="0" max_angle="360">
-    <origin xyz="0.1 0 0.420" rpy="3.1415 0 0"/>
+    <origin xyz="0.1 0 0.420" rpy="0 0 0"/>
   </xacro:rplidar>
 </robot>

Commit message: model visualization in kinetic

File: robots/turtlebot.urdf.xacro (robot description, xacro)
@@ -6,11 +6,12 @@
 -->
 <robot name="turtlebot" xmlns:xacro="http://ros.org/wiki/xacro">
-  <xacro:include filename="$(find turtlebot_description)/urdf/turtlebot_common_library.urdf.xacro" />
+<!--  <xacro:include filename="$(find turtlebot_description)/urdf/turtlebot_common_library.urdf.xacro" />-->
+  <xacro:include filename="$(find icclab_turtlebot)/robots/turtlebot_library.urdf.xacro" />
   <xacro:include filename="$(find icclab_turtlebot)/sensors/rplidar.urdf.xacro" />
   <kobuki/>
   <stack_hexagons parent="base_link"/>
   <sensor_kinect  parent="base_link"/>
-  <!--<xacro:rplidar name="rplidar" parent="base_link" ros_topic="scan" update_rate="5" ray_count="1040" min_angle="0" max_angle="360">
-    <origin xyz="0.1 0 0.420" rpy="0 0 0"/>
-  </xacro:rplidar>-->
+  <xacro:rplidar name="rplidar" parent="base_link" ros_topic="scan" update_rate="5" ray_count="1040" min_angle="0" max_angle="360">
+    <origin xyz="0.1 0 0.36" rpy="3.141 0 0"/>
+  </xacro:rplidar>
 </robot>

Commit message: updated robot description

File: robots/turtlebot.urdf.xacro (robot description, xacro)
@@ -6,11 +6,11 @@
 -->
 <robot name="turtlebot" xmlns:xacro="http://ros.org/wiki/xacro">
-  <xacro:include filename="$(find turtlebot_description)/urdf/turtlebot_common_library.urdf.xacro" />
+  <xacro:include filename="$(find turtlebot_description)/urdf/turtlebot_library.urdf.xacro" />
   <xacro:include filename="$(find icclab_turtlebot)/sensors/rplidar.urdf.xacro" />
   <kobuki/>
   <stack_hexagons parent="base_link"/>
   <sensor_kinect  parent="base_link"/>
-  <!--<xacro:rplidar name="rplidar" parent="base_link" ros_topic="scan" update_rate="5" ray_count="1040" min_angle="0" max_angle="360">
-    <origin xyz="0.1 0 0.420" rpy="0 0 0"/>
-  </xacro:rplidar>-->
+  <xacro:rplidar name="rplidar" parent="base_link" ros_topic="scan" update_rate="5" ray_count="1040" min_angle="0" max_angle="360">
+    <origin xyz="0.1 0 0.35" rpy="0 0 0"/>
+  </xacro:rplidar>
 </robot>

Commit message: merged turtlebot robot model

File: robots/turtlebot.urdf.xacro (robot description, xacro)
@@ -6,5 +6,4 @@
 -->
 <robot name="turtlebot" xmlns:xacro="http://ros.org/wiki/xacro">
-<!--  <xacro:include filename="$(find turtlebot_description)/urdf/turtlebot_common_library.urdf.xacro" />-->
   <xacro:include filename="$(find icclab_turtlebot)/robots/turtlebot_library.urdf.xacro" />
   <xacro:include filename="$(find icclab_turtlebot)/sensors/rplidar.urdf.xacro" />
@@ -13,5 +12,5 @@
   <sensor_kinect  parent="base_link"/>
   <xacro:rplidar name="rplidar" parent="base_link" ros_topic="scan" update_rate="5" ray_count="1040" min_angle="0" max_angle="360">
-    <origin xyz="0.1 0 0.36" rpy="3.141 0 0"/>
+    <origin xyz="0.1 0 0.35" rpy="0 0 0"/>
   </xacro:rplidar>
 </robot>
