Commit message: updated lidar coords and mesh

File: robots/irlab_summit_xls_std.urdf.xacro (robot description, xacro)
@@ -19,10 +19,16 @@
 	<xacro:property name="wheel_offset_y" value="0.2045" />
 	<xacro:property name="wheel_offset_z" value="0.0" />
-	<xacro:property name="front_laser_offset_x" value="0.377"/>
-	<xacro:property name="front_laser_offset_y" value="-0.20957"/>
-	<xacro:property name="front_laser_offset_z" value="0.2024"/>
-	<xacro:property name="rear_laser_offset_x" value="-0.377"/>
-	<xacro:property name="rear_laser_offset_y" value="0.20957"/>
-	<xacro:property name="rear_laser_offset_z" value="0.2024"/>
+	<!-- <xacro:property name="front_laser_offset_x" value="0.377"/>    -->
+	<xacro:property name="front_laser_offset_x" value="0.357"/>
+	<!-- <xacro:property name="front_laser_offset_y" value="-0.20957"/>     -->
+	<xacro:property name="front_laser_offset_y" value="-0.25957"/>
+	<!-- <xacro:property name="front_laser_offset_z" value="0.2024"/> -->
+	<xacro:property name="front_laser_offset_z" value="0.1566"/>
+	<!-- <xacro:property name="rear_laser_offset_x" value="-0.377"/> -->
+	<xacro:property name="rear_laser_offset_x" value="-0.357"/>
+	<!-- <xacro:property name="rear_laser_offset_y" value="0.20957"/>     -->
+	<xacro:property name="rear_laser_offset_y" value="0.25957"/>
+	<!-- <xacro:property name="rear_laser_offset_z" value="0.2024"/> -->
+	<xacro:property name="rear_laser_offset_z" value="0.1566"/>
 	<xacro:property name="front_ptz_camera_offset_x" value="0.308"/>
 	<xacro:property name="front_ptz_camera_offset_y" value="0.141"/>

File: sensors/scanse.urdf.xacro (robot description, xacro)
@@ -21,5 +21,5 @@
         <origin xyz="0 0 0" rpy="0 0 0"/>
         <geometry>
-            <mesh filename="package://icclab_turtlebot/meshes/hokuyo_utm_30lx.dae"/>
+            <mesh filename="package://icclab_turtlebot/meshes/sweep_lidar.stl"/>
         </geometry>
       </visual>

Commit message: added arm to urdf model. arm misbehaving in my gazebo

File: robots/irlab_summit_xls_std.urdf.xacro (robot description, xacro)
@@ -11,4 +11,6 @@
 	<xacro:include filename="$(find summit_xl_description)/urdf/wheels/rubber_wheel.urdf.xacro" />
 	<xacro:include filename="$(find summit_xl_description)/urdf/structures/structure_hokuyo.urdf.xacro" />
+	<!-- Import arm description -->
+	<xacro:include filename="$(find ur_description)/urdf/ur5.urdf.xacro" />
 	<!-- Import all available robotnik sensors -->
 	<xacro:include filename="$(find robotnik_sensors)/urdf/all_sensors.urdf.xacro" />
@@ -79,5 +81,32 @@
 		</xacro:scanse>
 		<!-- UR5 Arm -->
-		<!-- TODO -->
+		<xacro:ur5_robot prefix="arm_" joint_limited="true">
+	</xacro:ur5_robot>
+	<joint name="arm_base_joint" type="fixed">
+          <origin xyz="0.175 0 0.303" rpy="0 0 0" />
+          <parent link="$(arg prefix)base_link" />
+          <child link="arm_base_link" />
+	</joint>
+<!--	<joint name="gripper_joint" type="fixed">-->
+<!--	  <origin xyz="0.0 0.0 0.0" rpy="0.0 -1.5708 0.0" />-->
+<!--	  <parent link="arm_tool0" />-->
+<!--	  <child link="robotiq_85_adapter_link" />-->
+<!--	</joint>-->
+<!--	<joint name="tcp_joint" type="fixed">-->
+<!--	  <origin xyz="0.150 0.0 0.0" rpy="0.0 0.0 0.0" />-->
+<!--	  <parent link="robotiq_85_adapter_link"/>-->
+<!--          <child link="tcp_link"/>-->
+<!--        </joint>-->
+<!--        <link name="tcp_link">-->
+<!--          <visual>-->
+<!--          <origin xyz="0 0 0" rpy="0 0 0" />-->
+<!--          <geometry>-->
+<!--             <sphere radius="0.010"/>-->
+<!--          </geometry>-->
+<!--          <material name="green">-->
+<!--            <color rgba="0 1 0 1"/>-->
+<!--          </material>-->
+<!--          </visual>-->
+<!--        </link>-->
    </xacro:macro>
    <xacro:ros_control/>

Commit message: added gripper to model and flipped arm according to summit_xls_ur5_omni_170214A.urdf.xacro

File: robots/irlab_summit_xls_std.urdf.xacro (robot description, xacro)
@@ -15,4 +15,6 @@
 	<!-- Import all available robotnik sensors -->
 	<xacro:include filename="$(find robotnik_sensors)/urdf/all_sensors.urdf.xacro" />
+  <!-- Import gripper Schunk EGP40-->
+	<xacro:include filename="$(find summit_xl_description)/urdf/gripper/schunk_egp40.urdf.xacro" />
 	<!-- ICCLab sensors -->
 	<xacro:include filename="$(find icclab_turtlebot)/sensors/scanse.urdf.xacro" />
@@ -83,30 +85,13 @@
 		<xacro:ur5_robot prefix="arm_" joint_limited="true">
 	</xacro:ur5_robot>
-	<joint name="arm_base_joint" type="fixed">
-          <origin xyz="0.175 0 0.303" rpy="0 0 0" />
+	<joint name="$(arg prefix)arm_base_joint" type="fixed">
+          <origin xyz="0.255 0 0.275" rpy="0 0 ${PI}" />
           <parent link="$(arg prefix)base_link" />
           <child link="arm_base_link" />
-	</joint>
-<!--	<joint name="gripper_joint" type="fixed">-->
-<!--	  <origin xyz="0.0 0.0 0.0" rpy="0.0 -1.5708 0.0" />-->
-<!--	  <parent link="arm_tool0" />-->
-<!--	  <child link="robotiq_85_adapter_link" />-->
-<!--	</joint>-->
-<!--	<joint name="tcp_joint" type="fixed">-->
-<!--	  <origin xyz="0.150 0.0 0.0" rpy="0.0 0.0 0.0" />-->
-<!--	  <parent link="robotiq_85_adapter_link"/>-->
-<!--          <child link="tcp_link"/>-->
-<!--        </joint>-->
-<!--        <link name="tcp_link">-->
-<!--          <visual>-->
-<!--          <origin xyz="0 0 0" rpy="0 0 0" />-->
-<!--          <geometry>-->
-<!--             <sphere radius="0.010"/>-->
-<!--          </geometry>-->
-<!--          <material name="green">-->
-<!--            <color rgba="0 1 0 1"/>-->
-<!--          </material>-->
-<!--          </visual>-->
-<!--        </link>-->
+		</joint>
+		<!-- GRIPPER -->
+		<xacro:schunk_egp_40 prefix="gripper_" parent="arm_tool0" >
+			 <origin xyz="0.0 0 0.0" rpy="0 0 0" />
+		</xacro:schunk_egp_40>
    </xacro:macro>
    <xacro:ros_control/>

Commit message: path updates

File: robots/irlab_summit_xls_std.urdf.xacro (robot description, xacro)
@@ -16,5 +16,5 @@
 	<xacro:include filename="$(find robotnik_sensors)/urdf/all_sensors.urdf.xacro" />
   <!-- Import gripper Schunk EGP40-->
-	<xacro:include filename="$(find summit_xl_description)/urdf/gripper/schunk_egp40.urdf.xacro" />
+	<xacro:include filename="$(find icclab_turtlebot)/urdf/gripper/schunk_egp40.urdf.xacro" />
 	<!-- ICCLab sensors -->
 	<xacro:include filename="$(find icclab_turtlebot)/sensors/scanse.urdf.xacro" />

File: urdf/gripper/schunk_egp40.urdf.xacro (robot description, xacro)
@@ -26,5 +26,5 @@
           <origin xyz="0.0 0 0" rpy="0 0 0" />
           <geometry>
-             <mesh filename="package://summit_xl_description/meshes/gripper/schunk_epg40/schunk_epg40_base.stl" scale="1 1 1"/>
+             <mesh filename="package://icclab_turtlebot/meshes/gripper/schunk_epg40/schunk_epg40_base.stl" scale="1 1 1"/>
           </geometry>
           <material name="grey">
@@ -35,5 +35,5 @@
           <origin xyz="0.0 0 0" rpy="0 0 0" />
           <geometry>
-             <mesh filename="package://summit_xl_description/meshes/gripper/schunk_epg40/schunk_epg40_base.stl" scale="1 1 1"/>
+             <mesh filename="package://icclab_turtlebot/meshes/gripper/schunk_epg40/schunk_epg40_base.stl" scale="1 1 1"/>
           </geometry>
      </collision>
@@ -59,5 +59,5 @@
           <origin xyz="0.0 0 0" rpy="0 0 0" />
           <geometry>
-             <mesh filename="package://summit_xl_description/meshes/gripper/schunk_epg40/schunk_epg40_finger_base.stl" scale="1 1 1"/>
+             <mesh filename="package://icclab_turtlebot/meshes/gripper/schunk_epg40/schunk_epg40_finger_base.stl" scale="1 1 1"/>
           </geometry>
           <material name="grey">
@@ -68,5 +68,5 @@
           <origin xyz="0.0 0 0" rpy="0 0 0" />
           <geometry>
-             <mesh filename="package://summit_xl_description/meshes/gripper/schunk_epg40/schunk_epg40_finger_base.stl" scale="1 1 1"/>
+             <mesh filename="package://icclab_turtlebot/meshes/gripper/schunk_epg40/schunk_epg40_finger_base.stl" scale="1 1 1"/>
           </geometry>
      </collision>
@@ -86,5 +86,5 @@
           <origin xyz="0.0 0 0" rpy="0 0 0" />
           <geometry>
-             <mesh filename="package://summit_xl_description/meshes/gripper/schunk_epg40/schunk_epg40_finger.stl" scale="1 1 1"/>
+             <mesh filename="package://icclab_turtlebot/meshes/gripper/schunk_epg40/schunk_epg40_finger.stl" scale="1 1 1"/>
           </geometry>
           <material name="grey">
@@ -95,5 +95,5 @@
           <origin xyz="0.0 0 0" rpy="0 0 0" />
           <geometry>
-             <mesh filename="package://summit_xl_description/meshes/gripper/schunk_epg40/schunk_epg40_finger.stl" scale="1 1 1"/>
+             <mesh filename="package://icclab_turtlebot/meshes/gripper/schunk_epg40/schunk_epg40_finger.stl" scale="1 1 1"/>
           </geometry>
      </collision>
@@ -114,5 +114,5 @@
           <origin xyz="0.0 0 0" rpy="0 0 0" />
           <geometry>
-             <mesh filename="package://summit_xl_description/meshes/gripper/schunk_epg40/schunk_epg40_finger_base.stl" scale="1 1 1"/>
+             <mesh filename="package://icclab_turtlebot/meshes/gripper/schunk_epg40/schunk_epg40_finger_base.stl" scale="1 1 1"/>
           </geometry>
           <material name="grey">
@@ -123,5 +123,5 @@
           <origin xyz="0.0 0 0" rpy="0 0 0" />
           <geometry>
-             <mesh filename="package://summit_xl_description/meshes/gripper/schunk_epg40/schunk_epg40_finger_base.stl" scale="1 1 1"/>
+             <mesh filename="package://icclab_turtlebot/meshes/gripper/schunk_epg40/schunk_epg40_finger_base.stl" scale="1 1 1"/>
           </geometry>
      </collision>
@@ -141,5 +141,5 @@
           <origin xyz="0.0 0 0" rpy="0 0 0" />
           <geometry>
-             <mesh filename="package://summit_xl_description/meshes/gripper/schunk_epg40/schunk_epg40_finger.stl" scale="1 1 1"/>
+             <mesh filename="package://icclab_turtlebot/meshes/gripper/schunk_epg40/schunk_epg40_finger.stl" scale="1 1 1"/>
           </geometry>
           <material name="grey">
@@ -150,5 +150,5 @@
           <origin xyz="0.0 0 0" rpy="0 0 0" />
           <geometry>
-             <mesh filename="package://summit_xl_description/meshes/gripper/schunk_epg40/schunk_epg40_finger.stl" scale="1 1 1"/>
+             <mesh filename="package://icclab_turtlebot/meshes/gripper/schunk_epg40/schunk_epg40_finger.stl" scale="1 1 1"/>
           </geometry>
      </collision>
