Commit message: XML linting

File: robots/irlab_summit_xls_std.urdf.xacro (robot description, xacro)
@@ -1,4 +1,5 @@
 <?xml version="1.0"?>
-<robot name="summit_xl" xmlns:xacro="http://www.ros.org/wiki/xacro">
+<robot name="summit_xl"
+	xmlns:xacro="http://www.ros.org/wiki/xacro">
 	<!-- ***************** -->
 	<!-- Imported elements -->
@@ -15,10 +16,11 @@
 	<!-- Import all available robotnik sensors -->
 	<xacro:include filename="$(find robotnik_sensors)/urdf/all_sensors.urdf.xacro" />
-  <!-- Import gripper Schunk EGP40-->
+	<!-- Import gripper Schunk EGP40-->
 	<xacro:include filename="$(find icclab_turtlebot)/urdf/gripper/schunk_egp40.urdf.xacro" />
 	<!-- ICCLab sensors -->
 	<xacro:include filename="$(find icclab_turtlebot)/urdf/sensors/scanse.urdf.xacro" />
 	<xacro:property name="PI" value="3.1415926535897931"/>
-	<xacro:property name="wheel_offset_x" value="0.2225" />    <!-- x,y,z in translation from base_link to the center of the wheel -->
+	<xacro:property name="wheel_offset_x" value="0.2225" />
+	<!-- x,y,z in translation from base_link to the center of the wheel -->
 	<xacro:property name="wheel_offset_y" value="0.2045" />
 	<xacro:property name="wheel_offset_z" value="0.0" />
@@ -48,5 +50,5 @@
 	<xacro:arg name="prefix" default="summit_xl_"/>
 	<xacro:arg name="ros_planar_move_plugin" default="false"/>
-    <xacro:macro name="summit_xl" params="prefix publish_bf hq">
+	<xacro:macro name="summit_xl" params="prefix publish_bf hq">
 		<!-- Here we create the robot elements using the xacro:macros imported at the beggining of this file -->
 		<!-- Summit XL base -->
@@ -65,5 +67,5 @@
 			<origin xyz="-${wheel_offset_x} -${wheel_offset_y} ${wheel_offset_z}" rpy="0 0 0"/>
 		</xacro:omni_wheel>
-        <!-- IMU -->
+		<!-- IMU -->
 		<xacro:sensor_imu_hector prefix="$(arg prefix)imu" parent="$(arg prefix)base_link">
 			<origin xyz="-0.18 0.0 0.170" rpy="0 0 0"/>
@@ -84,19 +86,19 @@
 		<!-- UR5 Arm -->
 		<xacro:ur5_robot prefix="arm_" joint_limited="true">
-	</xacro:ur5_robot>
-	<joint name="$(arg prefix)arm_base_joint" type="fixed">
-          <origin xyz="0.255 0 0.275" rpy="0 0 ${PI}" />
-          <parent link="$(arg prefix)base_link" />
-          <child link="arm_base_link" />
+		</xacro:ur5_robot>
+		<joint name="$(arg prefix)arm_base_joint" type="fixed">
+			<origin xyz="0.255 0 0.275" rpy="0 0 ${PI}" />
+			<parent link="$(arg prefix)base_link" />
+			<child link="arm_base_link" />
 		</joint>
 		<!-- GRIPPER -->
-		<xacro:schunk_egp_40 prefix="gripper_" parent="arm_tool0" >
-			 <origin xyz="0.0 0 0.0" rpy="0 0 0" />
+		<xacro:schunk_egp_40 prefix="gripper_" parent="arm_tool0">
+			<origin xyz="0.0 0 0.0" rpy="0 0 0" />
 		</xacro:schunk_egp_40>
-   </xacro:macro>
-   <xacro:ros_control/>
-   <xacro:if value="$(arg ros_planar_move_plugin)">
-	   <xacro:omni_steering prefix="$(arg prefix)" publish_tf="false"/>
-   </xacro:if>
-   <xacro:summit_xl prefix="$(arg prefix)" publish_bf="true" hq="true"/>
+	</xacro:macro>
+	<xacro:ros_control/>
+	<xacro:if value="$(arg ros_planar_move_plugin)">
+		<xacro:omni_steering prefix="$(arg prefix)" publish_tf="false"/>
+	</xacro:if>
+	<xacro:summit_xl prefix="$(arg prefix)" publish_bf="true" hq="true"/>
 </robot>

File: urdf/gripper/schunk_egp40.urdf.xacro (robot description, xacro)
@@ -1,157 +1,154 @@
 <?xml version="1.0"?>
-<robot  xmlns:sensor="http://playerstage.sourceforge.net/gazebo/xmlschema/#sensor"
-	xmlns:controller="http://playerstage.sourceforge.net/gazebo/xmlschema/#controller"
-	xmlns:interface="http://playerstage.sourceforge.net/gazebo/xmlschema/#interface"
-        xmlns:xacro="http://ros.org/wiki/xacro"
-	name="egp_40">
-  <xacro:macro name="cylinder_inertia" params="m r h">
-    <inertia  ixx="${m*(3*r*r+h*h)/12}" ixy = "0" ixz = "0"
-              iyy="${m*(3*r*r+h*h)/12}" iyz = "0"
-              izz="${m*r*r/2}" />
-</xacro:macro>
-<xacro:macro name="schunk_egp_40" params="prefix parent *origin">
- <joint name="${prefix}base_joint" type="fixed">
-    <xacro:insert_block name="origin"/>
-    <parent link="${parent}"/>
-    <child link="${prefix}base_link"/>
- </joint>
-<!-- BASE LINK -->
- <link name="${prefix}base_link">
-      <inertial>
-          <mass value="0.25" />
-          <origin xyz="0 0 0" />
-          <cylinder_inertia m="0.20" r="0.05" h="0.05" />
-      </inertial>
-      <visual>
-          <origin xyz="0.0 0 0" rpy="0 0 0" />
-          <geometry>
-             <mesh filename="package://icclab_turtlebot/meshes/gripper/schunk_epg40/schunk_epg40_base.stl" scale="1 1 1"/>
-          </geometry>
-          <material name="grey">
-		     <color rgba="0.5 0.5 0.5 1"/>
-      	  </material>
-      </visual>
-      <collision>
-          <origin xyz="0.0 0 0" rpy="0 0 0" />
-          <geometry>
-             <mesh filename="package://icclab_turtlebot/meshes/gripper/schunk_epg40/schunk_epg40_base.stl" scale="1 1 1"/>
-          </geometry>
-     </collision>
-  </link>
-  <gazebo reference="${prefix}base_link">
-    <material>Gazebo/Grey</material>
-    <turnGravityOff>false</turnGravityOff>
-  </gazebo>
- <!-- GRIPPER FINGER LEFT -->
- <joint name="${prefix}left_finger_base_joint" type="fixed">
-    <parent link="${prefix}base_link"/>
-    <child link="${prefix}left_finger_base_link"/>
-    <origin xyz="-0.012 0 0.08915" rpy="0 0 0" />
-    <axis xyz="0 1 0" />
- </joint>
- <link name="${prefix}left_finger_base_link">
-      <inertial>
-          <mass value="0.02" />
-          <origin xyz="0 0 0" />
-          <cylinder_inertia m="0.02" r="0.01" h="0.01" />
-      </inertial>
-      <visual>
-          <origin xyz="0.0 0 0" rpy="0 0 0" />
-          <geometry>
-             <mesh filename="package://icclab_turtlebot/meshes/gripper/schunk_epg40/schunk_epg40_finger_base.stl" scale="1 1 1"/>
-          </geometry>
-          <material name="grey">
-		     <color rgba="0.5 0.5 0.5 1"/>
-      	  </material>
-      </visual>
-      <collision>
-          <origin xyz="0.0 0 0" rpy="0 0 0" />
-          <geometry>
-             <mesh filename="package://icclab_turtlebot/meshes/gripper/schunk_epg40/schunk_epg40_finger_base.stl" scale="1 1 1"/>
-          </geometry>
-     </collision>
-  </link>
- <joint name="${prefix}left_finger_joint" type="fixed">
-    <parent link="${prefix}left_finger_base_link"/>
-    <child link="${prefix}left_finger_link"/>
-    <origin xyz="0.012 0 0.05" rpy="0 0 0" />
- </joint>
- <link name="${prefix}left_finger_link">
-      <inertial>
-          <mass value="0.02" />
-          <origin xyz="0 0 0" />
-          <cylinder_inertia m="0.02" r="0.01" h="0.01" />
-      </inertial>
-      <visual>
-          <origin xyz="0.0 0 0" rpy="0 0 0" />
-          <geometry>
-             <mesh filename="package://icclab_turtlebot/meshes/gripper/schunk_epg40/schunk_epg40_finger.stl" scale="1 1 1"/>
-          </geometry>
-          <material name="grey">
-		     <color rgba="0.5 0.5 0.5 1"/>
-      	  </material>
-      </visual>
-      <collision>
-          <origin xyz="0.0 0 0" rpy="0 0 0" />
-          <geometry>
-             <mesh filename="package://icclab_turtlebot/meshes/gripper/schunk_epg40/schunk_epg40_finger.stl" scale="1 1 1"/>
-          </geometry>
-     </collision>
-  </link>
- <!-- GRIPPER FINGER RIGHT -->
- <joint name="${prefix}right_finger_base_joint" type="fixed">
-    <parent link="${prefix}base_link"/>
-    <child link="${prefix}right_finger_base_link"/>
-    <origin xyz="0.012 0 0.08915" rpy="0 0 3.14" />
- </joint>
- <link name="${prefix}right_finger_base_link">
-      <inertial>
-          <mass value="0.02" />
-          <origin xyz="0 0 0" />
-          <cylinder_inertia m="0.02" r="0.01" h="0.01" />
-      </inertial>
-      <visual>
-          <origin xyz="0.0 0 0" rpy="0 0 0" />
-          <geometry>
-             <mesh filename="package://icclab_turtlebot/meshes/gripper/schunk_epg40/schunk_epg40_finger_base.stl" scale="1 1 1"/>
-          </geometry>
-          <material name="grey">
-		     <color rgba="0.5 0.5 0.5 1"/>
-      	  </material>
-      </visual>
-      <collision>
-          <origin xyz="0.0 0 0" rpy="0 0 0" />
-          <geometry>
-             <mesh filename="package://icclab_turtlebot/meshes/gripper/schunk_epg40/schunk_epg40_finger_base.stl" scale="1 1 1"/>
-          </geometry>
-     </collision>
-  </link>
- <joint name="${prefix}right_finger_joint" type="fixed">
-    <parent link="${prefix}right_finger_base_link"/>
-    <child link="${prefix}right_finger_link"/>
-    <origin xyz="0.012 0 0.05" rpy="0 0 0" />
- </joint>
- <link name="${prefix}right_finger_link">
-      <inertial>
-          <mass value="0.02" />
-          <origin xyz="0 0 0" />
-          <cylinder_inertia m="0.02" r="0.01" h="0.01" />
-      </inertial>
-      <visual>
-          <origin xyz="0.0 0 0" rpy="0 0 0" />
-          <geometry>
-             <mesh filename="package://icclab_turtlebot/meshes/gripper/schunk_epg40/schunk_epg40_finger.stl" scale="1 1 1"/>
-          </geometry>
-          <material name="grey">
-		     <color rgba="0.5 0.5 0.5 1"/>
-      	  </material>
-      </visual>
-      <collision>
-          <origin xyz="0.0 0 0" rpy="0 0 0" />
-          <geometry>
-             <mesh filename="package://icclab_turtlebot/meshes/gripper/schunk_epg40/schunk_epg40_finger.stl" scale="1 1 1"/>
-          </geometry>
-     </collision>
-  </link>
-</xacro:macro>
+<robot xmlns:sensor="http://playerstage.sourceforge.net/gazebo/xmlschema/#sensor"
+   xmlns:controller="http://playerstage.sourceforge.net/gazebo/xmlschema/#controller"
+   xmlns:interface="http://playerstage.sourceforge.net/gazebo/xmlschema/#interface"
+   xmlns:xacro="http://ros.org/wiki/xacro" name="egp_40">
+   <xacro:macro name="cylinder_inertia" params="m r h">
+      <inertia ixx="${m*(3*r*r+h*h)/12}" ixy = "0" ixz = "0" iyy="${m*(3*r*r+h*h)/12}" iyz = "0" izz="${m*r*r/2}" />
+   </xacro:macro>
+   <xacro:macro name="schunk_egp_40" params="prefix parent *origin">
+      <joint name="${prefix}base_joint" type="fixed">
+         <xacro:insert_block name="origin"/>
+         <parent link="${parent}"/>
+         <child link="${prefix}base_link"/>
+      </joint>
+      <!-- BASE LINK -->
+      <link name="${prefix}base_link">
+         <inertial>
+            <mass value="0.25" />
+            <origin xyz="0 0 0" />
+            <cylinder_inertia m="0.20" r="0.05" h="0.05" />
+         </inertial>
+         <visual>
+            <origin xyz="0.0 0 0" rpy="0 0 0" />
+            <geometry>
+               <mesh filename="package://icclab_turtlebot/meshes/gripper/schunk_epg40/schunk_epg40_base.stl" scale="1 1 1"/>
+            </geometry>
+            <material name="grey">
+               <color rgba="0.5 0.5 0.5 1"/>
+            </material>
+         </visual>
+         <collision>
+            <origin xyz="0.0 0 0" rpy="0 0 0" />
+            <geometry>
+               <mesh filename="package://icclab_turtlebot/meshes/gripper/schunk_epg40/schunk_epg40_base.stl" scale="1 1 1"/>
+            </geometry>
+         </collision>
+      </link>
+      <gazebo reference="${prefix}base_link">
+         <material>Gazebo/Grey</material>
+         <turnGravityOff>false</turnGravityOff>
+      </gazebo>
+      <!-- GRIPPER FINGER LEFT -->
+      <joint name="${prefix}left_finger_base_joint" type="fixed">
+         <parent link="${prefix}base_link"/>
+         <child link="${prefix}left_finger_base_link"/>
+         <origin xyz="-0.012 0 0.08915" rpy="0 0 0" />
+         <axis xyz="0 1 0" />
+      </joint>
+      <link name="${prefix}left_finger_base_link">
+         <inertial>
+            <mass value="0.02" />
+            <origin xyz="0 0 0" />
+            <cylinder_inertia m="0.02" r="0.01" h="0.01" />
+         </inertial>
+         <visual>
+            <origin xyz="0.0 0 0" rpy="0 0 0" />
+            <geometry>
+               <mesh filename="package://icclab_turtlebot/meshes/gripper/schunk_epg40/schunk_epg40_finger_base.stl" scale="1 1 1"/>
+            </geometry>
+            <material name="grey">
+               <color rgba="0.5 0.5 0.5 1"/>
+            </material>
+         </visual>
+         <collision>
+            <origin xyz="0.0 0 0" rpy="0 0 0" />
+            <geometry>
+               <mesh filename="package://icclab_turtlebot/meshes/gripper/schunk_epg40/schunk_epg40_finger_base.stl" scale="1 1 1"/>
+            </geometry>
+         </collision>
+      </link>
+      <joint name="${prefix}left_finger_joint" type="fixed">
+         <parent link="${prefix}left_finger_base_link"/>
+         <child link="${prefix}left_finger_link"/>
+         <origin xyz="0.012 0 0.05" rpy="0 0 0" />
+      </joint>
+      <link name="${prefix}left_finger_link">
+         <inertial>
+            <mass value="0.02" />
+            <origin xyz="0 0 0" />
+            <cylinder_inertia m="0.02" r="0.01" h="0.01" />
+         </inertial>
+         <visual>
+            <origin xyz="0.0 0 0" rpy="0 0 0" />
+            <geometry>
+               <mesh filename="package://icclab_turtlebot/meshes/gripper/schunk_epg40/schunk_epg40_finger.stl" scale="1 1 1"/>
+            </geometry>
+            <material name="grey">
+               <color rgba="0.5 0.5 0.5 1"/>
+            </material>
+         </visual>
+         <collision>
+            <origin xyz="0.0 0 0" rpy="0 0 0" />
+            <geometry>
+               <mesh filename="package://icclab_turtlebot/meshes/gripper/schunk_epg40/schunk_epg40_finger.stl" scale="1 1 1"/>
+            </geometry>
+         </collision>
+      </link>
+      <!-- GRIPPER FINGER RIGHT -->
+      <joint name="${prefix}right_finger_base_joint" type="fixed">
+         <parent link="${prefix}base_link"/>
+         <child link="${prefix}right_finger_base_link"/>
+         <origin xyz="0.012 0 0.08915" rpy="0 0 3.14" />
+      </joint>
+      <link name="${prefix}right_finger_base_link">
+         <inertial>
+            <mass value="0.02" />
+            <origin xyz="0 0 0" />
+            <cylinder_inertia m="0.02" r="0.01" h="0.01" />
+         </inertial>
+         <visual>
+            <origin xyz="0.0 0 0" rpy="0 0 0" />
+            <geometry>
+               <mesh filename="package://icclab_turtlebot/meshes/gripper/schunk_epg40/schunk_epg40_finger_base.stl" scale="1 1 1"/>
+            </geometry>
+            <material name="grey">
+               <color rgba="0.5 0.5 0.5 1"/>
+            </material>
+         </visual>
+         <collision>
+            <origin xyz="0.0 0 0" rpy="0 0 0" />
+            <geometry>
+               <mesh filename="package://icclab_turtlebot/meshes/gripper/schunk_epg40/schunk_epg40_finger_base.stl" scale="1 1 1"/>
+            </geometry>
+         </collision>
+      </link>
+      <joint name="${prefix}right_finger_joint" type="fixed">
+         <parent link="${prefix}right_finger_base_link"/>
+         <child link="${prefix}right_finger_link"/>
+         <origin xyz="0.012 0 0.05" rpy="0 0 0" />
+      </joint>
+      <link name="${prefix}right_finger_link">
+         <inertial>
+            <mass value="0.02" />
+            <origin xyz="0 0 0" />
+            <cylinder_inertia m="0.02" r="0.01" h="0.01" />
+         </inertial>
+         <visual>
+            <origin xyz="0.0 0 0" rpy="0 0 0" />
+            <geometry>
+               <mesh filename="package://icclab_turtlebot/meshes/gripper/schunk_epg40/schunk_epg40_finger.stl" scale="1 1 1"/>
+            </geometry>
+            <material name="grey">
+               <color rgba="0.5 0.5 0.5 1"/>
+            </material>
+         </visual>
+         <collision>
+            <origin xyz="0.0 0 0" rpy="0 0 0" />
+            <geometry>
+               <mesh filename="package://icclab_turtlebot/meshes/gripper/schunk_epg40/schunk_epg40_finger.stl" scale="1 1 1"/>
+            </geometry>
+         </collision>
+      </link>
+   </xacro:macro>
 </robot>

File: urdf/sensors/scanse.urdf.xacro (robot description, xacro)
@@ -1,5 +1,6 @@
 <?xml version=  "1.0"?>
-<robot name="scanse" xmlns:xacro="http://www.ros.org/wiki/xacro"> <!-- sensor_hokuyo_utm30lx -->
-  <xacro:macro name="scanse" params="prefix parent prefix_topic:='front_laser' *origin min_angle:=-2.35 max_angle:=2.35"> <!-- sensor_hokuyo_utm30lx -->
+<robot name="scanse"
+  xmlns:xacro="http://www.ros.org/wiki/xacro">  <!-- sensor_hokuyo_utm30lx -->
+  <xacro:macro name="scanse" params="prefix parent prefix_topic:='front_laser' *origin min_angle:=-2.35 max_angle:=2.35">    <!-- sensor_hokuyo_utm30lx -->
     <joint name="${prefix}_base_joint" type="fixed">
       <!-- FRONT MOUNT  -->
@@ -12,5 +13,5 @@
     </joint>
     <link name="${prefix}_base_link">
-      <collision> <!-- added -->
+      <collision>        <!-- added -->
         <origin xyz="0 0 0" rpy="0 0 0"/>
         <geometry>
@@ -21,5 +22,5 @@
         <origin xyz="0 0 0" rpy="0 0 0"/>
         <geometry>
-            <mesh filename="package://icclab_turtlebot/meshes/sweep_lidar.stl"/>
+          <mesh filename="package://icclab_turtlebot/meshes/sweep_lidar.stl"/>
         </geometry>
       </visual>
@@ -30,11 +31,11 @@
       </inertial>
     </link>
-	<link name="${prefix}_link">
-	</link>
+    <link name="${prefix}_link">
+    </link>
     <joint name="${prefix}_joint" type="fixed">
       <parent link="${prefix}_base_link"/>
       <child link="${prefix}_link"/>
       <origin xyz="0.00 0 0.055" rpy="0 0 0"/>
-	</joint>
+    </joint>
     <!-- Hokuyo sensor for simulation -->
     <sensor_hokuyo_utm_gazebo/>
@@ -42,34 +43,34 @@
   <xacro:macro name="sensor_hokuyo_utm_gazebo">
     <gazebo reference="${prefix}_link">
-			<sensor type="ray" name="${prefix}_sensor">
-				<pose>0 0 0 0 0 0</pose>
-				<visualize>false</visualize>
-				<update_rate>30</update_rate> <!-- 30 -->
-				<ray>
-					<scan>
-						<horizontal>
-							<samples>1081</samples>
-							<resolution>1</resolution>
-							<min_angle>${min_angle}</min_angle>
-							<max_angle>${max_angle}</max_angle>
-						</horizontal>
-					</scan>
-					<range>
-						<min>0.10</min>
-						<max>30.0</max> <!-- 30.0 -->
-						<resolution>0.01</resolution>
-					</range>
-					<noise>
-						<type>gaussian</type>
-						<mean>0.0</mean>
-						<stddev>0.01</stddev>
-					</noise>
-				</ray>
-				<plugin name="${prefix}_controller" filename="libgazebo_ros_laser.so">
-					<topicName>${prefix_topic}/scan</topicName>
-					<frameName>/${prefix}_link</frameName>
-				</plugin>
-			</sensor>
-		</gazebo>
+      <sensor type="ray" name="${prefix}_sensor">
+        <pose>0 0 0 0 0 0</pose>
+        <visualize>false</visualize>
+        <update_rate>30</update_rate>        <!-- 30 -->
+        <ray>
+          <scan>
+            <horizontal>
+              <samples>1081</samples>
+              <resolution>1</resolution>
+              <min_angle>${min_angle}</min_angle>
+              <max_angle>${max_angle}</max_angle>
+            </horizontal>
+          </scan>
+          <range>
+            <min>0.10</min>
+            <max>30.0</max>            <!-- 30.0 -->
+            <resolution>0.01</resolution>
+          </range>
+          <noise>
+            <type>gaussian</type>
+            <mean>0.0</mean>
+            <stddev>0.01</stddev>
+          </noise>
+        </ray>
+        <plugin name="${prefix}_controller" filename="libgazebo_ros_laser.so">
+          <topicName>${prefix_topic}/scan</topicName>
+          <frameName>/${prefix}_link</frameName>
+        </plugin>
+      </sensor>
+    </gazebo>
   </xacro:macro>
 </robot>

Commit message: added schunk pg70. dependency from https://github.com/ipa320/schunk_modular_robotics

File: robots/irlab_summit_xls_std.urdf.xacro (robot description, xacro)
@@ -96,5 +96,9 @@
 			 <origin xyz="0.0 0 0.0" rpy="0 0 0" />
 		</xacro:schunk_egp_40> -->
-		 <xacro:include filename="$(find icclab_turtlebot)/urdf/gripper/ur5_robotiq85_gripper.urdf.xacro"/>
+		 <!--<xacro:include filename="$(find icclab_turtlebot)/urdf/gripper/ur5_robotiq85_gripper.urdf.xacro"/>-->
+		 <xacro:include filename="$(find icclab_turtlebot)/urdf/gripper/pg70.urdf.xacro"/>
+		 <xacro:schunk_pg70 name="gripper" parent="arm_tool0" has_podest="false">
+			 <origin xyz="0.0 0 0.0" rpy="0 0 0" />
+		</xacro:schunk_pg70>
    </xacro:macro>
    <xacro:ros_control/>
