Commit message: made schunk_egp40 a proper gripper with prismatic joints and control

File: robots/irlab_summit_xls_std.urdf.xacro (robot description, xacro)
@@ -93,12 +93,12 @@
 		</joint>
 		<!-- GRIPPER -->
-		<!-- <xacro:schunk_egp_40 prefix="gripper_" parent="arm_tool0" >
+		<xacro:schunk_egp_40 prefix="gripper_" parent="arm_tool0" >
 			 <origin xyz="0.0 0 0.0" rpy="0 0 0" />
-		</xacro:schunk_egp_40> -->
+		</xacro:schunk_egp_40>
 		 <!--<xacro:include filename="$(find icclab_turtlebot)/urdf/gripper/ur5_robotiq85_gripper.urdf.xacro"/>-->
-		 <xacro:include filename="$(find icclab_turtlebot)/urdf/gripper/pg70.urdf.xacro"/>
+		 <!-- <xacro:include filename="$(find icclab_turtlebot)/urdf/gripper/pg70.urdf.xacro"/>
 		 <xacro:schunk_pg70 name="gripper" parent="arm_tool0" has_podest="false">
 			 <origin xyz="0.0 0 0.0" rpy="0 0 0" />
-		</xacro:schunk_pg70>
+		</xacro:schunk_pg70> -->
    </xacro:macro>
    <xacro:ros_control/>

File: urdf/gripper/schunk_egp40.urdf.xacro (robot description, xacro)
@@ -7,4 +7,17 @@
       <inertia ixx="${m*(3*r*r+h*h)/12}" ixy = "0" ixz = "0" iyy="${m*(3*r*r+h*h)/12}" iyz = "0" izz="${m*r*r/2}" />
    </xacro:macro>
+   <xacro:macro name="default_transmission" params="jname">
+    <transmission name="${jname}_trans">
+      <type>transmission_interface/SimpleTransmission</type>
+      <joint name="${jname}_joint">
+        <hardwareInterface>PositionJointInterface</hardwareInterface>
+        <hardwareInterface>VelocityJointInterface</hardwareInterface>
+        <!--hardwareInterface>EffortJointInterface</hardwareInterface-->
+      </joint>
+      <actuator name="${jname}_motor">
+        <mechanicalReduction>1</mechanicalReduction>
+      </actuator>
+    </transmission>
+  </xacro:macro>
    <xacro:macro name="schunk_egp_40" params="prefix parent *origin">
       <joint name="${prefix}base_joint" type="fixed">
@@ -41,9 +54,10 @@
       </gazebo>
       <!-- GRIPPER FINGER LEFT -->
-      <joint name="${prefix}left_finger_base_joint" type="fixed">
+      <joint name="${prefix}left_finger_base_joint" type="prismatic">
          <parent link="${prefix}base_link"/>
          <child link="${prefix}left_finger_base_link"/>
          <origin xyz="-0.012 0 0.08915" rpy="0 0 0" />
-         <axis xyz="0 1 0" />
+         <axis xyz="-1 0 0" />
+         <limit effort="10" lower="0.001" upper="0.015" velocity="0.041"/>
       </joint>
       <link name="${prefix}left_finger_base_link">
@@ -97,8 +111,10 @@
       </link>
       <!-- GRIPPER FINGER RIGHT -->
-      <joint name="${prefix}right_finger_base_joint" type="fixed">
+      <joint name="${prefix}right_finger_base_joint" type="prismatic">
          <parent link="${prefix}base_link"/>
          <child link="${prefix}right_finger_base_link"/>
          <origin xyz="0.012 0 0.08915" rpy="0 0 3.14" />
+         <axis xyz="-1 0 0" />
+         <limit effort="10" lower="0.001" upper="0.015" velocity="0.041"/>
       </joint>
       <link name="${prefix}right_finger_base_link">
@@ -151,4 +167,6 @@
          </collision>
       </link>
+    <xacro:default_transmission jname="${prefix}left_finger_base"/>
+    <xacro:default_transmission jname="${prefix}right_finger_base"/>
    </xacro:macro>
 </robot>

Commit message: added realsense camera on arm. works in gazebo and rviz producing camera image

File: robots/irlab_summit_xls_std.urdf.xacro (robot description, xacro)
@@ -96,9 +96,8 @@
 			 <origin xyz="0.0 0 0.0" rpy="0 0 0" />
 		</xacro:schunk_egp_40>
-		 <!--<xacro:include filename="$(find icclab_turtlebot)/urdf/gripper/ur5_robotiq85_gripper.urdf.xacro"/>-->
-		 <!-- <xacro:include filename="$(find icclab_turtlebot)/urdf/gripper/pg70.urdf.xacro"/>
-		 <xacro:schunk_pg70 name="gripper" parent="arm_tool0" has_podest="false">
-			 <origin xyz="0.0 0 0.0" rpy="0 0 0" />
-		</xacro:schunk_pg70> -->
+		<!-- Camera on gripper -->
+		<sensor_r430 prefix="arm" prefix_topic="arm_camera" parent="arm_tool0">
+      <origin xyz="0 0.03 0.05" rpy="${-PI/2} ${-PI/2} 0"/>
+    </sensor_r430>
    </xacro:macro>
    <xacro:ros_control/>

Commit message: changed gripper to used effort based control

File: robots/irlab_summit_xls_std.urdf.xacro (robot description, xacro)
@@ -85,5 +85,5 @@
 		</xacro:scanse>
 		<!-- UR5 Arm -->
-		<xacro:ur5_robot prefix="arm_" joint_limited="true">
+		<xacro:ur5_robot prefix="arm_" joint_limited="false">
 		</xacro:ur5_robot>
 		<joint name="$(arg prefix)arm_base_joint" type="fixed">
@@ -98,5 +98,5 @@
 		<!-- Camera on gripper -->
 		<sensor_r430 prefix="arm" prefix_topic="arm_camera" parent="arm_tool0">
-      <origin xyz="0 0.03 0.05" rpy="${-PI/2} ${-PI/2} 0"/>
+      <origin xyz="0 0.045 -0.015" rpy="${-PI/2} ${-PI/2} 0"/>
     </sensor_r430>
    </xacro:macro>

File: urdf/gripper/schunk_egp40.urdf.xacro (robot description, xacro)
@@ -11,7 +11,7 @@
       <type>transmission_interface/SimpleTransmission</type>
       <joint name="${jname}_joint">
-        <hardwareInterface>PositionJointInterface</hardwareInterface>
-        <hardwareInterface>VelocityJointInterface</hardwareInterface>
-        <!--hardwareInterface>EffortJointInterface</hardwareInterface-->
+        <hardwareInterface>hardware_interface/EffortJointInterface</hardwareInterface>
+        <!--<hardwareInterface>hardware_interface/PositionJointInterface</hardwareInterface>
+        <hardwareInterface>hardware_interface/VelocityJointInterface</hardwareInterface>-->
       </joint>
       <actuator name="${jname}_motor">

Commit message: grasping starts its own simulation and world. no need to use complete anymore

File: robots/irlab_summit_xls_std.urdf.xacro (robot description, xacro)
@@ -1,5 +1,4 @@
 <?xml version="1.0"?>
-<robot name="summit_xl"
-	xmlns:xacro="http://www.ros.org/wiki/xacro">
+<robot name="summit_xl" xmlns:xacro="http://www.ros.org/wiki/xacro">
 	<!-- ***************** -->
 	<!-- Imported elements -->
@@ -46,4 +45,7 @@
 	<xacro:property name="front_rgbd_camera_offset_y" value="0.012"/>
 	<xacro:property name="front_rgbd_camera_offset_z" value="0.230"/>
+  <xacro:property name="base_arm_x" value="0.225"/>
+  <xacro:property name="base_arm_y" value="0.0"/>
+  <xacro:property name="base_arm_z" value="0.355"/>
 	<!-- Flag to select the high or low quality model -->
 	<xacro:property name="hq" value="true" />
@@ -85,5 +87,5 @@
 		</xacro:scanse>
 		<!-- UR5 Arm -->
-		<xacro:ur5_robot prefix="arm_" joint_limited="false">
+		<xacro:ur5_robot prefix="arm_" joint_limited="true">
 		</xacro:ur5_robot>
 		<joint name="$(arg prefix)arm_base_joint" type="fixed">

Commit message: replaced all occurrences of icclab_turtlebot

File: robots/irlab_summit_xls_std.urdf.xacro (robot description, xacro)
@@ -16,7 +16,7 @@
 	<xacro:include filename="$(find robotnik_sensors)/urdf/all_sensors.urdf.xacro" />
 	<!-- Import gripper Schunk EGP40-->
-	<xacro:include filename="$(find icclab_turtlebot)/urdf/gripper/schunk_egp40.urdf.xacro" />
+	<xacro:include filename="$(find icclab_summit_xl)/urdf/gripper/schunk_egp40.urdf.xacro" />
 	<!-- ICCLab sensors -->
-	<xacro:include filename="$(find icclab_turtlebot)/urdf/sensors/scanse.urdf.xacro" />
+	<xacro:include filename="$(find icclab_summit_xl)/urdf/sensors/scanse.urdf.xacro" />
 	<xacro:property name="PI" value="3.1415926535897931"/>
 	<xacro:property name="wheel_offset_x" value="0.2225" />

File: urdf/gripper/schunk_egp40.urdf.xacro (robot description, xacro)
@@ -36,14 +36,14 @@
             <origin xyz="0.0 0 0" rpy="0 0 0" />
             <geometry>
-               <mesh filename="package://icclab_turtlebot/meshes/gripper/schunk_epg40/schunk_epg40_base.stl" scale="1 1 1"/>
-            </geometry>
-            <material name="grey">
-               <color rgba="0.5 0.5 0.5 1"/>
-            </material>
-         </visual>
-         <collision>
-            <origin xyz="0.0 0 0" rpy="0 0 0" />
-            <geometry>
-               <mesh filename="package://icclab_turtlebot/meshes/gripper/schunk_epg40/schunk_epg40_base.stl" scale="1 1 1"/>
+               <mesh filename="package://icclab_summit_xl/meshes/gripper/schunk_epg40/schunk_epg40_base.stl" scale="1 1 1"/>
+            </geometry>
+            <material name="grey">
+               <color rgba="0.5 0.5 0.5 1"/>
+            </material>
+         </visual>
+         <collision>
+            <origin xyz="0.0 0 0" rpy="0 0 0" />
+            <geometry>
+               <mesh filename="package://icclab_summit_xl/meshes/gripper/schunk_epg40/schunk_epg40_base.stl" scale="1 1 1"/>
             </geometry>
          </collision>
@@ -73,14 +73,14 @@
             <origin xyz="0.0 0 0" rpy="0 0 0" />
             <geometry>
-               <mesh filename="package://icclab_turtlebot/meshes/gripper/schunk_epg40/schunk_epg40_finger_base.stl" scale="1 1 1"/>
-            </geometry>
-            <material name="grey">
-               <color rgba="0.5 0.5 0.5 1"/>
-            </material>
-         </visual>
-         <collision>
-            <origin xyz="0.0 0 0" rpy="0 0 0" />
-            <geometry>
-               <mesh filename="package://icclab_turtlebot/meshes/gripper/schunk_epg40/schunk_epg40_finger_base.stl" scale="1 1 1"/>
+               <mesh filename="package://icclab_summit_xl/meshes/gripper/schunk_epg40/schunk_epg40_finger_base.stl" scale="1 1 1"/>
+            </geometry>
+            <material name="grey">
+               <color rgba="0.5 0.5 0.5 1"/>
+            </material>
+         </visual>
+         <collision>
+            <origin xyz="0.0 0 0" rpy="0 0 0" />
+            <geometry>
+               <mesh filename="package://icclab_summit_xl/meshes/gripper/schunk_epg40/schunk_epg40_finger_base.stl" scale="1 1 1"/>
             </geometry>
          </collision>
@@ -100,14 +100,14 @@
             <origin xyz="0.0 0 0" rpy="0 0 0" />
             <geometry>
-               <mesh filename="package://icclab_turtlebot/meshes/gripper/schunk_epg40/schunk_epg40_finger.stl" scale="1 1 1"/>
-            </geometry>
-            <material name="grey">
-               <color rgba="0.5 0.5 0.5 1"/>
-            </material>
-         </visual>
-         <collision>
-            <origin xyz="0.0 0 0" rpy="0 0 0" />
-            <geometry>
-               <mesh filename="package://icclab_turtlebot/meshes/gripper/schunk_epg40/schunk_epg40_finger.stl" scale="1 1 1"/>
+               <mesh filename="package://icclab_summit_xl/meshes/gripper/schunk_epg40/schunk_epg40_finger.stl" scale="1 1 1"/>
+            </geometry>
+            <material name="grey">
+               <color rgba="0.5 0.5 0.5 1"/>
+            </material>
+         </visual>
+         <collision>
+            <origin xyz="0.0 0 0" rpy="0 0 0" />
+            <geometry>
+               <mesh filename="package://icclab_summit_xl/meshes/gripper/schunk_epg40/schunk_epg40_finger.stl" scale="1 1 1"/>
             </geometry>
          </collision>
@@ -140,14 +140,14 @@
             <origin xyz="0.0 0 0" rpy="0 0 0" />
             <geometry>
-               <mesh filename="package://icclab_turtlebot/meshes/gripper/schunk_epg40/schunk_epg40_finger_base.stl" scale="1 1 1"/>
-            </geometry>
-            <material name="grey">
-               <color rgba="0.5 0.5 0.5 1"/>
-            </material>
-         </visual>
-         <collision>
-            <origin xyz="0.0 0 0" rpy="0 0 0" />
-            <geometry>
-               <mesh filename="package://icclab_turtlebot/meshes/gripper/schunk_epg40/schunk_epg40_finger_base.stl" scale="1 1 1"/>
+               <mesh filename="package://icclab_summit_xl/meshes/gripper/schunk_epg40/schunk_epg40_finger_base.stl" scale="1 1 1"/>
+            </geometry>
+            <material name="grey">
+               <color rgba="0.5 0.5 0.5 1"/>
+            </material>
+         </visual>
+         <collision>
+            <origin xyz="0.0 0 0" rpy="0 0 0" />
+            <geometry>
+               <mesh filename="package://icclab_summit_xl/meshes/gripper/schunk_epg40/schunk_epg40_finger_base.stl" scale="1 1 1"/>
             </geometry>
          </collision>
@@ -167,5 +167,5 @@
             <origin xyz="0.0 0 0" rpy="0 0 0" />
             <geometry>
-               <mesh filename="package://icclab_turtlebot/meshes/gripper/schunk_epg40/schunk_epg40_finger.stl" scale="1 1 1"/>
+               <mesh filename="package://icclab_summit_xl/meshes/gripper/schunk_epg40/schunk_epg40_finger.stl" scale="1 1 1"/>
             </geometry>
             <material name="grey">
@@ -176,5 +176,5 @@
             <origin xyz="0.0 0 0" rpy="0 0 0" />
             <geometry>
-               <mesh filename="package://icclab_turtlebot/meshes/gripper/schunk_epg40/schunk_epg40_finger.stl" scale="1 1 1"/>
+               <mesh filename="package://icclab_summit_xl/meshes/gripper/schunk_epg40/schunk_epg40_finger.stl" scale="1 1 1"/>
             </geometry>
          </collision>

File: urdf/sensors/scanse.urdf.xacro (robot description, xacro)
@@ -22,5 +22,5 @@
         <origin xyz="0 0 0" rpy="0 0 0"/>
         <geometry>
-          <mesh filename="package://icclab_turtlebot/meshes/sweep_lidar.stl"/>
+          <mesh filename="package://icclab_summit_xl/meshes/sweep_lidar.stl"/>
         </geometry>
       </visual>

Commit message: changed camera position in model, updated start script on robot, created remote grasping launch file

File: robots/irlab_summit_xls_std.urdf.xacro (robot description, xacro)
@@ -100,5 +100,5 @@
 		<!-- Camera on gripper -->
 		<sensor_r430 prefix="arm" prefix_topic="arm_camera" parent="arm_tool0">
-      <origin xyz="0 0.045 -0.015" rpy="${-PI/2} ${-PI/2} 0"/>
+      <origin xyz="0 -0.065 -0.015" rpy="${-PI/2} ${-PI/2} ${PI}"/>
     </sensor_r430>
    </xacro:macro>

Commit message: changed parent link of arm camera to arm_wrist_3_link because camera should not rotate

File: robots/irlab_summit_xls_std.urdf.xacro (robot description, xacro)
@@ -99,6 +99,6 @@
 		</xacro:schunk_egp_40>
 		<!-- Camera on gripper -->
-		<sensor_r430 prefix="arm" prefix_topic="arm_camera" parent="arm_tool0">
-      <origin xyz="0 -0.065 -0.015" rpy="${-PI/2} ${-PI/2} ${PI}"/>
+		<sensor_r430 prefix="arm" prefix_topic="arm_camera" parent="arm_wrist_3_link">
+      <origin xyz="0 0.07 0.06" rpy="0 0 ${PI/2}"/>
     </sensor_r430>
    </xacro:macro>

Commit message: changed parent link of arm camera to arm_wrist_2_link because camera should not rotate

File: robots/irlab_summit_xls_std.urdf.xacro (robot description, xacro)
@@ -99,6 +99,6 @@
 		</xacro:schunk_egp_40>
 		<!-- Camera on gripper -->
-		<sensor_r430 prefix="arm" prefix_topic="arm_camera" parent="arm_wrist_3_link">
-      <origin xyz="0 0.07 0.06" rpy="0 0 ${PI/2}"/>
+		<sensor_r430 prefix="arm" prefix_topic="arm_camera" parent="arm_wrist_2_link">
+      <origin xyz="0 0.07 0.155" rpy="0 0 ${PI/2}"/>
     </sensor_r430>
    </xacro:macro>

Commit message: adds intel camera mount to model

File: robots/irlab_summit_xls_std.urdf.xacro (robot description, xacro)
@@ -20,4 +20,6 @@
 	<xacro:include filename="$(find icclab_summit_xl)/urdf/sensors/scanse.urdf.xacro" />
 	<xacro:include filename="$(find icclab_summit_xl)/urdf/sensors/intel_d435.urdf.xacro" />
+	<!-- Intel camera mount -->
+	<xacro:include filename="$(find icclab_summit_xl)/urdf/sensors/intel_camera_mount.urdf.xacro" />
 	<xacro:property name="PI" value="3.1415926535897931"/>
 	<xacro:property name="wheel_offset_x" value="0.2225" />
@@ -104,4 +106,8 @@
       <origin xyz="0 0.07 0.155" rpy="0 0 ${PI/2}"/>
     </sensor_r430_icclab>
+		<!-- Camera mount -->
+		<xacro:camera_mount prefix="arm" parent="arm_wrist_2_link">
+			 <origin xyz="-0.005 0.04 0.100" rpy="${PI/2} 0 ${PI}" />
+		</xacro:camera_mount>
    </xacro:macro>
    <xacro:ros_control/>

Commit message: Updated the d435 camera model

File: robots/irlab_summit_xls_std.urdf.xacro (robot description, xacro)
@@ -20,4 +20,5 @@
 	<xacro:include filename="$(find icclab_summit_xl)/urdf/sensors/scanse.urdf.xacro" />
 	<xacro:include filename="$(find icclab_summit_xl)/urdf/sensors/intel_d435.urdf.xacro" />
+	<!--<xacro:include filename="$(find icclab_summit_xl)/urdf/sensors/intel_d410.urdf.xacro" />-->
 	<!-- Intel camera mount -->
 	<xacro:include filename="$(find icclab_summit_xl)/urdf/sensors/intel_camera_mount.urdf.xacro" />
@@ -103,7 +104,10 @@
 		<!-- Camera on gripper -->
 		<!-- had to copy and modidy camera to avoid name clash with robotnik defined sensors -->
-		<sensor_r430_icclab prefix="arm" prefix_topic="arm_camera" parent="arm_wrist_2_link">
-      <origin xyz="0 0.07 0.155" rpy="0 0 ${PI/2}"/>
-    </sensor_r430_icclab>
+		<sensor_d435_icclab prefix="arm" prefix_topic="arm_camera" parent="arm_wrist_2_link">
+     		<origin xyz="0 0.07 0.155" rpy="0 0 ${PI/2}"/>
+   		</sensor_d435_icclab>
+		<!-- <sensor_d415_icclab prefix="arm" prefix_topic="arm_camera" parent="arm_wrist_2_link">
+     		<origin xyz="0 0.07 0.155" rpy="0 0 ${PI/2}"/>
+   		</sensor_d415_icclab> -->
 		<!-- Camera mount -->
 		<xacro:camera_mount prefix="arm" parent="arm_wrist_2_link">

Commit message: Added the d415 camera model

File: robots/irlab_summit_xls_std.urdf.xacro (robot description, xacro)
@@ -19,6 +19,6 @@
 	<!-- ICCLab sensors -->
 	<xacro:include filename="$(find icclab_summit_xl)/urdf/sensors/scanse.urdf.xacro" />
-	<xacro:include filename="$(find icclab_summit_xl)/urdf/sensors/intel_d435.urdf.xacro" />
-	<!--<xacro:include filename="$(find icclab_summit_xl)/urdf/sensors/intel_d410.urdf.xacro" />-->
+	<!--<xacro:include filename="$(find icclab_summit_xl)/urdf/sensors/intel_d435.urdf.xacro" /> -->
+	<xacro:include filename="$(find icclab_summit_xl)/urdf/sensors/intel_d415.urdf.xacro" />
 	<!-- Intel camera mount -->
 	<xacro:include filename="$(find icclab_summit_xl)/urdf/sensors/intel_camera_mount.urdf.xacro" />
@@ -104,10 +104,10 @@
 		<!-- Camera on gripper -->
 		<!-- had to copy and modidy camera to avoid name clash with robotnik defined sensors -->
-		<sensor_d435_icclab prefix="arm" prefix_topic="arm_camera" parent="arm_wrist_2_link">
+		<!--<sensor_d435_icclab prefix="arm" prefix_topic="arm_camera" parent="arm_wrist_2_link">
      		<origin xyz="0 0.07 0.155" rpy="0 0 ${PI/2}"/>
-   		</sensor_d435_icclab>
-		<!-- <sensor_d415_icclab prefix="arm" prefix_topic="arm_camera" parent="arm_wrist_2_link">
-     		<origin xyz="0 0.07 0.155" rpy="0 0 ${PI/2}"/>
-   		</sensor_d415_icclab> -->
+   		</sensor_d435_icclab> -->
+		<sensor_d415_icclab prefix="arm" prefix_topic="arm_camera" parent="arm_wrist_2_link">
+     		<origin xyz="0 0.05 0.155" rpy="0 0 ${PI/2}"/> <!-- Note the position seems to be wrong in gazebo beacuase we use the d435 mesh file, but it is correct considering the real size of the camera-->
+   		</sensor_d415_icclab>
 		<!-- Camera mount -->
 		<xacro:camera_mount prefix="arm" parent="arm_wrist_2_link">

Commit message: aligns front and rear LIDARs with front depth camera

File: robots/irlab_summit_xls_std.urdf.xacro (robot description, xacro)
@@ -29,13 +29,13 @@
 	<xacro:property name="wheel_offset_z" value="0.0" />
 	<!-- <xacro:property name="front_laser_offset_x" value="0.377"/>    -->
-	<xacro:property name="front_laser_offset_x" value="0.357"/>
+	<xacro:property name="front_laser_offset_x" value="0.34"/>
 	<!-- <xacro:property name="front_laser_offset_y" value="-0.20957"/>     -->
-	<xacro:property name="front_laser_offset_y" value="-0.25957"/>
+	<xacro:property name="front_laser_offset_y" value="-0.235"/>
 	<!-- <xacro:property name="front_laser_offset_z" value="0.2024"/> -->
 	<xacro:property name="front_laser_offset_z" value="0.1566"/>
 	<!-- <xacro:property name="rear_laser_offset_x" value="-0.377"/> -->
-	<xacro:property name="rear_laser_offset_x" value="-0.357"/>
+	<xacro:property name="rear_laser_offset_x" value="-0.34"/>
 	<!-- <xacro:property name="rear_laser_offset_y" value="0.20957"/>     -->
-	<xacro:property name="rear_laser_offset_y" value="0.25957"/>
+	<xacro:property name="rear_laser_offset_y" value="0.235"/>
 	<!-- <xacro:property name="rear_laser_offset_z" value="0.2024"/> -->
 	<xacro:property name="rear_laser_offset_z" value="0.1566"/>

Commit message: Using UR5 joint limited model for better moveit planning

File: robots/irlab_summit_xls_std.urdf.xacro (robot description, xacro)
@@ -91,5 +91,5 @@
 		</xacro:scanse>
 		<!-- UR5 Arm -->
-		<xacro:ur5_robot prefix="arm_" joint_limited="false">
+		<xacro:ur5_robot prefix="arm_" joint_limited="true">
 		</xacro:ur5_robot>
 		<joint name="$(arg prefix)arm_base_joint" type="fixed">
@@ -108,5 +108,5 @@
    		</sensor_d435_icclab> -->
 		<sensor_d415_icclab prefix="arm" prefix_topic="arm_camera" parent="arm_wrist_2_link">
-     		<origin xyz="0 0.05 0.155" rpy="0 0 ${PI/2}"/> <!-- Note the position seems to be wrong in gazebo beacuase we use the d435 mesh file, but it is correct considering the real size of the camera-->
+     		<origin xyz="0 0.05 0.155" rpy="0 0 ${PI/2}"/> <!-- Note the position seems to be wrong in gazebo beacuase we use the d435 mesh file, but it is correct considering the realsize of the camera-->
    		</sensor_d415_icclab>
 		<!-- Camera mount -->
