Commit message: Updated model with calibrated cameras

File: robots/irlab_summit_xls_std.urdf.xacro (robot description, xacro)
@@ -19,6 +19,6 @@
 	<!-- ICCLab sensors -->
 	<xacro:include filename="$(find icclab_summit_xl)/urdf/sensors/scanse.urdf.xacro" />
-	<!--<xacro:include filename="$(find icclab_summit_xl)/urdf/sensors/intel_d435.urdf.xacro" /> -->
-	<xacro:include filename="$(find icclab_summit_xl)/urdf/sensors/intel_d415.urdf.xacro" />
+	<xacro:include filename="$(find icclab_summit_xl)/urdf/sensors/intel_d435.urdf.xacro" />
+<!--	<xacro:include filename="$(find icclab_summit_xl)/urdf/sensors/intel_d415.urdf.xacro" /> -->
 	<!-- Intel camera mount -->
 	<xacro:include filename="$(find icclab_summit_xl)/urdf/sensors/intel_camera_mount.urdf.xacro" />
@@ -46,5 +46,5 @@
 	<xacro:property name="imu_offset_y" value="-0.15"/>
 	<xacro:property name="imu_offset_z" value="0.18"/>
-	<xacro:property name="front_rgbd_camera_offset_x" value="0.324"/>
+	<xacro:property name="front_rgbd_camera_offset_x" value="0.35"/>
 	<xacro:property name="front_rgbd_camera_offset_y" value="0.012"/>
 	<xacro:property name="front_rgbd_camera_offset_z" value="0.230"/>
@@ -104,13 +104,13 @@
 		<!-- Camera on gripper -->
 		<!-- had to copy and modidy camera to avoid name clash with robotnik defined sensors -->
-		<!--<sensor_d435_icclab prefix="arm" prefix_topic="arm_camera" parent="arm_wrist_2_link">
-     		<origin xyz="0 0.07 0.155" rpy="0 0 ${PI/2}"/>
-   		</sensor_d435_icclab> -->
-		<sensor_d415_icclab prefix="arm" prefix_topic="arm_camera" parent="arm_wrist_2_link">
-     		<origin xyz="0 0.05 0.155" rpy="0 0 ${PI/2}"/> <!-- Note the position seems to be wrong in gazebo beacuase we use the d435 mesh file, but it is correct considering the realsize of the camera-->
-   		</sensor_d415_icclab>
+		<sensor_d435_icclab prefix="arm" prefix_topic="arm_camera" parent="arm_wrist_2_link">
+     		<origin xyz="0 0.07 0.14" rpy="0 0 ${PI/2}"/>
+   		</sensor_d435_icclab>
+<!--		<sensor_d415_icclab prefix="arm" prefix_topic="arm_camera" parent="arm_wrist_2_link">
+     		<origin xyz="0 0.05 0.155" rpy="0 0 ${PI/2}"/>--> <!-- Note the position seems to be wrong in gazebo beacuase we use the d435 mesh file, but it is correct considering the realsize of the camera-->
+   		<!--</sensor_d415_icclab>-->
 		<!-- Camera mount -->
 		<xacro:camera_mount prefix="arm" parent="arm_wrist_2_link">
-			 <origin xyz="-0.005 0.04 0.100" rpy="${PI/2} 0 ${PI}" />
+			 <origin xyz="-0.005 0.04 0.09" rpy="${PI/2} 0 ${PI}" />
 		</xacro:camera_mount>
    </xacro:macro>

Commit message: Updated model with calibrated cameras

File: robots/irlab_summit_xls_std.urdf.xacro (robot description, xacro)
@@ -105,5 +105,5 @@
 		<!-- had to copy and modidy camera to avoid name clash with robotnik defined sensors -->
 		<sensor_d435_icclab prefix="arm" prefix_topic="arm_camera" parent="arm_wrist_2_link">
-     		<origin xyz="0 0.07 0.14" rpy="0 0 ${PI/2}"/>
+     		<origin xyz="0 0.07 0.145" rpy="0 0 ${PI/2}"/>
    		</sensor_d435_icclab>
 <!--		<sensor_d415_icclab prefix="arm" prefix_topic="arm_camera" parent="arm_wrist_2_link">
@@ -112,5 +112,5 @@
 		<!-- Camera mount -->
 		<xacro:camera_mount prefix="arm" parent="arm_wrist_2_link">
-			 <origin xyz="-0.005 0.04 0.09" rpy="${PI/2} 0 ${PI}" />
+			 <origin xyz="-0.005 0.04 0.095" rpy="${PI/2} 0 ${PI}" />
 		</xacro:camera_mount>
    </xacro:macro>

Commit message: Added collision boxes to wrist 2 and wrist 3

File: robots/irlab_summit_xls_std.urdf.xacro (robot description, xacro)
@@ -23,4 +23,8 @@
 	<!-- Intel camera mount -->
 	<xacro:include filename="$(find icclab_summit_xl)/urdf/sensors/intel_camera_mount.urdf.xacro" />
+	<!-- Collision box on arm wrist 3 -->
+	<xacro:include filename="$(find icclab_summit_xl)/robots/ur5_arm_wrist3_collision_box.urdf.xacro" />
+	<!-- Collision box on arm wrist 2 -->
+	<xacro:include filename="$(find icclab_summit_xl)/robots/ur5_arm_wrist2_collision_box.urdf.xacro" />
 	<xacro:property name="PI" value="3.1415926535897931"/>
 	<xacro:property name="wheel_offset_x" value="0.2225" />
@@ -114,4 +118,12 @@
 			 <origin xyz="-0.005 0.04 0.095" rpy="${PI/2} 0 ${PI}" />
 		</xacro:camera_mount>
+		<!-- Collision box wrist 3 -->
+		<xacro:collision_box_wrist3 prefix="arm" parent="arm_wrist_3_link">
+			 <origin xyz="0 -0.06 0" rpy="0 0 0" />
+		</xacro:collision_box_wrist3>
+		<!-- Collision box wrist 2 -->
+		<xacro:collision_box_wrist2 prefix="arm" parent="arm_wrist_2_link">
+			 <origin xyz="0 0 -0.06" rpy="${PI/2} 0 0" />
+		</xacro:collision_box_wrist2>
    </xacro:macro>
    <xacro:ros_control/>

Commit message: Rotated camera 90deg and added cable collision box

File: robots/irlab_summit_xls_std.urdf.xacro (robot description, xacro)
@@ -23,4 +23,6 @@
 	<!-- Intel camera mount -->
 	<xacro:include filename="$(find icclab_summit_xl)/urdf/sensors/intel_camera_mount.urdf.xacro" />
+	<!-- Collision box on arm camera cable -->
+	<xacro:include filename="$(find icclab_summit_xl)/robots/ur5_arm_camera_cable_collision_box.urdf.xacro" />
 	<!-- Collision box on arm wrist 3 -->
 	<xacro:include filename="$(find icclab_summit_xl)/robots/ur5_arm_wrist3_collision_box.urdf.xacro" />
@@ -109,5 +111,7 @@
 		<!-- had to copy and modidy camera to avoid name clash with robotnik defined sensors -->
 		<sensor_d435_icclab prefix="arm" prefix_topic="arm_camera" parent="arm_wrist_2_link">
-     		<origin xyz="0 0.07 0.145" rpy="0 0 ${PI/2}"/>
+     		<!-- <origin xyz="0 0.07 0.145" rpy="0 0 ${PI/2}"/> -->
+			<!--<origin xyz="-0.075 0.07 0.09" rpy="${PI/2} 0 ${PI/2}"/>  --><!-- camera on the one side -->
+			<origin xyz="0.075 0.07 0.1" rpy="${-PI/2} 0 ${PI/2}"/> <!-- camera on the other oner side -->
    		</sensor_d435_icclab>
 <!--		<sensor_d415_icclab prefix="arm" prefix_topic="arm_camera" parent="arm_wrist_2_link">
@@ -116,6 +120,12 @@
 		<!-- Camera mount -->
 		<xacro:camera_mount prefix="arm" parent="arm_wrist_2_link">
-			 <origin xyz="-0.005 0.04 0.095" rpy="${PI/2} 0 ${PI}" />
+			<!-- <origin xyz="-0.005 0.04 0.095" rpy="${PI/2} 0 ${PI}" /> -->
+			<!-- <origin xyz="-0.005 0.04 0.095" rpy=" ${PI/2} ${PI/2} ${PI}" /> --> <!-- camera on the one side -->
+			<origin xyz="0 0.04 0.1" rpy=" ${PI/2} ${-PI/2} ${PI}" /> <!-- camera on the other one side -->
 		</xacro:camera_mount>
+		<!-- Collision box camera cable -->
+		<xacro:collision_box_camera_cable prefix="arm" parent="arm_camera_link">
+			 <origin xyz="-0.02 -0.08 0" rpy="0 0 0" />
+		</xacro:collision_box_camera_cable>
 		<!-- Collision box wrist 3 -->
 		<xacro:collision_box_wrist3 prefix="arm" parent="arm_wrist_3_link">

Commit message: Rotated camera 90deg and added cable collision box

File: robots/irlab_summit_xls_std.urdf.xacro (robot description, xacro)
@@ -112,6 +112,6 @@
 		<sensor_d435_icclab prefix="arm" prefix_topic="arm_camera" parent="arm_wrist_2_link">
      		<!-- <origin xyz="0 0.07 0.145" rpy="0 0 ${PI/2}"/> -->
-			<!--<origin xyz="-0.075 0.07 0.09" rpy="${PI/2} 0 ${PI/2}"/>  --><!-- camera on the one side -->
-			<origin xyz="0.075 0.07 0.1" rpy="${-PI/2} 0 ${PI/2}"/> <!-- camera on the other oner side -->
+			<origin xyz="-0.075 0.07 0.09" rpy="${PI/2} 0 ${PI/2}"/>  <!-- camera on the one side -->
+			<!--<origin xyz="0.075 0.07 0.1" rpy="${-PI/2} 0 ${PI/2}"/> --><!-- camera on the other oner side -->
    		</sensor_d435_icclab>
 <!--		<sensor_d415_icclab prefix="arm" prefix_topic="arm_camera" parent="arm_wrist_2_link">
@@ -121,6 +121,6 @@
 		<xacro:camera_mount prefix="arm" parent="arm_wrist_2_link">
 			<!-- <origin xyz="-0.005 0.04 0.095" rpy="${PI/2} 0 ${PI}" /> -->
-			<!-- <origin xyz="-0.005 0.04 0.095" rpy=" ${PI/2} ${PI/2} ${PI}" /> --> <!-- camera on the one side -->
-			<origin xyz="0 0.04 0.1" rpy=" ${PI/2} ${-PI/2} ${PI}" /> <!-- camera on the other one side -->
+			 <origin xyz="0 0.04 0.09" rpy=" ${PI/2} ${PI/2} ${PI}" />  <!-- camera on the one side -->
+			<!--<origin xyz="0 0.04 0.1" rpy=" ${PI/2} ${-PI/2} ${PI}" /> --><!-- camera on the other one side -->
 		</xacro:camera_mount>
 		<!-- Collision box camera cable -->

Commit message: Rotated camera 90deg and added cable collision box

File: robots/irlab_summit_xls_std.urdf.xacro (robot description, xacro)
@@ -112,5 +112,5 @@
 		<sensor_d435_icclab prefix="arm" prefix_topic="arm_camera" parent="arm_wrist_2_link">
      		<!-- <origin xyz="0 0.07 0.145" rpy="0 0 ${PI/2}"/> -->
-			<origin xyz="-0.075 0.07 0.09" rpy="${PI/2} 0 ${PI/2}"/>  <!-- camera on the one side -->
+			<origin xyz="-0.075 0.07 0.09" rpy="${PI/2} 0 ${-PI/2}"/>  <!-- camera on the one side -->
 			<!--<origin xyz="0.075 0.07 0.1" rpy="${-PI/2} 0 ${PI/2}"/> --><!-- camera on the other oner side -->
    		</sensor_d435_icclab>

Commit message: Rotated camera 90deg and added cable collision box

File: robots/irlab_summit_xls_std.urdf.xacro (robot description, xacro)
@@ -112,5 +112,5 @@
 		<sensor_d435_icclab prefix="arm" prefix_topic="arm_camera" parent="arm_wrist_2_link">
      		<!-- <origin xyz="0 0.07 0.145" rpy="0 0 ${PI/2}"/> -->
-			<origin xyz="-0.075 0.07 0.09" rpy="${PI/2} 0 ${-PI/2}"/>  <!-- camera on the one side -->
+			<origin xyz="-0.075 0.07 0.09" rpy="${-PI/2} 0 ${PI/2}"/>  <!-- camera on the one side -->
 			<!--<origin xyz="0.075 0.07 0.1" rpy="${-PI/2} 0 ${PI/2}"/> --><!-- camera on the other oner side -->
    		</sensor_d435_icclab>

Commit message: Rotated camera 90deg and added cable collision box

File: robots/irlab_summit_xls_std.urdf.xacro (robot description, xacro)
@@ -112,5 +112,5 @@
 		<sensor_d435_icclab prefix="arm" prefix_topic="arm_camera" parent="arm_wrist_2_link">
      		<!-- <origin xyz="0 0.07 0.145" rpy="0 0 ${PI/2}"/> -->
-			<origin xyz="-0.075 0.07 0.09" rpy="${-PI/2} 0 ${PI/2}"/>  <!-- camera on the one side -->
+			<origin xyz="-0.045 0.07 0.09" rpy="${-PI/2} 0 ${PI/2}"/>  <!-- camera on the one side -->
 			<!--<origin xyz="0.075 0.07 0.1" rpy="${-PI/2} 0 ${PI/2}"/> --><!-- camera on the other oner side -->
    		</sensor_d435_icclab>

Commit message: Rotated camera 90deg and added cable collision box

File: robots/irlab_summit_xls_std.urdf.xacro (robot description, xacro)
@@ -112,5 +112,5 @@
 		<sensor_d435_icclab prefix="arm" prefix_topic="arm_camera" parent="arm_wrist_2_link">
      		<!-- <origin xyz="0 0.07 0.145" rpy="0 0 ${PI/2}"/> -->
-			<origin xyz="-0.045 0.07 0.09" rpy="${-PI/2} 0 ${PI/2}"/>  <!-- camera on the one side -->
+			<origin xyz="-0.05 0.07 0.09" rpy="${-PI/2} 0 ${PI/2}"/>  <!-- camera on the one side -->
 			<!--<origin xyz="0.075 0.07 0.1" rpy="${-PI/2} 0 ${PI/2}"/> --><!-- camera on the other oner side -->
    		</sensor_d435_icclab>

Commit message: Rotated camera 90deg and added cable collision box

File: robots/irlab_summit_xls_std.urdf.xacro (robot description, xacro)
@@ -112,5 +112,5 @@
 		<sensor_d435_icclab prefix="arm" prefix_topic="arm_camera" parent="arm_wrist_2_link">
      		<!-- <origin xyz="0 0.07 0.145" rpy="0 0 ${PI/2}"/> -->
-			<origin xyz="-0.05 0.07 0.09" rpy="${-PI/2} 0 ${PI/2}"/>  <!-- camera on the one side -->
+			<origin xyz="-0.05 0.07 0.095" rpy="${-PI/2} 0 ${PI/2}"/>  <!-- camera on the one side -->
 			<!--<origin xyz="0.075 0.07 0.1" rpy="${-PI/2} 0 ${PI/2}"/> --><!-- camera on the other oner side -->
    		</sensor_d435_icclab>

Commit message: Recalibrating front camera

File: robots/irlab_summit_xls_std.urdf.xacro (robot description, xacro)
@@ -52,7 +52,7 @@
 	<xacro:property name="imu_offset_y" value="-0.15"/>
 	<xacro:property name="imu_offset_z" value="0.18"/>
-	<xacro:property name="front_rgbd_camera_offset_x" value="0.35"/>
+	<xacro:property name="front_rgbd_camera_offset_x" value="0.324"/>  <!-- 328 --> <!-- 35 leo-->
 	<xacro:property name="front_rgbd_camera_offset_y" value="0.012"/>
-	<xacro:property name="front_rgbd_camera_offset_z" value="0.230"/>
+	<xacro:property name="front_rgbd_camera_offset_z" value="0.230"/>  <!-- 214 -->
   <xacro:property name="base_arm_x" value="0.225"/>
   <xacro:property name="base_arm_y" value="0.0"/>

Commit message: Recalibrating front camera

File: robots/irlab_summit_xls_std.urdf.xacro (robot description, xacro)
@@ -52,5 +52,5 @@
 	<xacro:property name="imu_offset_y" value="-0.15"/>
 	<xacro:property name="imu_offset_z" value="0.18"/>
-	<xacro:property name="front_rgbd_camera_offset_x" value="0.324"/>  <!-- 328 --> <!-- 35 leo-->
+	<xacro:property name="front_rgbd_camera_offset_x" value="0.35"/>  <!-- 328 --> <!-- 35 leo-->
 	<xacro:property name="front_rgbd_camera_offset_y" value="0.012"/>
 	<xacro:property name="front_rgbd_camera_offset_z" value="0.230"/>  <!-- 214 -->
@@ -112,5 +112,5 @@
 		<sensor_d435_icclab prefix="arm" prefix_topic="arm_camera" parent="arm_wrist_2_link">
      		<!-- <origin xyz="0 0.07 0.145" rpy="0 0 ${PI/2}"/> -->
-			<origin xyz="-0.05 0.07 0.095" rpy="${-PI/2} 0 ${PI/2}"/>  <!-- camera on the one side -->
+			<origin xyz="-0.05 0.085 0.095" rpy="${-PI/2} 0 ${PI/2}"/>  <!-- camera on the one side -->
 			<!--<origin xyz="0.075 0.07 0.1" rpy="${-PI/2} 0 ${PI/2}"/> --><!-- camera on the other oner side -->
    		</sensor_d435_icclab>
@@ -121,5 +121,5 @@
 		<xacro:camera_mount prefix="arm" parent="arm_wrist_2_link">
 			<!-- <origin xyz="-0.005 0.04 0.095" rpy="${PI/2} 0 ${PI}" /> -->
-			 <origin xyz="0 0.04 0.09" rpy=" ${PI/2} ${PI/2} ${PI}" />  <!-- camera on the one side -->
+			 <origin xyz="0 0.055 0.09" rpy=" ${PI/2} ${PI/2} ${PI}" />  <!-- camera on the one side -->
 			<!--<origin xyz="0 0.04 0.1" rpy=" ${PI/2} ${-PI/2} ${PI}" /> --><!-- camera on the other one side -->
 		</xacro:camera_mount>

Commit message: Recalibrating front camera

File: robots/irlab_summit_xls_std.urdf.xacro (robot description, xacro)
@@ -112,5 +112,5 @@
 		<sensor_d435_icclab prefix="arm" prefix_topic="arm_camera" parent="arm_wrist_2_link">
      		<!-- <origin xyz="0 0.07 0.145" rpy="0 0 ${PI/2}"/> -->
-			<origin xyz="-0.05 0.085 0.095" rpy="${-PI/2} 0 ${PI/2}"/>  <!-- camera on the one side -->
+			<origin xyz="-0.05 0.071 0.095" rpy="${-PI/2} 0 ${PI/2}"/>  <!-- camera on the one side -->
 			<!--<origin xyz="0.075 0.07 0.1" rpy="${-PI/2} 0 ${PI/2}"/> --><!-- camera on the other oner side -->
    		</sensor_d435_icclab>
@@ -121,5 +121,5 @@
 		<xacro:camera_mount prefix="arm" parent="arm_wrist_2_link">
 			<!-- <origin xyz="-0.005 0.04 0.095" rpy="${PI/2} 0 ${PI}" /> -->
-			 <origin xyz="0 0.055 0.09" rpy=" ${PI/2} ${PI/2} ${PI}" />  <!-- camera on the one side -->
+			 <origin xyz="0 0.041 0.09" rpy=" ${PI/2} ${PI/2} ${PI}" />  <!-- camera on the one side -->
 			<!--<origin xyz="0 0.04 0.1" rpy=" ${PI/2} ${-PI/2} ${PI}" /> --><!-- camera on the other one side -->
 		</xacro:camera_mount>

Commit message: replaces scanse sweep lidar with rplidar in simulation and model

File: robots/irlab_summit_xls_std.urdf.xacro (robot description, xacro)
@@ -19,4 +19,5 @@
 	<!-- ICCLab sensors -->
 	<xacro:include filename="$(find icclab_summit_xl)/urdf/sensors/scanse.urdf.xacro" />
+	<xacro:include filename="$(find icclab_summit_xl)/urdf/sensors/rplidar.urdf.xacro" />
 	<xacro:include filename="$(find icclab_summit_xl)/urdf/sensors/intel_d435.urdf.xacro" />
 <!--	<xacro:include filename="$(find icclab_summit_xl)/urdf/sensors/intel_d415.urdf.xacro" /> -->
@@ -35,5 +36,5 @@
 	<xacro:property name="wheel_offset_z" value="0.0" />
 	<!-- <xacro:property name="front_laser_offset_x" value="0.377"/>    -->
-	<xacro:property name="front_laser_offset_x" value="0.34"/>
+	<xacro:property name="front_laser_offset_x" value="0.346"/>
 	<!-- <xacro:property name="front_laser_offset_y" value="-0.20957"/>     -->
 	<xacro:property name="front_laser_offset_y" value="-0.235"/>
@@ -88,8 +89,8 @@
 			<origin xyz="${front_rgbd_camera_offset_x} ${front_rgbd_camera_offset_y} ${front_rgbd_camera_offset_z}" rpy="0 0 0"/>
 		</xacro:sensor_orbbec_astra>
-		<!-- Scanse front lidar -->
-		<xacro:scanse prefix="$(arg prefix)front_laser" parent="$(arg prefix)base_link" prefix_topic="scan_front">
-			<origin xyz="${front_laser_offset_x} ${front_laser_offset_y} ${front_laser_offset_z}" rpy="0 0 ${-PI/4.0}"/>
-		</xacro:scanse>
+		<!-- RPLidar front lidar -->
+		<xacro:rplidar prefix="$(arg prefix)front_laser" parent="$(arg prefix)base_link" prefix_topic="scan_front">
+			<origin xyz="${front_laser_offset_x} ${front_laser_offset_y} ${front_laser_offset_z}" rpy="0 0 ${PI/2}"/>
+		</xacro:rplidar>
 		<!-- Scanse rear lidar -->
 		<xacro:scanse prefix="$(arg prefix)rear_laser" parent="$(arg prefix)base_link" prefix_topic="scan_rear">

File: urdf/sensors/rplidar.urdf.xacro (robot description, xacro)
@@ -1,6 +1,6 @@
 <?xml version=  "1.0"?>
-<robot name="scanse"
+<robot name="rplidar"
   xmlns:xacro="http://www.ros.org/wiki/xacro">
-  <xacro:macro name="scanse" params="prefix parent prefix_topic:='front_laser' *origin min_angle:=-2.35 max_angle:=2.35">
+  <xacro:macro name="rplidar" params="prefix parent prefix_topic:='front_laser' *origin min_angle:=1.5708 max_angle:=6.2832">
     <joint name="${prefix}_base_joint" type="fixed">
       <!-- FRONT MOUNT  -->
@@ -14,19 +14,19 @@
     <link name="${prefix}_base_link">
       <collision>        <!-- added -->
-        <origin xyz="0 0 0.02" rpy="0 0 0"/>
+        <origin xyz="0.005 0 0.02" rpy="0 0 0"/>
         <geometry>
-          <cylinder length="0.06" radius="0.035"/>
+          <cylinder length="0.0315" radius="0.040"/>
         </geometry>
       </collision>
       <visual>
-        <origin xyz="0 0 0" rpy="0 0 0"/>
+        <origin xyz="0 0 0.02" rpy="0 0 0"/>
         <geometry>
-          <mesh filename="package://icclab_summit_xl/meshes/sensors/sweep_lidar.stl"/>
+          <mesh filename="package://icclab_summit_xl/meshes/sensors/lds.stl" scale="0.001 0.001 0.001"/>
         </geometry>
       </visual>
       <inertial>
-        <mass value="1e-5" />
+        <mass value="0.114" />
         <origin xyz="0 0 0" rpy="0 0 0"/>
-        <inertia ixx="1e-6" ixy="0" ixz="0" iyy="1e-6" iyz="0" izz="1e-6" />
+        <inertia ixx="0.001" ixy="0" ixz="0" iyy="0.001" iyz="0" izz="0.001" />
       </inertial>
     </link>
@@ -39,8 +39,8 @@
     </joint>
     <!-- simulation -->
-    <sensor_scanse_gazebo/>
+    <sensor_rplidar_gazebo/>
   </xacro:macro>
 <!-- uses ROS Laser Scanner Controller plugin -->
-  <xacro:macro name="sensor_scanse_gazebo">
+  <xacro:macro name="sensor_rplidar_gazebo">
     <gazebo reference="${prefix}_link">
       <sensor type="ray" name="${prefix}_sensor">

Commit message: Moved front camera for calibrated front/arm camera pcl

File: robots/irlab_summit_xls_std.urdf.xacro (robot description, xacro)
@@ -52,7 +52,7 @@
 	<xacro:property name="imu_offset_y" value="-0.15"/>
 	<xacro:property name="imu_offset_z" value="0.18"/>
-	<xacro:property name="front_rgbd_camera_offset_x" value="0.35"/>  <!-- 328 --> <!-- 35 leo-->
+	<xacro:property name="front_rgbd_camera_offset_x" value="0.375"/>  <!-- 328 --> <!-- 35 leo-->
 	<xacro:property name="front_rgbd_camera_offset_y" value="0.012"/>
-	<xacro:property name="front_rgbd_camera_offset_z" value="0.230"/>  <!-- 214 -->
+	<xacro:property name="front_rgbd_camera_offset_z" value="0.26"/>  <!-- 214 -->
   <xacro:property name="base_arm_x" value="0.225"/>
   <xacro:property name="base_arm_y" value="0.0"/>

Commit message: replaces rplidar with lds (front lidar is LDS-01)

File: robots/irlab_summit_xls_std.urdf.xacro (robot description, xacro)
@@ -19,5 +19,5 @@
 	<!-- ICCLab sensors -->
 	<xacro:include filename="$(find icclab_summit_xl)/urdf/sensors/scanse.urdf.xacro" />
-	<xacro:include filename="$(find icclab_summit_xl)/urdf/sensors/rplidar.urdf.xacro" />
+	<xacro:include filename="$(find icclab_summit_xl)/urdf/sensors/lds.urdf.xacro" />
 	<xacro:include filename="$(find icclab_summit_xl)/urdf/sensors/intel_d435.urdf.xacro" />
 <!--	<xacro:include filename="$(find icclab_summit_xl)/urdf/sensors/intel_d415.urdf.xacro" /> -->
@@ -89,8 +89,8 @@
 			<origin xyz="${front_rgbd_camera_offset_x} ${front_rgbd_camera_offset_y} ${front_rgbd_camera_offset_z}" rpy="0 0 0"/>
 		</xacro:sensor_orbbec_astra>
-		<!-- RPLidar front lidar -->
-		<xacro:rplidar prefix="$(arg prefix)front_laser" parent="$(arg prefix)base_link" prefix_topic="scan_front">
+		<!-- LDS-01 front lidar -->
+		<xacro:lds prefix="$(arg prefix)front_laser" parent="$(arg prefix)base_link" prefix_topic="scan_front">
 			<origin xyz="${front_laser_offset_x} ${front_laser_offset_y} ${front_laser_offset_z}" rpy="0 0 ${PI/2}"/>
-		</xacro:rplidar>
+		</xacro:lds>
 		<!-- Scanse rear lidar -->
 		<xacro:scanse prefix="$(arg prefix)rear_laser" parent="$(arg prefix)base_link" prefix_topic="scan_rear">

File: urdf/sensors/lds.urdf.xacro (robot description, xacro)
@@ -1,6 +1,6 @@
 <?xml version=  "1.0"?>
-<robot name="rplidar"
+<robot name="lds"
   xmlns:xacro="http://www.ros.org/wiki/xacro">
-  <xacro:macro name="rplidar" params="prefix parent prefix_topic:='front_laser' *origin min_angle:=1.5708 max_angle:=6.2832">
+  <xacro:macro name="lds" params="prefix parent prefix_topic:='front_laser' *origin min_angle:=1.5708 max_angle:=6.2832">
     <joint name="${prefix}_base_joint" type="fixed">
       <!-- FRONT MOUNT  -->
@@ -39,8 +39,8 @@
     </joint>
     <!-- simulation -->
-    <sensor_rplidar_gazebo/>
+    <sensor_lds_gazebo/>
   </xacro:macro>
 <!-- uses ROS Laser Scanner Controller plugin -->
-  <xacro:macro name="sensor_rplidar_gazebo">
+  <xacro:macro name="sensor_lds_gazebo">
     <gazebo reference="${prefix}_link">
       <sensor type="ray" name="${prefix}_sensor">
