Commit message: Updates with robotiq_gripper as parameter for launch file

File: robots/irlab_summit_xls_std.urdf.xacro (robot description, xacro)
@@ -15,6 +15,13 @@
 	<!-- Import all available robotnik sensors -->
 	<xacro:include filename="$(find robotnik_sensors)/urdf/all_sensors.urdf.xacro" />
-	<!-- Import gripper Schunk EGP40-->
-	<xacro:include filename="$(find icclab_summit_xl)/urdf/gripper/schunk_egp40.urdf.xacro" />
+	<xacro:arg name="robotiq_gripper" default="true"/>
+   	<xacro:unless value="$(arg robotiq_gripper)">
+		<!-- Import gripper Schunk EGP40-->
+	   	<xacro:include filename="$(find icclab_summit_xl)/urdf/gripper/schunk_egp40.urdf.xacro" />
+   	</xacro:unless>
+	<xacro:if value="$(arg robotiq_gripper)">
+		<!-- Import gripper Robotiq85-->
+		<xacro:include filename="$(find icclab_summit_xl)/urdf/gripper/ur5_robotiq85_gripper_mod.urdf.xacro" />
+	</xacro:if>
 	<!-- ICCLab sensors -->
 	<xacro:include filename="$(find icclab_summit_xl)/urdf/sensors/scanse.urdf.xacro" />
@@ -106,7 +113,17 @@
 		</joint>
 		<!-- GRIPPER -->
-		<xacro:schunk_egp_40 prefix="gripper_" parent="arm_tool0" >
-			 <origin xyz="0.0 0 0.0" rpy="0 0 0" />
-		</xacro:schunk_egp_40>
+		<xacro:unless value="$(arg robotiq_gripper)">
+			<xacro:schunk_egp_40 prefix="gripper_" parent="arm_tool0" >
+				 <origin xyz="0.0 0 0.0" rpy="0 0 0" />
+			</xacro:schunk_egp_40>
+  		</xacro:unless>
+		<xacro:if value="$(arg robotiq_gripper)">
+    			  <!-- Plugin -->
+			<plugin name="gazebo_ros_control" filename="libgazebo_ros_control.so" >
+				 <robotNamespace>/summit_xl</robotNamespace>
+   				 <robotSimType>gazebo_ros_control/DefaultRobotHWSim</robotSimType>
+   				 <legacyModeNS>true</legacyModeNS>
+			</plugin>
+		</xacro:if>
 		<!-- Camera on gripper  -->
 		<!-- had to copy and modidy camera to avoid name clash with robotnik defined sensors -->

Commit message: Added collision walls

File: robots/irlab_summit_xls_std.urdf.xacro (robot description, xacro)
@@ -15,5 +15,5 @@
 	<!-- Import all available robotnik sensors -->
 	<xacro:include filename="$(find robotnik_sensors)/urdf/all_sensors.urdf.xacro" />
-	<xacro:arg name="robotiq_gripper" default="true"/>
+	<xacro:arg name="robotiq_gripper" default="false"/>
    	<xacro:unless value="$(arg robotiq_gripper)">
 		<!-- Import gripper Schunk EGP40-->
@@ -37,4 +37,6 @@
 	<!-- Collision box on arm wrist 2 -->
 	<xacro:include filename="$(find icclab_summit_xl)/robots/ur5_arm_wrist2_collision_box.urdf.xacro" />
+	<!-- Collision wall robot side -->
+	<xacro:include filename="$(find icclab_summit_xl)/robots/wall_collision_box.urdf.xacro" />
 	<xacro:property name="PI" value="3.1415926535897931"/>
 	<xacro:property name="wheel_offset_x" value="0.2225" />
@@ -154,4 +156,12 @@
 			 <origin xyz="0 0 -0.06" rpy="${PI/2} 0 0" />
 		</xacro:collision_box_wrist2>
+		<!-- Collision box side 1 -->
+		<xacro:collision_box_wall prefix="right" parent="summit_xl_base_footprint">
+			 <origin xyz="0 0.9 0.5" rpy="0 0 0" />
+		</xacro:collision_box_wall>
+		<!-- Collision box side 2 -->
+		<xacro:collision_box_wall prefix="left" parent="summit_xl_base_footprint">
+			 <origin xyz="0 -0.9 0.5" rpy="0 0 0" />
+		</xacro:collision_box_wall>
    </xacro:macro>
    <xacro:ros_control/>

Commit message: Moved collision walls

File: robots/irlab_summit_xls_std.urdf.xacro (robot description, xacro)
@@ -158,9 +158,9 @@
 		<!-- Collision box side 1 -->
 		<xacro:collision_box_wall prefix="right" parent="summit_xl_base_footprint">
-			 <origin xyz="0 0.9 0.5" rpy="0 0 0" />
+			 <origin xyz="0 0.8 0.5" rpy="0 0 0" />
 		</xacro:collision_box_wall>
 		<!-- Collision box side 2 -->
 		<xacro:collision_box_wall prefix="left" parent="summit_xl_base_footprint">
-			 <origin xyz="0 -0.9 0.5" rpy="0 0 0" />
+			 <origin xyz="0 -0.8 0.5" rpy="0 0 0" />
 		</xacro:collision_box_wall>
    </xacro:macro>

Commit message: Added collisions_walls parameter for launch file

File: robots/irlab_summit_xls_std.urdf.xacro (robot description, xacro)
@@ -15,4 +15,5 @@
 	<!-- Import all available robotnik sensors -->
 	<xacro:include filename="$(find robotnik_sensors)/urdf/all_sensors.urdf.xacro" />
+	<xacro:arg name="collision_walls" default="false"/>
 	<xacro:arg name="robotiq_gripper" default="false"/>
    	<xacro:unless value="$(arg robotiq_gripper)">
@@ -156,12 +157,13 @@
 			 <origin xyz="0 0 -0.06" rpy="${PI/2} 0 0" />
 		</xacro:collision_box_wrist2>
-		<!-- Collision box side 1 -->
-		<xacro:collision_box_wall prefix="right" parent="summit_xl_base_footprint">
-			 <origin xyz="0 0.8 0.5" rpy="0 0 0" />
-		</xacro:collision_box_wall>
-		<!-- Collision box side 2 -->
-		<xacro:collision_box_wall prefix="left" parent="summit_xl_base_footprint">
-			 <origin xyz="0 -0.8 0.5" rpy="0 0 0" />
-		</xacro:collision_box_wall>
+		<!-- Collision walls right/left-->
+		<xacro:if value="$(arg collision_walls)">
+			<xacro:collision_box_wall prefix="right" parent="summit_xl_base_footprint">
+				 <origin xyz="0 0.8 0.5" rpy="0 0 0" />
+			</xacro:collision_box_wall>
+			<xacro:collision_box_wall prefix="left" parent="summit_xl_base_footprint">
+				 <origin xyz="0 -0.8 0.5" rpy="0 0 0" />
+			</xacro:collision_box_wall>
+		</xacro:if>
    </xacro:macro>
    <xacro:ros_control/>

Commit message: trying to fix the gripper

File: robots/irlab_summit_xls_std.urdf.xacro (robot description, xacro)
@@ -18,10 +18,12 @@
 	<xacro:arg name="robotiq_gripper" default="false"/>
    	<xacro:unless value="$(arg robotiq_gripper)">
-		<!-- Import gripper Schunk EGP40-->
-	   	<xacro:include filename="$(find icclab_summit_xl)/urdf/gripper/schunk_egp40.urdf.xacro" />
+	<!-- Import gripper Schunk EGP40-->
+	<xacro:include filename="$(find icclab_summit_xl)/urdf/gripper/schunk_egp40.urdf.xacro" />
    	</xacro:unless>
 	<xacro:if value="$(arg robotiq_gripper)">
-		<!-- Import gripper Robotiq85-->
+		<!-- Import gripper Robotiq85 -->
 		<xacro:include filename="$(find icclab_summit_xl)/urdf/gripper/ur5_robotiq85_gripper_mod.urdf.xacro" />
+		<!-- Import gripper Robotiq140 -->
+		<!--xacro:include filename="$(find icclab_summit_xl)/urdf/gripper/robotiq_arg2f_140_model.xacro"/-->
 	</xacro:if>
 	<!-- ICCLab sensors -->

File: urdf/gripper/robotiq_arg2f.xacro (robot description, xacro)
@@ -11,5 +11,5 @@
         <origin xyz="0 0 0" rpy="0 0 0" />
         <geometry>
-          <mesh filename="package://robotiq_2f_140_gripper_visualization/meshes/visual/robotiq_arg2f_base_link.stl" />
+          <mesh filename="package://icclab_summit_xl/meshes/gripper/robotiq/visual/robotiq_arg2f_base_link.stl" />
         </geometry>
         <material name="">
@@ -20,5 +20,5 @@
         <origin xyz="0 0 0" rpy="0 0 0" />
         <geometry>
-          <mesh filename="package://robotiq_2f_140_gripper_visualization/meshes/collision/robotiq_arg2f_base_link.stl" />
+          <mesh filename="package://icclab_summit_xl/meshes/gripper/robotiq/collision/robotiq_arg2f_base_link.stl" />
         </geometry>
       </collision>

File: urdf/gripper/robotiq_arg2f_140_model.xacro (robot description, xacro)
@@ -1,5 +1,5 @@
 <?xml version="1.0"?>
 <robot name="robotiq_arg2f_140_model" xmlns:xacro="http://ros.org/wiki/xacro">
-  <xacro:include filename="$(find robotiq_2f_140_gripper_visualization)/urdf/robotiq_arg2f_140_model_macro.xacro" />
+  <xacro:include filename="$(find icclab_summit_xl)/urdf/gripper/robotiq_arg2f_140_model_macro.xacro" />
   <xacro:robotiq_arg2f_140 prefix=""/>
 </robot>

File: urdf/gripper/robotiq_arg2f_140_model_macro.xacro (robot description, xacro)
@@ -1,5 +1,5 @@
 <?xml version="1.0"?>
 <robot xmlns:xacro="http://ros.org/wiki/xacro">
-  <xacro:include filename="$(find robotiq_2f_140_gripper_visualization)/urdf/robotiq_arg2f_transmission.xacro" />
+  <xacro:include filename="$(find icclab_summit_xl)/urdf/gripper/robotiq_arg2f_transmission.xacro" />
   <xacro:macro name="outer_knuckle" params="prefix fingerprefix stroke">
     <link name="${prefix}${fingerprefix}_outer_knuckle">
@@ -18,5 +18,5 @@
         <origin xyz="0 0 0" rpy="0 0 0" />
         <geometry>
-          <mesh filename="package://robotiq_2f_140_gripper_visualization/meshes/visual/robotiq_arg2f_${stroke}_outer_knuckle.stl" />
+          <mesh filename="package://icclab_summit_xl/meshes/gripper/robotiq/visual/robotiq_arg2f_${stroke}_outer_knuckle.stl" />
         </geometry>
         <material name="">
@@ -27,5 +27,5 @@
         <origin xyz="0 0 0" rpy="0 0 0" />
         <geometry>
-          <mesh filename="package://robotiq_2f_140_gripper_visualization/meshes/collision/robotiq_arg2f_${stroke}_outer_knuckle.stl" />
+          <mesh filename="package://icclab_summit_xl/meshes/gripper/robotiq/collision/robotiq_arg2f_${stroke}_outer_knuckle.stl" />
         </geometry>
       </collision>
@@ -48,5 +48,5 @@
         <origin xyz="0 0 0" rpy="0 0 0" />
         <geometry>
-          <mesh filename="package://robotiq_2f_140_gripper_visualization/meshes/visual/robotiq_arg2f_${stroke}_outer_finger.stl" />
+          <mesh filename="package://icclab_summit_xl/meshes/gripper/robotiq/visual/robotiq_arg2f_${stroke}_outer_finger.stl" />
         </geometry>
         <material name="">
@@ -57,5 +57,5 @@
         <origin xyz="0 0 0" rpy="0 0 0" />
         <geometry>
-          <mesh filename="package://robotiq_2f_140_gripper_visualization/meshes/collision/robotiq_arg2f_${stroke}_outer_finger.stl" />
+          <mesh filename="package://icclab_summit_xl/meshes/gripper/robotiq/collision/robotiq_arg2f_${stroke}_outer_finger.stl" />
         </geometry>
       </collision>
@@ -78,5 +78,5 @@
         <origin xyz="0 0 0" rpy="0 0 0" />
         <geometry>
-          <mesh filename="package://robotiq_2f_140_gripper_visualization/meshes/visual/robotiq_arg2f_${stroke}_inner_knuckle.stl" />
+          <mesh filename="package://icclab_summit_xl/meshes/gripper/robotiq/visual/robotiq_arg2f_${stroke}_inner_knuckle.stl" />
         </geometry>
         <material name="">
@@ -87,5 +87,5 @@
         <origin xyz="0 0 0" rpy="0 0 0" />
         <geometry>
-          <mesh filename="package://robotiq_2f_140_gripper_visualization/meshes/collision/robotiq_arg2f_${stroke}_inner_knuckle.stl" />
+          <mesh filename="package://icclab_summit_xl/meshes/gripper/robotiq/collision/robotiq_arg2f_${stroke}_inner_knuckle.stl" />
         </geometry>
       </collision>
@@ -108,5 +108,5 @@
         <origin xyz="0 0 0" rpy="0 0 0" />
         <geometry>
-          <mesh filename="package://robotiq_2f_140_gripper_visualization/meshes/visual/robotiq_arg2f_${stroke}_inner_finger.stl" />
+          <mesh filename="package://icclab_summit_xl/meshes/gripper/robotiq/visual/robotiq_arg2f_${stroke}_inner_finger.stl" />
         </geometry>
         <material name="">
@@ -117,5 +117,5 @@
         <origin xyz="0 0 0" rpy="0 0 0" />
         <geometry>
-          <mesh filename="package://robotiq_2f_140_gripper_visualization/meshes/collision/robotiq_arg2f_${stroke}_inner_finger.stl" />
+          <mesh filename="package://icclab_summit_xl/meshes/gripper/robotiq/collision/robotiq_arg2f_${stroke}_inner_finger.stl" />
         </geometry>
       </collision>
@@ -181,5 +181,5 @@
     </joint>
   </xacro:macro>
-  <xacro:include filename="$(find robotiq_2f_140_gripper_visualization)/urdf/robotiq_arg2f.xacro" />
+  <xacro:include filename="$(find icclab_summit_xl)/urdf/gripper/robotiq_arg2f.xacro" />
   <xacro:macro name="finger_joint" params="prefix">
     <joint name="${prefix}finger_joint" type="revolute">

Commit message: Added the urdf and meshes for the new gripper

File: robots/irlab_summit_xls_std.urdf.xacro (robot description, xacro)
@@ -23,7 +23,6 @@
 	<xacro:if value="$(arg robotiq_gripper)">
 		<!-- Import gripper Robotiq85 -->
-		<xacro:include filename="$(find icclab_summit_xl)/urdf/gripper/ur5_robotiq85_gripper_mod.urdf.xacro" />
-		<!-- Import gripper Robotiq140 -->
-		<!--xacro:include filename="$(find icclab_summit_xl)/urdf/gripper/robotiq_arg2f_140_model.xacro"/-->
+		<!--xacro:include filename="$(find icclab_summit_xl)/urdf/gripper/ur5_robotiq85_gripper_mod.urdf.xacro"/-->
+		<xacro:include filename="$(find icclab_summit_xl)/urdf/Danfoa_140_2f_robotiq/robotiq_arg2f_140_model_macro.xacro"/>
 	</xacro:if>
 	<!-- ICCLab sensors -->
@@ -68,7 +67,7 @@
 	<xacro:property name="front_rgbd_camera_offset_y" value="0.012"/>
 	<xacro:property name="front_rgbd_camera_offset_z" value="0.26"/>  <!-- 214 -->
-  <xacro:property name="base_arm_x" value="0.225"/>
-  <xacro:property name="base_arm_y" value="0.0"/>
-  <xacro:property name="base_arm_z" value="0.355"/>
+  	<xacro:property name="base_arm_x" value="0.225"/>
+  	<xacro:property name="base_arm_y" value="0.0"/>
+  	<xacro:property name="base_arm_z" value="0.355"/>
 	<!-- Flag to select the high or low quality model -->
 	<xacro:property name="hq" value="true" />
@@ -124,5 +123,11 @@
   		</xacro:unless>
 		<xacro:if value="$(arg robotiq_gripper)">
-    			  <!-- Plugin -->
+			<xacro:robotiq_arg2f_140 prefix="gripper_"/>
+     				<joint name="gripper_base_joint" type="fixed">
+					<origin xyz="0.0 0 0.0" rpy="0 0 0" />
+					<parent link="arm_tool0" />
+					<child link="gripper_robotiq_arg2f_base_link" />
+				</joint>
+    			<!-- Plugin -->
 			<plugin name="gazebo_ros_control" filename="libgazebo_ros_control.so" >
 				 <robotNamespace>/summit_xl</robotNamespace>

Commit message: checked the new gripper on master branch controllers missing

File: robots/irlab_summit_xls_std.urdf.xacro (robot description, xacro)
@@ -22,6 +22,7 @@
    	</xacro:unless>
 	<xacro:if value="$(arg robotiq_gripper)">
-		<!-- Import gripper Robotiq85-->
-		<xacro:include filename="$(find icclab_summit_xl)/urdf/gripper/ur5_robotiq85_gripper_mod.urdf.xacro" />
+		<!-- Import gripper Robotiq85 -->
+		<!--xacro:include filename="$(find icclab_summit_xl)/urdf/gripper/ur5_robotiq85_gripper_mod.urdf.xacro"/-->
+		<xacro:include filename="$(find icclab_summit_xl)/urdf/Danfoa_140_2f_robotiq/robotiq_arg2f_140_model_macro.xacro"/>
 	</xacro:if>
 	<!-- ICCLab sensors -->
@@ -66,7 +67,7 @@
 	<xacro:property name="front_rgbd_camera_offset_y" value="0.012"/>
 	<xacro:property name="front_rgbd_camera_offset_z" value="0.26"/>  <!-- 214 -->
-  <xacro:property name="base_arm_x" value="0.225"/>
-  <xacro:property name="base_arm_y" value="0.0"/>
-  <xacro:property name="base_arm_z" value="0.355"/>
+  	<xacro:property name="base_arm_x" value="0.225"/>
+  	<xacro:property name="base_arm_y" value="0.0"/>
+  	<xacro:property name="base_arm_z" value="0.355"/>
 	<!-- Flag to select the high or low quality model -->
 	<xacro:property name="hq" value="true" />
@@ -122,5 +123,11 @@
   		</xacro:unless>
 		<xacro:if value="$(arg robotiq_gripper)">
-    			  <!-- Plugin -->
+			<xacro:robotiq_arg2f_140 prefix="gripper_"/>
+     				<joint name="gripper_base_joint" type="fixed">
+					<origin xyz="0.0 0 0.0" rpy="0 0 0" />
+					<parent link="arm_tool0" />
+					<child link="gripper_robotiq_arg2f_base_link" />
+				</joint>
+    			<!-- Plugin -->
 			<plugin name="gazebo_ros_control" filename="libgazebo_ros_control.so" >
 				 <robotNamespace>/summit_xl</robotNamespace>

Commit message: change summit lidars to hokuyo

File: robots/irlab_summit_xls_std.urdf.xacro (robot description, xacro)
@@ -27,5 +27,5 @@
 	</xacro:if>
 	<!-- ICCLab sensors -->
-	<xacro:include filename="$(find icclab_summit_xl)/urdf/sensors/scanse.urdf.xacro" />
+	<xacro:include filename="$(find icclab_summit_xl)/urdf/sensors/hokuyo.urdf.xacro" />
 	<xacro:include filename="$(find icclab_summit_xl)/urdf/sensors/lds.urdf.xacro" />
 	<xacro:include filename="$(find icclab_summit_xl)/urdf/sensors/intel_d435.urdf.xacro" />
@@ -46,15 +46,13 @@
 	<xacro:property name="wheel_offset_y" value="0.2045" />
 	<xacro:property name="wheel_offset_z" value="0.0" />
-	<!-- <xacro:property name="front_laser_offset_x" value="0.377"/>    -->
-	<xacro:property name="front_laser_offset_x" value="0.346"/>
-	<!-- <xacro:property name="front_laser_offset_y" value="-0.20957"/>     -->
-	<xacro:property name="front_laser_offset_y" value="-0.235"/>
-	<!-- <xacro:property name="front_laser_offset_z" value="0.2024"/> -->
+	<!--xacro:property name="front_laser_offset_x" value="0.346"/-->
+	<xacro:property name="front_laser_offset_x" value="0.356"/>
+	<!--xacro:property name="front_laser_offset_y" value="-0.235"/-->
+	<xacro:property name="front_laser_offset_y" value="-0.251"/>
 	<xacro:property name="front_laser_offset_z" value="0.1566"/>
-	<!-- <xacro:property name="rear_laser_offset_x" value="-0.377"/> -->
-	<xacro:property name="rear_laser_offset_x" value="-0.34"/>
-	<!-- <xacro:property name="rear_laser_offset_y" value="0.20957"/>     -->
-	<xacro:property name="rear_laser_offset_y" value="0.235"/>
-	<!-- <xacro:property name="rear_laser_offset_z" value="0.2024"/> -->
+	<!--xacro:property name="rear_laser_offset_x" value="-0.34"/-->
+	<xacro:property name="rear_laser_offset_x" value="-0.35"/>
+	<!--xacro:property name="rear_laser_offset_y" value="0.235"/-->
+	<xacro:property name="rear_laser_offset_y" value="0.251"/>
 	<xacro:property name="rear_laser_offset_z" value="0.1566"/>
 	<xacro:property name="front_ptz_camera_offset_x" value="0.308"/>
@@ -100,12 +98,12 @@
 			<origin xyz="${front_rgbd_camera_offset_x} ${front_rgbd_camera_offset_y} ${front_rgbd_camera_offset_z}" rpy="0 0 0"/>
 		</xacro:sensor_orbbec_astra>
-		<!-- LDS-01 front lidar -->
-		<xacro:lds prefix="$(arg prefix)front_laser" parent="$(arg prefix)base_link" prefix_topic="scan_front">
-			<origin xyz="${front_laser_offset_x} ${front_laser_offset_y} ${front_laser_offset_z}" rpy="0 0 ${PI/2}"/>
-		</xacro:lds>
-		<!-- Scanse rear lidar -->
-		<xacro:scanse prefix="$(arg prefix)rear_laser" parent="$(arg prefix)base_link" prefix_topic="scan_rear">
+		<!-- Hokuyo front lidar -->
+		<xacro:hokuyo prefix="$(arg prefix)front_laser" parent="$(arg prefix)base_link" prefix_topic="scan_front">
+			<origin xyz="${front_laser_offset_x} ${front_laser_offset_y} ${front_laser_offset_z}" rpy="0 0 ${3.0*PI/4.0}"/>
+		</xacro:hokuyo>
+		<!-- Hokuyo rear lidar -->
+		<xacro:hokuyo prefix="$(arg prefix)rear_laser" parent="$(arg prefix)base_link" prefix_topic="scan_rear">
 			<origin xyz="${rear_laser_offset_x} ${rear_laser_offset_y} ${rear_laser_offset_z}" rpy="0 0 ${3.0*PI/4.0}"/>
-		</xacro:scanse>
+		</xacro:hokuyo>
 		<!-- UR5 Arm -->
 		<xacro:ur5_robot prefix="arm_" joint_limited="true">

Commit message: configure hokuyo lidars for summit

File: robots/irlab_summit_xls_std.urdf.xacro (robot description, xacro)
@@ -28,5 +28,4 @@
 	<!-- ICCLab sensors -->
 	<xacro:include filename="$(find icclab_summit_xl)/urdf/sensors/hokuyo.urdf.xacro" />
-	<xacro:include filename="$(find icclab_summit_xl)/urdf/sensors/lds.urdf.xacro" />
 	<xacro:include filename="$(find icclab_summit_xl)/urdf/sensors/intel_d435.urdf.xacro" />
 <!--	<xacro:include filename="$(find icclab_summit_xl)/urdf/sensors/intel_d415.urdf.xacro" /> -->
@@ -100,5 +99,5 @@
 		<!-- Hokuyo front lidar -->
 		<xacro:hokuyo prefix="$(arg prefix)front_laser" parent="$(arg prefix)base_link" prefix_topic="scan_front">
-			<origin xyz="${front_laser_offset_x} ${front_laser_offset_y} ${front_laser_offset_z}" rpy="0 0 ${3.0*PI/4.0}"/>
+			<origin xyz="${front_laser_offset_x} ${front_laser_offset_y} ${front_laser_offset_z}" rpy="0 0 ${7.0*PI/4.0}"/>
 		</xacro:hokuyo>
 		<!-- Hokuyo rear lidar -->
