Commit message: added the controllers for the gripper

File: robots/irlab_summit_xls_std.urdf.xacro (robot description, xacro)
@@ -127,4 +127,5 @@
 				</joint>
     			<!-- Plugin -->
+			<gazebo>
 			<plugin name="gazebo_ros_control" filename="libgazebo_ros_control.so" >
 				 <robotNamespace>/summit_xl</robotNamespace>
@@ -132,4 +133,5 @@
    				 <legacyModeNS>true</legacyModeNS>
 			</plugin>
+			</gazebo>
 		</xacro:if>
 		<!-- Camera on gripper  -->

File: urdf/Danfoa_140_2f_robotiq/robotiq_arg2f.gazebo.xacro (robot description, xacro)
@@ -6,5 +6,5 @@
                 <joint>${prefix}finger_joint</joint>
                 <mimicJoint>${prefix}right_outer_knuckle_joint</mimicJoint>
-                <multiplier>-1.0</multiplier>
+                <multiplier>1.0</multiplier>
                 <offset>0.0</offset>
             </plugin>
@@ -12,5 +12,5 @@
                 <joint>${prefix}finger_joint</joint>
                 <mimicJoint>${prefix}left_inner_knuckle_joint</mimicJoint>
-                <multiplier>-1.0</multiplier>
+                <multiplier>1.0</multiplier>
                 <offset>0.0</offset>
             </plugin>
@@ -18,5 +18,5 @@
                 <joint>${prefix}finger_joint</joint>
                 <mimicJoint>${prefix}right_inner_knuckle_joint</mimicJoint>
-                <multiplier>-1.0</multiplier>
+                <multiplier>1.0</multiplier>
                 <offset>0.0</offset>
             </plugin>

File: urdf/Danfoa_140_2f_robotiq/robotiq_arg2f_140_model_macro.xacro (robot description, xacro)
@@ -170,6 +170,7 @@
     <xacro:finger_joint prefix="${prefix}"/>
     <xacro:right_outer_knuckle_joint prefix="${prefix}"/>
-    <xacro:robotiq_arg2f_transmission prefix="${prefix}"/>
-    <xacro:robotiq_arg2f_gazebo prefix="${prefix}"/>
+    <xacro:robotiq_arg2f_transmission0 prefix="${prefix}"/>
+    <xacro:robotiq_arg2f_transmission1 prefix="${prefix}"/>
+        <xacro:robotiq_arg2f_gazebo prefix="${prefix}"/>
 </xacro:macro><mimic joint="${prefix}finger_joint" multiplier="-1" offset="0" />
     </joint>
@@ -221,6 +222,7 @@
     <xacro:finger_joint prefix="${prefix}"/>
     <xacro:right_outer_knuckle_joint prefix="${prefix}"/>
-    <xacro:robotiq_arg2f_transmission prefix="${prefix}"/>
-    <xacro:robotiq_arg2f_gazebo prefix="${prefix}"/>
+    <xacro:robotiq_arg2f_transmission0 prefix="${prefix}"/>
+    <xacro:robotiq_arg2f_transmission1 prefix="${prefix}"/>
+        <xacro:robotiq_arg2f_gazebo prefix="${prefix}"/>
   </xacro:macro>
 </robot>

File: urdf/Danfoa_140_2f_robotiq/robotiq_arg2f_transmission.xacro (robot description, xacro)
@@ -1,9 +1,10 @@
 <?xml version="1.0"?>
 <robot xmlns:xacro="http://ros.org/wiki/xacro">
-  <xacro:macro name="robotiq_arg2f_transmission" params="prefix">
+  <xacro:macro name="robotiq_arg2f_transmission0" params="prefix">
     <transmission name="${prefix}finger_joint_trans">
       <type>transmission_interface/SimpleTransmission</type>
       <joint name="${prefix}finger_joint">
-        <hardwareInterface>PositionJointInterface</hardwareInterface>
+        <!--hardwareInterface>hardware_interface/PositionJointInterface</hardwareInterface-->
+        <hardwareInterface>hardware_interface/EffortJointInterface</hardwareInterface>
       </joint>
       <actuator name="${prefix}finger_joint_motor">
@@ -12,3 +13,15 @@
     </transmission>
   </xacro:macro>
+  <xacro:macro name="robotiq_arg2f_transmission1" params="prefix">
+    <transmission name="${prefix}right_outer_knuckle_joint_trans">
+      <type>transmission_interface/SimpleTransmission</type>
+      <joint name="${prefix}right_outer_knuckle_joint">
+        <!--hardwareInterface>hardware_interface/PositionJointInterface</hardwareInterface-->
+        <hardwareInterface>hardware_interface/EffortJointInterface</hardwareInterface>
+      </joint>
+      <actuator name="${prefix}right_outer_knuckle_joint_motor">
+        <mechanicalReduction>1</mechanicalReduction>
+      </actuator>
+    </transmission>
+  </xacro:macro>
 </robot>

Commit message: repositioned camera and gripper in the URDF

File: robots/irlab_summit_xls_std.urdf.xacro (robot description, xacro)
@@ -122,5 +122,5 @@
 			<xacro:robotiq_arg2f_140 prefix="gripper_"/>
      				<joint name="gripper_base_joint" type="fixed">
-					<origin xyz="0.0 0 0.0" rpy="0 0 0" />
+					<origin xyz="0.0 0 0.0" rpy="0 0 ${PI/2}" />
 					<parent link="arm_tool0" />
 					<child link="gripper_robotiq_arg2f_base_link" />
@@ -137,6 +137,7 @@
 		<sensor_d435_icclab prefix="arm" prefix_topic="arm_camera" parent="arm_wrist_2_link">
      		<!-- <origin xyz="0 0.07 0.145" rpy="0 0 ${PI/2}"/> -->
-			<origin xyz="-0.05 0.071 0.095" rpy="${-PI/2} 0 ${PI/2}"/>  <!-- camera on the one side -->
-			<!--<origin xyz="0.075 0.07 0.1" rpy="${-PI/2} 0 ${PI/2}"/> --><!-- camera on the other oner side -->
+			<!-- origin xyz="-0.05 0.071 0.095" rpy="${-PI/2} 0 ${PI/2}"/ -->  <!-- camera on the one side -->
+			<!--origin xyz="0.075 0.07 0.1" rpy="${-PI/2} 0 ${PI/2}"/--> <!-- camera on the other oner side -->
+			<origin xyz="-0.001 0.07 0.045" rpy="${-PI} 0 ${PI/2}"/> <!-- camera on top -->
    		</sensor_d435_icclab>
 <!--		<sensor_d415_icclab prefix="arm" prefix_topic="arm_camera" parent="arm_wrist_2_link">
@@ -146,6 +147,6 @@
 		<xacro:camera_mount prefix="arm" parent="arm_wrist_2_link">
 			<!-- <origin xyz="-0.005 0.04 0.095" rpy="${PI/2} 0 ${PI}" /> -->
-			 <origin xyz="0 0.041 0.09" rpy=" ${PI/2} ${PI/2} ${PI}" />  <!-- camera on the one side -->
-			<!--<origin xyz="0 0.04 0.1" rpy=" ${PI/2} ${-PI/2} ${PI}" /> --><!-- camera on the other one side -->
+			 <!--origin xyz="0 0.041 0.09" rpy=" ${PI/2} ${PI/2} ${PI}" /-->  <!-- camera on the one side -->
+			<origin xyz="0.005 0.045 0.09" rpy="${PI/2} ${PI} ${PI}" /><!-- camera on top  -->
 		</xacro:camera_mount>
 		<!-- Collision box camera cable -->

Commit message: repositioned camera and gripper in the URDF

File: robots/irlab_summit_xls_std.urdf.xacro (robot description, xacro)
@@ -122,5 +122,5 @@
 			<xacro:robotiq_arg2f_140 prefix="gripper_"/>
      				<joint name="gripper_base_joint" type="fixed">
-					<origin xyz="0.0 0 0.0" rpy="0 0 0" />
+					<origin xyz="0.0 0 0.0" rpy="0 0 ${PI/2}" />
 					<parent link="arm_tool0" />
 					<child link="gripper_robotiq_arg2f_base_link" />
@@ -139,6 +139,7 @@
 		<sensor_d435_icclab prefix="arm" prefix_topic="arm_camera" parent="arm_wrist_2_link">
      		<!-- <origin xyz="0 0.07 0.145" rpy="0 0 ${PI/2}"/> -->
-			<origin xyz="-0.05 0.071 0.095" rpy="${-PI/2} 0 ${PI/2}"/>  <!-- camera on the one side -->
-			<!--<origin xyz="0.075 0.07 0.1" rpy="${-PI/2} 0 ${PI/2}"/> --><!-- camera on the other oner side -->
+			<!-- origin xyz="-0.05 0.071 0.095" rpy="${-PI/2} 0 ${PI/2}"/ -->  <!-- camera on the one side -->
+			<!--origin xyz="0.075 0.07 0.1" rpy="${-PI/2} 0 ${PI/2}"/--> <!-- camera on the other oner side -->
+			<origin xyz="-0.001 0.07 0.045" rpy="${-PI} 0 ${PI/2}"/> <!-- camera on top -->
    		</sensor_d435_icclab>
 <!--		<sensor_d415_icclab prefix="arm" prefix_topic="arm_camera" parent="arm_wrist_2_link">
@@ -148,6 +149,6 @@
 		<xacro:camera_mount prefix="arm" parent="arm_wrist_2_link">
 			<!-- <origin xyz="-0.005 0.04 0.095" rpy="${PI/2} 0 ${PI}" /> -->
-			 <origin xyz="0 0.041 0.09" rpy=" ${PI/2} ${PI/2} ${PI}" />  <!-- camera on the one side -->
-			<!--<origin xyz="0 0.04 0.1" rpy=" ${PI/2} ${-PI/2} ${PI}" /> --><!-- camera on the other one side -->
+			 <!--origin xyz="0 0.041 0.09" rpy=" ${PI/2} ${PI/2} ${PI}" /-->  <!-- camera on the one side -->
+			<origin xyz="0.005 0.045 0.09" rpy="${PI/2} ${PI} ${PI}" /><!-- camera on top  -->
 		</xacro:camera_mount>
 		<!-- Collision box camera cable -->

Commit message: camera postion reconfigured

File: robots/irlab_summit_xls_std.urdf.xacro (robot description, xacro)
@@ -141,5 +141,6 @@
 			<!-- origin xyz="-0.05 0.071 0.095" rpy="${-PI/2} 0 ${PI/2}"/ -->  <!-- camera on the one side -->
 			<!--origin xyz="0.075 0.07 0.1" rpy="${-PI/2} 0 ${PI/2}"/--> <!-- camera on the other oner side -->
-			<origin xyz="-0.001 0.07 0.045" rpy="${-PI} 0 ${PI/2}"/> <!-- camera on top -->
+			<!--origin xyz="-0.001 0.07 0.045" rpy="${-PI} 0 ${PI/2}"/--> <!-- camera on top -->
+			<origin xyz="-0.001 0.07 0.175" rpy="${-PI} 0 ${PI/2}"/> <!-- camera on bot -->
    		</sensor_d435_icclab>
 <!--		<sensor_d415_icclab prefix="arm" prefix_topic="arm_camera" parent="arm_wrist_2_link">
@@ -150,5 +151,6 @@
 			<!-- <origin xyz="-0.005 0.04 0.095" rpy="${PI/2} 0 ${PI}" /> -->
 			 <!--origin xyz="0 0.041 0.09" rpy=" ${PI/2} ${PI/2} ${PI}" /-->  <!-- camera on the one side -->
-			<origin xyz="0.005 0.045 0.09" rpy="${PI/2} ${PI} ${PI}" /><!-- camera on top  -->
+			<!--origin xyz="0.005 0.045 0.09" rpy="${PI/2} ${PI} ${PI}" /--><!-- camera on top  -->
+			<origin xyz="-0.0036 0.045 0.1" rpy="${PI/2} 0 ${PI}" /><!-- camera on bot  -->
 		</xacro:camera_mount>
 		<!-- Collision box camera cable -->

Commit message: Fixed proper xacro macro invocations in robot and arm camera

File: robots/irlab_summit_xls_std.urdf.xacro (robot description, xacro)
@@ -137,5 +137,5 @@
 		<!-- Camera on gripper  -->
 		<!-- had to copy and modidy camera to avoid name clash with robotnik defined sensors -->
-		<sensor_d435_icclab prefix="arm" prefix_topic="arm_camera" parent="arm_wrist_2_link">
+		<xacro:sensor_d435_icclab prefix="arm" prefix_topic="arm_camera" parent="arm_wrist_2_link">
      		<!-- <origin xyz="0 0.07 0.145" rpy="0 0 ${PI/2}"/> -->
 			<!-- origin xyz="-0.05 0.071 0.095" rpy="${-PI/2} 0 ${PI/2}"/ -->  <!-- camera on the one side -->
@@ -143,5 +143,5 @@
 			<!--origin xyz="-0.001 0.07 0.045" rpy="${-PI} 0 ${PI/2}"/--> <!-- camera on top -->
 			<origin xyz="-0.001 0.07 0.175" rpy="${-PI} 0 ${PI/2}"/> <!-- camera on bot -->
-   		</sensor_d435_icclab>
+   		</xacro:sensor_d435_icclab>
 <!--		<sensor_d415_icclab prefix="arm" prefix_topic="arm_camera" parent="arm_wrist_2_link">
      		<origin xyz="0 0.05 0.155" rpy="0 0 ${PI/2}"/>--> <!-- Note the position seems to be wrong in gazebo beacuase we use the d435 mesh file, but it is correct considering the realsize of the camera-->
@@ -154,8 +154,8 @@
 			<origin xyz="-0.0036 0.045 0.1" rpy="${PI/2} 0 ${PI}" /><!-- camera on bot  -->
 		</xacro:camera_mount>
-		<!-- Collision box camera cable -->
+		<!-- Collision box camera cable
 		<xacro:collision_box_camera_cable prefix="arm" parent="arm_camera_link">
 			 <origin xyz="-0.02 -0.08 0" rpy="0 0 0" />
-		</xacro:collision_box_camera_cable>
+		</xacro:collision_box_camera_cable> -->
 		<!-- Collision box wrist 3 -->
 		<xacro:collision_box_wrist3 prefix="arm" parent="arm_wrist_3_link">

File: urdf/sensors/intel_d435.urdf.xacro (robot description, xacro)
@@ -48,5 +48,5 @@
         <geometry>
           <!-- <box size="${d435_cam_width} ${d435_cam_height} ${d435_cam_depth}"/> -->
-	  <mesh filename="package://robotnik_sensors/meshes/intel_realsense_depth_camera_d435.dae" />
+	  <mesh filename="package://robotnik_sensors/meshes/intel_d435.dae" />
           <!--<mesh filename="package://realsense2_camera/meshes/d435/d435.dae" />-->
         </geometry>
@@ -119,5 +119,5 @@
     <link name="${prefix}_camera_color_optical_frame"/>
   <!-- RGBD sensor for simulation, same as Kinect -->
-  <sensor_d435_icclab_gazebo/>
+  <xacro:sensor_d435_icclab_gazebo/>
   </xacro:macro>
    <xacro:macro name="sensor_d435_icclab_gazebo">

Commit message: Added wheel size to robot.urdf because new version of summit_xl_common for melodic had it not set

File: robots/irlab_summit_xls_std.urdf.xacro (robot description, xacro)
@@ -6,4 +6,5 @@
 	<!-- First we import all posible elements defined in the urdf.xacro files. All these elements are defined as macro:xacros -->
 	<!-- Import summit XL base elements -->
+	<xacro:property name="wheel_radius" value="0.1025" />
 	<xacro:include filename="$(find summit_xl_description)/urdf/bases/summit_xl_hls_base.urdf.xacro" />
 	<!-- Import summit XL wheels -->

Commit message: Updated arm to use UR descriptions from apt

File: robots/irlab_summit_xls_std.urdf.xacro (robot description, xacro)
@@ -13,5 +13,5 @@
 	<xacro:include filename="$(find summit_xl_description)/urdf/structures/structure_hokuyo.urdf.xacro" />
 	<!-- Import arm description -->
-	<xacro:include filename="$(find ur_description)/urdf/ur5.urdf.xacro" />
+	<xacro:include filename="$(find ur_description)/urdf/inc/ur5_macro.xacro" />
 	<!-- Import all available robotnik sensors -->
 	<xacro:include filename="$(find robotnik_sensors)/urdf/all_sensors.urdf.xacro" />
@@ -107,6 +107,5 @@
 		</xacro:hokuyo>
 		<!-- UR5 Arm -->
-		<xacro:ur5_robot prefix="arm_" joint_limited="true">
-		</xacro:ur5_robot>
+		<xacro:ur5_robot prefix="arm_"/>
 		<joint name="$(arg prefix)arm_base_joint" type="fixed">
 			<origin xyz="0.255 0 0.275" rpy="0 0 ${PI}" />
@@ -130,10 +129,10 @@
 		<!-- Camera on gripper  -->
 		<!-- had to copy and modidy camera to avoid name clash with robotnik defined sensors -->
-		<xacro:sensor_d435_icclab prefix="arm" prefix_topic="arm_camera" parent="arm_wrist_2_link">
+		<xacro:sensor_d435_icclab prefix="arm" prefix_topic="arm_camera" parent="gripper_robotiq_arg2f_base_link">
      		<!-- <origin xyz="0 0.07 0.145" rpy="0 0 ${PI/2}"/> -->
 			<!-- origin xyz="-0.05 0.071 0.095" rpy="${-PI/2} 0 ${PI/2}"/ -->  <!-- camera on the one side -->
 			<!--origin xyz="0.075 0.07 0.1" rpy="${-PI/2} 0 ${PI/2}"/--> <!-- camera on the other oner side -->
 			<!--origin xyz="-0.001 0.07 0.045" rpy="${-PI} 0 ${PI/2}"/--> <!-- camera on top -->
-			<origin xyz="-0.001 0.07 0.175" rpy="${-PI} 0 ${PI/2}"/> <!-- camera on bot -->
+			<origin xyz="0.07 0.0 0.03" rpy="0 ${-PI/2} 0"/> <!-- camera on bot -->
    		</xacro:sensor_d435_icclab>
 <!--		<sensor_d415_icclab prefix="arm" prefix_topic="arm_camera" parent="arm_wrist_2_link">
@@ -141,9 +140,9 @@
    		<!--</sensor_d415_icclab>-->
 		<!-- Camera mount -->
-		<xacro:camera_mount prefix="arm" parent="arm_wrist_2_link">
+		<xacro:camera_mount prefix="arm" parent="gripper_robotiq_arg2f_base_link">
 			<!-- <origin xyz="-0.005 0.04 0.095" rpy="${PI/2} 0 ${PI}" /> -->
 			 <!--origin xyz="0 0.041 0.09" rpy=" ${PI/2} ${PI/2} ${PI}" /-->  <!-- camera on the one side -->
 			<!--origin xyz="0.005 0.045 0.09" rpy="${PI/2} ${PI} ${PI}" /--><!-- camera on top  -->
-			<origin xyz="-0.0036 0.045 0.1" rpy="${PI/2} 0 ${PI}" /><!-- camera on bot  -->
+			<origin xyz="0 0 0" rpy="0 0 ${-PI/2}" /><!-- camera on bot  -->
 		</xacro:camera_mount>
 		<!-- Collision box camera cable -->
