Commit message: reuse realsense camera from grasping package

File: robots/irlab_summit_xls_std.urdf.xacro (robot description, xacro)
@@ -129,10 +129,6 @@
 		<!-- Camera on gripper  -->
 		<!-- had to copy and modidy camera to avoid name clash with robotnik defined sensors -->
-		<xacro:sensor_d435_icclab prefix="arm" prefix_topic="arm_camera" parent="gripper_robotiq_arg2f_base_link">
-     		<!-- <origin xyz="0 0.07 0.145" rpy="0 0 ${PI/2}"/> -->
-			<!-- origin xyz="-0.05 0.071 0.095" rpy="${-PI/2} 0 ${PI/2}"/ -->  <!-- camera on the one side -->
-			<!--origin xyz="0.075 0.07 0.1" rpy="${-PI/2} 0 ${PI/2}"/--> <!-- camera on the other oner side -->
-			<!--origin xyz="-0.001 0.07 0.045" rpy="${-PI} 0 ${PI/2}"/--> <!-- camera on top -->
-			<origin xyz="0.07 0.0 0.03" rpy="0 ${-PI/2} 0"/> <!-- camera on bot -->
+		<xacro:sensor_d435_icclab prefix="arm" prefix_topic="summit_xl/arm_camera" parent="gripper_robotiq_arg2f_base_link">
+     		  <origin xyz="0.06 0.0 0.01" rpy="${PI} ${-PI/2} 0"/> <!-- camera on gripper -->
    		</xacro:sensor_d435_icclab>
 <!--		<sensor_d415_icclab prefix="arm" prefix_topic="arm_camera" parent="arm_wrist_2_link">

File: urdf/sensors/intel_d435.urdf.xacro (robot description, xacro)
@@ -1,163 +1,17 @@
 <?xml version="1.0"?>
-<!--
-License: Apache 2.0. See LICENSE file in root directory.
-Copyright(c) 2017 Intel Corporation. All Rights Reserved
-This is the URDF model for the Intel RealSense 430 camera, in it's
-aluminum peripherial evaluation case.
--->
-<!-- <robot name="sensor_d435" xmlns:xacro="http://ros.org/wiki/xacro"> -->
-<robot name="sensor_d435_icclab" xmlns:xacro="http://ros.org/wiki/xacro">
-  <xacro:macro name="sensor_d435_icclab"  params="prefix parent prefix_topic:='front_rgbd_camera' *origin">
-    <xacro:property name="M_PI" value="3.1415926535897931" />
-    <!-- The following values are approximate, and the camera node
-     publishing TF values with actual calibrated camera extrinsic values -->
-    <xacro:property name="d435_cam_depth_to_left_ir_offset" value="0.0"/>
-    <xacro:property name="d435_cam_depth_to_right_ir_offset" value="-0.050"/>
-    <xacro:property name="d435_cam_depth_to_color_offset" value="0.015"/>
-    <!-- The following values model the aluminum peripherial case for the
-  	D435 camera, with the camera joint represented by the actual
-  	peripherial camera tripod mount -->
-    <xacro:property name="d435_cam_width" value="0.090"/>
-    <xacro:property name="d435_cam_height" value="0.025"/>
-    <xacro:property name="d435_cam_depth" value="0.02505"/>
-    <xacro:property name="d435_cam_mount_from_center_offset" value="0.0149"/>
-    <!-- The following offset is relative the the physical D435 camera peripherial
-  	camera tripod mount -->
-    <xacro:property name="d435_cam_depth_px" value="${d435_cam_mount_from_center_offset}"/>
-    <xacro:property name="d435_cam_depth_py" value="0.0175"/>
-    <xacro:property name="d435_cam_depth_pz" value="${d435_cam_height/2}"/>
-<!--  <material name="aluminum">-->
-<!--    <color rgba="0.5 0.5 0.5 1"/>-->
-<!--  </material>-->
-    <!-- camera body, with origin at bottom screw mount -->
-    <joint name="${prefix}_camera_joint" type="fixed">
-      <xacro:insert_block name="origin" />
-      <parent link="${parent}"/>
-      <child link="${prefix}_camera_bottom_screw_frame" />
-    </joint>
-    <link name="${prefix}_camera_bottom_screw_frame"/>
-    <joint name="${prefix}_camera_link_joint" type="fixed">
-      <origin xyz="0 ${d435_cam_depth_py} ${d435_cam_depth_pz}" rpy="0 0 0"/>
-      <parent link="${prefix}_camera_bottom_screw_frame"/>
-      <child link="${prefix}_camera_link" />
-    </joint>
-    <link name="${prefix}_camera_link">
-      <visual>
-      <!-- <origin xyz="${d435_cam_mount_from_center_offset} ${-d435_cam_depth_py} 0" rpy="${M_PI/2} 0 ${M_PI/2}"/> -->
-      <origin xyz="0 ${-d435_cam_mount_from_center_offset} 0" rpy="0 0 0"/>
-        <geometry>
-          <!-- <box size="${d435_cam_width} ${d435_cam_height} ${d435_cam_depth}"/> -->
-	  <mesh filename="package://robotnik_sensors/meshes/intel_d435.dae" />
-          <!--<mesh filename="package://realsense2_camera/meshes/d435/d435.dae" />-->
-        </geometry>
-        <material name="aluminum"/>
-      </visual>
-      <collision>
-        <origin xyz="0 ${-d435_cam_depth_py} 0" rpy="0 0 0"/>
-        <geometry>
-        <box size="${d435_cam_depth} ${d435_cam_width} ${d435_cam_height}"/>
-        </geometry>
-      </collision>
-      <inertial>
-        <!-- The following are not reliable values, and should not be used for modeling -->
-        <mass value="0.564" />
-        <origin xyz="0 0 0" />
-        <inertia ixx="0.003881243" ixy="0.0" ixz="0.0" iyy="0.000498940" iyz="0.0" izz="0.003879257" />
-      </inertial>
-    </link>
-    <!-- camera depth joints and links -->
-    <joint name="${prefix}_camera_depth_joint" type="fixed">
-      <origin xyz="0 0 0" rpy="0 0 0"/>
-      <parent link="${prefix}_camera_link"/>
-      <child link="${prefix}_camera_depth_frame" />
-    </joint>
-    <link name="${prefix}_camera_depth_frame"/>
-    <joint name="${prefix}_camera_depth_optical_joint" type="fixed">
-      <origin xyz="0 0 0" rpy="${-M_PI/2} 0 ${-M_PI/2}" />
-      <parent link="${prefix}_camera_depth_frame" />
-      <child link="${prefix}_camera_depth_optical_frame" />
-    </joint>
-    <link name="${prefix}_camera_depth_optical_frame"/>
-    <!-- camera left IR joints and links -->
-    <joint name="${prefix}_camera_left_ir_joint" type="fixed">
-      <origin xyz="0 ${d435_cam_depth_to_left_ir_offset} 0" rpy="0 0 0" />
-      <parent link="${prefix}_camera_depth_frame" />
-      <child link="${prefix}_camera_left_ir_frame" />
-    </joint>
-    <link name="${prefix}_camera_left_ir_frame"/>
-    <joint name="${prefix}_camera_left_ir_optical_joint" type="fixed">
-      <origin xyz="0 0 0" rpy="${-M_PI/2} 0 ${-M_PI/2}" />
-      <parent link="${prefix}_camera_left_ir_frame" />
-      <child link="${prefix}_camera_left_ir_optical_frame" />
-    </joint>
-    <link name="${prefix}_camera_left_ir_optical_frame"/>
-    <!-- camera right IR joints and links -->
-    <joint name="${prefix}_camera_right_ir_joint" type="fixed">
-      <origin xyz="0 ${d435_cam_depth_to_right_ir_offset} 0" rpy="0 0 0" />
-      <parent link="${prefix}_camera_depth_frame" />
-      <child link="${prefix}_camera_right_ir_frame" />
-    </joint>
-    <link name="${prefix}_camera_right_ir_frame"/>
-    <joint name="${prefix}_camera_right_ir_optical_joint" type="fixed">
-      <origin xyz="0 0 0" rpy="${-M_PI/2} 0 ${-M_PI/2}" />
-      <parent link="${prefix}_camera_right_ir_frame" />
-      <child link="${prefix}_camera_right_ir_optical_frame" />
-    </joint>
-    <link name="${prefix}_camera_right_ir_optical_frame"/>
-    <!-- camera color joints and links -->
-    <joint name="${prefix}_camera_color_joint" type="fixed">
-      <origin xyz="0 ${d435_cam_depth_to_color_offset} 0" rpy="0 0 0" />
-      <parent link="${prefix}_camera_depth_frame" />
-      <child link="${prefix}_camera_color_frame" />
-    </joint>
-    <link name="${prefix}_camera_color_frame"/>
-    <joint name="${prefix}_camera_color_optical_joint" type="fixed">
-      <origin xyz="0 0 0" rpy="${-M_PI/2} 0 ${-M_PI/2}" />
-      <parent link="${prefix}_camera_color_frame" />
-      <child link="${prefix}_camera_color_optical_frame" />
-    </joint>
-    <link name="${prefix}_camera_color_optical_frame"/>
-  <!-- RGBD sensor for simulation, same as Kinect -->
-  <xacro:sensor_d435_icclab_gazebo/>
-  </xacro:macro>
-   <xacro:macro name="sensor_d435_icclab_gazebo">
-    <!-- gazebo reference="${prefix}_rgb_base_link" -->
-    <gazebo reference="${prefix}_camera_link">
-      <sensor type="depth" name="${prefix}_depth_sensor">
-        <always_on>true</always_on>
-        <update_rate>5.0</update_rate>
-        <camera>
-          <horizontal_fov>${91.2*M_PI/180.0}</horizontal_fov>
-          <image>
-            <format>R8G8B8</format>
-            <width>640</width>
-            <height>480</height>
-          </image>
-          <clip>
-            <near>0.3</near>
-            <far>10.0</far>
-          </clip>
-        </camera>
-        <plugin name="${prefix}_controller" filename="libgazebo_ros_openni_kinect.so">
-          <cameraName>${prefix_topic}</cameraName>
-          <alwaysOn>true</alwaysOn>
-          <updateRate>5</updateRate>
-          <imageTopicName>rgb/image_raw</imageTopicName>
-          <depthImageTopicName>depth/image_raw</depthImageTopicName>
-          <!-- changed topic to be consistent with what we have on phys robot -->
-          <pointCloudTopicName>depth_registered/points</pointCloudTopicName>
-          <cameraInfoTopicName>rgb/camera_info</cameraInfoTopicName>
-          <depthImageCameraInfoTopicName>depth/camera_info</depthImageCameraInfoTopicName>
-          <frameName>/${prefix}_camera_depth_optical_frame</frameName>
-          <baseline>0.1</baseline>
-          <distortion_k1>0.0</distortion_k1>
-          <distortion_k2>0.0</distortion_k2>
-          <distortion_k3>0.0</distortion_k3>
-          <distortion_t1>0.0</distortion_t1>
-          <distortion_t2>0.0</distortion_t2>
-          <pointCloudCutoff>0.4</pointCloudCutoff>
-        </plugin>
-      </sensor>
-    </gazebo>
-  </xacro:macro>
+<robot xmlns:xacro="http://www.ros.org/wiki/xacro" name="realsense">
+<xacro:include filename="$(find realsense2_description)/urdf/_d435.urdf.xacro" />
+<xacro:include filename="$(find icclab_grasping_niryo)/urdf/_d435.gazebo.kinect.xacro"/>
+<xacro:macro name="sensor_d435_icclab" params="parent *origin prefix:=arm prefix_topic:=arm_camera use_nominal_extrinsics:=true add_plug:=false use_mesh:=true">
+	<xacro:sensor_d435 parent="${parent}" name="${prefix}_camera" use_nominal_extrinsics="${use_nominal_extrinsics}" add_plug="${add_plug}" use_mesh="${use_mesh}">
+	  <xacro:insert_block name="origin" />
+	</xacro:sensor_d435>
+	<xacro:gazebo_d435 camera_name="${prefix}_camera"/>
+	<!-- Realsense Gazebo Plugin -->
+	<!--
+	<xacro:include filename="$(find icclab_grasping_niryo)/urdf/_d435.gazebo.xacro"/>
+	<xacro:gazebo_d435 camera_name="${prefix}_camera_" reference_link="${prefix}_camera_link" topics_ns="${prefix_topic}"
+	depth_optical_frame="${prefix}_camera_depth_optical_frame" color_optical_frame="${prefix}_camera_color_optical_frame"
+infrared1_optical_frame="${prefix}_camera_left_ir_optical_frame" infrared2_optical_frame="${prefix}_camera_right_ir_optical_frame"/>-->
+</xacro:macro>
 </robot>
