Commit message: Updated the d435 camera model

File: urdf/sensors/old_intel_d435.urdf.xacro (robot description, xacro)
@@ -1,60 +1,46 @@
 <?xml version="1.0"?>
-<!--
-License: Apache 2.0. See LICENSE file in root directory.
-Copyright(c) 2017 Intel Corporation. All Rights Reserved
-This is the URDF model for the Intel RealSense 430 camera, in it's
-aluminum peripherial evaluation case.
--->
-<!-- <robot name="sensor_d435" xmlns:xacro="http://ros.org/wiki/xacro"> -->
-<robot name="sensor_d435_icclab" xmlns:xacro="http://ros.org/wiki/xacro">
-  <xacro:macro name="sensor_d435_icclab"  params="prefix parent prefix_topic:='front_rgbd_camera' *origin">
-    <xacro:property name="M_PI" value="3.1415926535897931" />
-    <!-- The following values are approximate, and the camera node
-     publishing TF values with actual calibrated camera extrinsic values -->
-    <xacro:property name="d435_cam_depth_to_left_ir_offset" value="0.0"/>
-    <xacro:property name="d435_cam_depth_to_right_ir_offset" value="-0.050"/>
-    <xacro:property name="d435_cam_depth_to_color_offset" value="0.015"/>
-    <!-- The following values model the aluminum peripherial case for the
-  	D435 camera, with the camera joint represented by the actual
-  	peripherial camera tripod mount -->
-    <xacro:property name="d435_cam_width" value="0.090"/>
-    <xacro:property name="d435_cam_height" value="0.025"/>
-    <xacro:property name="d435_cam_depth" value="0.02505"/>
-    <xacro:property name="d435_cam_mount_from_center_offset" value="0.0149"/>
-    <!-- The following offset is relative the the physical D435 camera peripherial
-  	camera tripod mount -->
-    <xacro:property name="d435_cam_depth_px" value="${d435_cam_mount_from_center_offset}"/>
-    <xacro:property name="d435_cam_depth_py" value="0.0175"/>
-    <xacro:property name="d435_cam_depth_pz" value="${d435_cam_height/2}"/>
+<robot name="sensor_r430_icclab" xmlns:xacro="http://www.ros.org/wiki/xacro">
+  <xacro:property name="M_PI" value="3.1415926535897931" />
+  <!-- The following values are approximate, and the camera node
+   publishing TF values with actual calibrated camera extrinsic values -->
+  <xacro:property name="r430_cam_depth_to_left_ir_offset" value="-0.021"/>
+  <xacro:property name="r430_cam_depth_to_right_ir_offset" value="0.029"/>
+  <xacro:property name="r430_cam_depth_to_fisheye_offset" value="0.044"/>
+  <!-- The following values model the aluminum peripherial case for the
+    R430 camera, with the camera joint represented by the actual
+    peripherial camera tripod mount -->
+  <xacro:property name="r430_cam_width" value="0.100"/>
+  <xacro:property name="r430_cam_depth" value="0.025"/>
+  <xacro:property name="r430_cam_height" value="0.025"/>
+  <xacro:property name="r430_cam_mount_from_center_offset" value="0.0"/>
+  <!-- The following offset is relative the the physical R430 camera peripherial
+    camera tripod mount -->
+  <xacro:property name="r430_cam_depth_px" value="0.00"/>
+  <xacro:property name="r430_cam_depth_py" value="-0.0115"/>
+  <xacro:property name="r430_cam_depth_pz" value="0.0"/>
 <!--  <material name="aluminum">-->
 <!--    <color rgba="0.5 0.5 0.5 1"/>-->
 <!--  </material>-->
+  <xacro:macro name="sensor_r430_icclab" params="prefix parent prefix_topic:='front_rgbd_camera' *origin">
     <!-- camera body, with origin at bottom screw mount -->
     <joint name="${prefix}_camera_joint" type="fixed">
       <xacro:insert_block name="origin" />
       <parent link="${parent}"/>
-      <child link="${prefix}_camera_bottom_screw_frame" />
-    </joint>
-    <link name="${prefix}_camera_bottom_screw_frame"/>
-    <joint name="${prefix}_camera_link_joint" type="fixed">
-      <origin xyz="0 ${d435_cam_depth_py} ${d435_cam_depth_pz}" rpy="0 0 0"/>
-      <parent link="${prefix}_camera_bottom_screw_frame"/>
       <child link="${prefix}_camera_link" />
     </joint>
     <link name="${prefix}_camera_link">
       <visual>
-      <!-- <origin xyz="${d435_cam_mount_from_center_offset} ${-d435_cam_depth_py} 0" rpy="${M_PI/2} 0 ${M_PI/2}"/> -->
-      <origin xyz="0 ${-d435_cam_mount_from_center_offset} 0" rpy="0 0 0"/>
+      <!-- origin xyz="0 ${-r430_cam_mount_from_center_offset} ${r430_cam_height/2}" rpy="${M_PI/2} 0 ${M_PI/2}"/ -->
+      <origin xyz="0 ${-r430_cam_mount_from_center_offset} 0" rpy="0 0 0"/>
         <geometry>
-          <!-- <box size="${d435_cam_width} ${d435_cam_height} ${d435_cam_depth}"/> -->
-	  <mesh filename="package://robotnik_sensors/meshes/intel_realsense_depth_camera_d435.dae" />
-          <!--<mesh filename="package://realsense2_camera/meshes/d435/d435.dae" />-->
+          <!-- box size="${r430_cam_width} ${r430_cam_height} ${r430_cam_depth}"/ -->
+          <mesh filename="package://robotnik_sensors/meshes/intel_realsense_depth_camera_d435.dae" />
         </geometry>
         <material name="aluminum"/>
       </visual>
       <collision>
-        <origin xyz="0 ${-d435_cam_depth_py} 0" rpy="0 0 0"/>
+        <origin xyz="${-r430_cam_depth/2} 0.0 0.0" rpy="0 0 0"/>
         <geometry>
-        <box size="${d435_cam_depth} ${d435_cam_width} ${d435_cam_height}"/>
+        <box size="${r430_cam_depth} ${r430_cam_width} ${r430_cam_height}"/>
         </geometry>
       </collision>
@@ -68,5 +54,5 @@
     <!-- camera depth joints and links -->
     <joint name="${prefix}_camera_depth_joint" type="fixed">
-      <origin xyz="0 0 0" rpy="0 0 0"/>
+      <origin xyz="${r430_cam_depth_px} ${r430_cam_depth_py} ${r430_cam_depth_pz}" rpy="0 0 0"/>
       <parent link="${prefix}_camera_link"/>
       <child link="${prefix}_camera_depth_frame" />
@@ -81,5 +67,5 @@
     <!-- camera left IR joints and links -->
     <joint name="${prefix}_camera_left_ir_joint" type="fixed">
-      <origin xyz="0 ${d435_cam_depth_to_left_ir_offset} 0" rpy="0 0 0" />
+      <origin xyz="0 ${r430_cam_depth_to_left_ir_offset} 0" rpy="0 0 0" />
       <parent link="${prefix}_camera_depth_frame" />
       <child link="${prefix}_camera_left_ir_frame" />
@@ -94,5 +80,5 @@
     <!-- camera right IR joints and links -->
     <joint name="${prefix}_camera_right_ir_joint" type="fixed">
-      <origin xyz="0 ${d435_cam_depth_to_right_ir_offset} 0" rpy="0 0 0" />
+      <origin xyz="0 ${r430_cam_depth_to_right_ir_offset} 0" rpy="0 0 0" />
       <parent link="${prefix}_camera_depth_frame" />
       <child link="${prefix}_camera_right_ir_frame" />
@@ -105,21 +91,21 @@
     </joint>
     <link name="${prefix}_camera_right_ir_optical_frame"/>
-    <!-- camera color joints and links -->
-    <joint name="${prefix}_camera_color_joint" type="fixed">
-      <origin xyz="0 ${d435_cam_depth_to_color_offset} 0" rpy="0 0 0" />
+    <!-- camera fisheye joints and links -->
+    <joint name="${prefix}_camera_fisheye_joint" type="fixed">
+      <origin xyz="0 ${r430_cam_depth_to_fisheye_offset} 0" rpy="0 0 0" />
       <parent link="${prefix}_camera_depth_frame" />
-      <child link="${prefix}_camera_color_frame" />
+      <child link="${prefix}_camera_fisheye_frame" />
     </joint>
-    <link name="${prefix}_camera_color_frame"/>
-    <joint name="${prefix}_camera_color_optical_joint" type="fixed">
+    <link name="${prefix}_camera_fisheye_frame"/>
+    <joint name="${prefix}_camera_fisheye_optical_joint" type="fixed">
       <origin xyz="0 0 0" rpy="${-M_PI/2} 0 ${-M_PI/2}" />
-      <parent link="${prefix}_camera_color_frame" />
-      <child link="${prefix}_camera_color_optical_frame" />
+      <parent link="${prefix}_camera_fisheye_frame" />
+      <child link="${prefix}_camera_fisheye_optical_frame" />
     </joint>
-    <link name="${prefix}_camera_color_optical_frame"/>
+    <link name="${prefix}_camera_fisheye_optical_frame"/>
   <!-- RGBD sensor for simulation, same as Kinect -->
-  <sensor_d435_icclab_gazebo/>
+  <sensor_r430_icclab_gazebo/>
   </xacro:macro>
-   <xacro:macro name="sensor_d435_icclab_gazebo">
+   <xacro:macro name="sensor_r430_icclab_gazebo">
     <!-- gazebo reference="${prefix}_rgb_base_link" -->
     <gazebo reference="${prefix}_camera_link">
