Commit message: Updated camera models for d415 d435

File: urdf/sensors/intel_d415.urdf.xacro (robot description, xacro)
@@ -3,28 +3,28 @@
 License: Apache 2.0. See LICENSE file in root directory.
 Copyright(c) 2017 Intel Corporation. All Rights Reserved
-This is the URDF model for the Intel RealSense 430 camera, in it's
+This is the URDF model for the Intel RealSense 415 camera, in it's
 aluminum peripherial evaluation case.
 -->
-<!-- <robot name="sensor_d435" xmlns:xacro="http://ros.org/wiki/xacro"> -->
-<robot name="sensor_d435_icclab" xmlns:xacro="http://ros.org/wiki/xacro">
-  <xacro:macro name="sensor_d435_icclab"  params="prefix parent prefix_topic:='front_rgbd_camera' *origin">
+<!-- <robot name="sensor_d415" xmlns:xacro="http://ros.org/wiki/xacro"> -->
+<robot name="sensor_d415_icclab" xmlns:xacro="http://ros.org/wiki/xacro">
+  <xacro:macro name="sensor_d415_icclab" params="prefix parent prefix_topic:='front_rgbd_camera' *origin">
     <xacro:property name="M_PI" value="3.1415926535897931" />
     <!-- The following values are approximate, and the camera node
      publishing TF values with actual calibrated camera extrinsic values -->
-    <xacro:property name="d435_cam_depth_to_left_ir_offset" value="0.0"/>
-    <xacro:property name="d435_cam_depth_to_right_ir_offset" value="-0.050"/>
-    <xacro:property name="d435_cam_depth_to_color_offset" value="0.015"/>
+    <xacro:property name="d415_cam_depth_to_left_ir_offset" value="0.0"/>
+    <xacro:property name="d415_cam_depth_to_right_ir_offset" value="-0.055"/>
+    <xacro:property name="d415_cam_depth_to_color_offset" value="0.015"/>
     <!-- The following values model the aluminum peripherial case for the
-  	D435 camera, with the camera joint represented by the actual
+  	d415 camera, with the camera joint represented by the actual
   	peripherial camera tripod mount -->
-    <xacro:property name="d435_cam_width" value="0.090"/>
-    <xacro:property name="d435_cam_height" value="0.025"/>
-    <xacro:property name="d435_cam_depth" value="0.02505"/>
-    <xacro:property name="d435_cam_mount_from_center_offset" value="0.0149"/>
-    <!-- The following offset is relative the the physical D435 camera peripherial
+    <xacro:property name="d415_cam_width" value="0.099"/>
+    <xacro:property name="d415_cam_height" value="0.023"/>
+    <xacro:property name="d415_cam_depth" value="0.02005"/>
+    <xacro:property name="d415_cam_mount_from_center_offset" value="0.00987"/>
+    <!-- The following offset is relative the the physical d415 camera peripherial
   	camera tripod mount -->
-    <xacro:property name="d435_cam_depth_px" value="${d435_cam_mount_from_center_offset}"/>
-    <xacro:property name="d435_cam_depth_py" value="0.0175"/>
-    <xacro:property name="d435_cam_depth_pz" value="${d435_cam_height/2}"/>
+    <xacro:property name="d415_cam_depth_px" value="${d415_cam_mount_from_center_offset}"/>
+    <xacro:property name="d415_cam_depth_py" value="0.020"/>
+    <xacro:property name="d415_cam_depth_pz" value="${d415_cam_height/2}"/>
 <!--  <material name="aluminum">-->
 <!--    <color rgba="0.5 0.5 0.5 1"/>-->
@@ -38,5 +38,5 @@
     <link name="${prefix}_camera_bottom_screw_frame"/>
     <joint name="${prefix}_camera_link_joint" type="fixed">
-      <origin xyz="0 ${d435_cam_depth_py} ${d435_cam_depth_pz}" rpy="0 0 0"/>
+      <origin xyz="0 ${d415_cam_depth_py} ${d415_cam_depth_pz}" rpy="0 0 0"/>
       <parent link="${prefix}_camera_bottom_screw_frame"/>
       <child link="${prefix}_camera_link" />
@@ -44,17 +44,18 @@
     <link name="${prefix}_camera_link">
       <visual>
-      <!-- <origin xyz="${d435_cam_mount_from_center_offset} ${-d435_cam_depth_py} 0" rpy="${M_PI/2} 0 ${M_PI/2}"/> -->
-      <origin xyz="0 ${-d435_cam_mount_from_center_offset} 0" rpy="0 0 0"/>
+      <!-- <origin xyz="${d415_cam_mount_from_center_offset} ${-d415_cam_depth_py} 0" rpy="${M_PI/2} 0 ${M_PI/2}"/> -->
+      <origin xyz="0 ${-d415_cam_mount_from_center_offset} 0" rpy="0 0 0"/>
         <geometry>
-          <!-- <box size="${d435_cam_width} ${d435_cam_height} ${d435_cam_depth}"/> -->
-	  <mesh filename="package://robotnik_sensors/meshes/intel_realsense_depth_camera_d435.dae" />
-          <!--<mesh filename="package://realsense2_camera/meshes/d435/d435.dae" />-->
+          <!-- <box size="${d415_cam_width} ${d415_cam_height} ${d415_cam_depth}"/> -->
+ 	  <mesh filename="package://robotnik_sensors/meshes/intel_realsense_depth_camera_d435.dae" />
+ 	  <!--<mesh filename="package://robotnik_sensors/meshes/intel_realsense_depth_camera_d415.stl" />  -->
+          <!--<mesh filename="package://realsense2_camera/meshes/d415.stl" />-->
         </geometry>
         <material name="aluminum"/>
       </visual>
       <collision>
-        <origin xyz="0 ${-d435_cam_depth_py} 0" rpy="0 0 0"/>
+        <origin xyz="0 ${-d415_cam_depth_py} 0" rpy="0 0 0"/>
         <geometry>
-        <box size="${d435_cam_depth} ${d435_cam_width} ${d435_cam_height}"/>
+        <box size="${d415_cam_depth} ${d415_cam_width} ${d415_cam_height}"/>
         </geometry>
       </collision>
@@ -81,5 +82,5 @@
     <!-- camera left IR joints and links -->
     <joint name="${prefix}_camera_left_ir_joint" type="fixed">
-      <origin xyz="0 ${d435_cam_depth_to_left_ir_offset} 0" rpy="0 0 0" />
+      <origin xyz="0 ${d415_cam_depth_to_left_ir_offset} 0" rpy="0 0 0" />
       <parent link="${prefix}_camera_depth_frame" />
       <child link="${prefix}_camera_left_ir_frame" />
@@ -94,5 +95,5 @@
     <!-- camera right IR joints and links -->
     <joint name="${prefix}_camera_right_ir_joint" type="fixed">
-      <origin xyz="0 ${d435_cam_depth_to_right_ir_offset} 0" rpy="0 0 0" />
+      <origin xyz="0 ${d415_cam_depth_to_right_ir_offset} 0" rpy="0 0 0" />
       <parent link="${prefix}_camera_depth_frame" />
       <child link="${prefix}_camera_right_ir_frame" />
@@ -107,5 +108,5 @@
     <!-- camera color joints and links -->
     <joint name="${prefix}_camera_color_joint" type="fixed">
-      <origin xyz="0 ${d435_cam_depth_to_color_offset} 0" rpy="0 0 0" />
+      <origin xyz="0 ${d415_cam_depth_to_color_offset} 0" rpy="0 0 0" />
       <parent link="${prefix}_camera_depth_frame" />
       <child link="${prefix}_camera_color_frame" />
@@ -119,7 +120,7 @@
     <link name="${prefix}_camera_color_optical_frame"/>
   <!-- RGBD sensor for simulation, same as Kinect -->
-  <sensor_d435_icclab_gazebo/>
+  <sensor_d415_icclab_gazebo/>
   </xacro:macro>
-   <xacro:macro name="sensor_d435_icclab_gazebo">
+   <xacro:macro name="sensor_d415_icclab_gazebo">
     <!-- gazebo reference="${prefix}_rgb_base_link" -->
     <gazebo reference="${prefix}_camera_link">
