Commit message: refactor hokuyo lidars implementation

File: urdf/sensors/hokuyo.urdf.xacro (robot description, xacro)
@@ -42,8 +42,8 @@
     </joint>
     <!-- simulation -->
-    <sensor_scanse_gazebo/>
+    <sensor_hokuyo_gazebo/>
   </xacro:macro>
 <!-- uses ROS Laser Scanner Controller plugin -->
-  <xacro:macro name="sensor_scanse_gazebo">
+  <xacro:macro name="sensor_hokuyo_gazebo">
     <gazebo reference="${prefix}_link">
       <sensor type="ray" name="${prefix}_sensor">
