Commit message: fine tuning gripper

File: urdf/Danfoa_140_2f_robotiq/robotiq_arg2f.gazebo.xacro (robot description, xacro)
@@ -3,32 +3,32 @@
     <xacro:macro name="robotiq_arg2f_gazebo" params="prefix">
         <gazebo>
-            <plugin filename="libroboticsgroup_gazebo_mimic_joint_plugin.so" name="${prefix}mimic_robotiq_140_1">
+            <plugin filename="libroboticsgroup_gazebo_mimic_joint_plugin.so" name="${prefix}mimic_robotiq_140_4">
                 <joint>${prefix}finger_joint</joint>
                 <mimicJoint>${prefix}right_outer_knuckle_joint</mimicJoint>
-                <multiplier>1.0</multiplier>
+                <multiplier>-1.0</multiplier>
                 <offset>0.0</offset>
             </plugin>
             <plugin filename="libroboticsgroup_gazebo_mimic_joint_plugin.so" name="${prefix}mimic_robotiq_140_2">
                 <joint>${prefix}finger_joint</joint>
-                <mimicJoint>${prefix}left_inner_knuckle_joint</mimicJoint>
-                <multiplier>1.0</multiplier>
+                <mimicJoint>${prefix}left_inner_finger_joint</mimicJoint>
+                <multiplier>-1.0</multiplier>
+                <offset>0.0</offset>
+            </plugin>
+            <plugin filename="libroboticsgroup_gazebo_mimic_joint_plugin.so" name="${prefix}mimic_robotiq_140_1">
+                <joint>${prefix}finger_joint</joint>
+                <mimicJoint>${prefix}right_inner_finger_joint</mimicJoint>
+                <multiplier>-1.0</multiplier>
                 <offset>0.0</offset>
             </plugin>
             <plugin filename="libroboticsgroup_gazebo_mimic_joint_plugin.so" name="${prefix}mimic_robotiq_140_3">
                 <joint>${prefix}finger_joint</joint>
-                <mimicJoint>${prefix}right_inner_knuckle_joint</mimicJoint>
-                <multiplier>1.0</multiplier>
-                <offset>0.0</offset>
-            </plugin>
-            <plugin filename="libroboticsgroup_gazebo_mimic_joint_plugin.so" name="${prefix}mimic_robotiq_140_4">
-                <joint>${prefix}finger_joint</joint>
-                <mimicJoint>${prefix}left_inner_finger_joint</mimicJoint>
-                <multiplier>1.0</multiplier>
+                <mimicJoint>${prefix}left_inner_knuckle_joint</mimicJoint>
+                <multiplier>-1.0</multiplier>
                 <offset>0.0</offset>
             </plugin>
             <plugin filename="libroboticsgroup_gazebo_mimic_joint_plugin.so" name="${prefix}mimic_robotiq_140_5">
                 <joint>${prefix}finger_joint</joint>
-                <mimicJoint>${prefix}right_inner_finger_joint</mimicJoint>
-                <multiplier>1.0</multiplier>
+                <mimicJoint>${prefix}right_inner_knuckle_joint</mimicJoint>
+                <multiplier>-1.0</multiplier>
                 <offset>0.0</offset>
             </plugin>

File: urdf/Danfoa_140_2f_robotiq/robotiq_arg2f_140_model_macro.xacro (robot description, xacro)
@@ -2,5 +2,6 @@
 <robot name="ur5" xmlns:xacro="http://ros.org/wiki/xacro">
   <xacro:include filename="$(find icclab_summit_xl)/urdf/Danfoa_140_2f_robotiq/robotiq_arg2f_transmission.xacro" />
-  <xacro:include filename="$(find icclab_summit_xl)/urdf/Danfoa_140_2f_robotiq/robotiq_arg2f.gazebo.xacro" />
+ <!-- import the xacro file -->
+ <xacro:include filename="$(find icclab_summit_xl)/urdf/Danfoa_140_2f_robotiq/robotiq_arg2f.gazebo.xacro" />
   <xacro:macro name="outer_knuckle" params="prefix fingerprefix stroke">
     <link name="${prefix}${fingerprefix}_outer_knuckle">
@@ -161,17 +162,5 @@
       <axis xyz="1 0 0" />
       <limit lower="0" upper="0.8757" velocity="2.0" effort="1000" />
-      <!-- mport the xacro file -->
-<xacro:include filename="$(find icclab_summit_xl)/urdf/Danfoa_140_2f_robotiq/robotiq_arg2f.gazebo.xacro" />
-<!-- Use it in the last xacro block -->
-<xacro:macro name="robotiq_arg2f_140" params="prefix">
-    <xacro:robotiq_arg2f_base_link prefix="${prefix}"/>
-    <xacro:finger_links prefix="${prefix}" fingerprefix="left" stroke="140"/>
-    <xacro:finger_links prefix="${prefix}" fingerprefix="right" stroke="140"/>
-    <xacro:finger_joint prefix="${prefix}"/>
-    <xacro:right_outer_knuckle_joint prefix="${prefix}"/>
-    <xacro:robotiq_arg2f_transmission0 prefix="${prefix}"/>
-    <xacro:robotiq_arg2f_transmission1 prefix="${prefix}"/>
-        <xacro:robotiq_arg2f_gazebo prefix="${prefix}"/>
-</xacro:macro><mimic joint="${prefix}finger_joint" multiplier="-1" offset="0" />
+      <mimic joint="${prefix}finger_joint" multiplier="1" offset="0" />
     </joint>
   </xacro:macro>
@@ -216,4 +205,5 @@
     <xacro:finger_joints prefix="${prefix}" fingerprefix="right" reflect="-1.0"/>
   </xacro:macro>
+  <!-- Use it in the last xacro block -->
   <xacro:macro name="robotiq_arg2f_140" params="prefix">
     <xacro:robotiq_arg2f_base_link prefix="${prefix}"/>
@@ -224,5 +214,5 @@
     <xacro:robotiq_arg2f_transmission0 prefix="${prefix}"/>
     <xacro:robotiq_arg2f_transmission1 prefix="${prefix}"/>
-        <xacro:robotiq_arg2f_gazebo prefix="${prefix}"/>
+    <xacro:robotiq_arg2f_gazebo prefix="${prefix}"/>
   </xacro:macro>
 </robot>

File: urdf/Danfoa_140_2f_robotiq/robotiq_arg2f_transmission.xacro (robot description, xacro)
@@ -14,11 +14,10 @@
   </xacro:macro>
   <xacro:macro name="robotiq_arg2f_transmission1" params="prefix">
-    <transmission name="${prefix}right_outer_knuckle_joint_trans">
+    <transmission name="${prefix}right_inner_finger_joint_trans">
       <type>transmission_interface/SimpleTransmission</type>
-      <joint name="${prefix}right_outer_knuckle_joint">
-        <!--hardwareInterface>hardware_interface/PositionJointInterface</hardwareInterface-->
+      <joint name="${prefix}right_inner_finger_joint">
         <hardwareInterface>hardware_interface/EffortJointInterface</hardwareInterface>
       </joint>
-      <actuator name="${prefix}right_outer_knuckle_joint_motor">
+      <actuator name="${prefix}right_inner_finger_joint_motor">
         <mechanicalReduction>1</mechanicalReduction>
       </actuator>

Commit message: gripper fixed and renders as it should on gazebo and rviz

File: urdf/Danfoa_140_2f_robotiq/robotiq_arg2f.gazebo.xacro (robot description, xacro)
@@ -3,5 +3,5 @@
     <xacro:macro name="robotiq_arg2f_gazebo" params="prefix">
         <gazebo>
-            <plugin filename="libroboticsgroup_gazebo_mimic_joint_plugin.so" name="${prefix}mimic_robotiq_140_4">
+            <plugin filename="libroboticsgroup_gazebo_mimic_joint_plugin.so" name="${prefix}mimic_robotiq_140_1">
                 <joint>${prefix}finger_joint</joint>
                 <mimicJoint>${prefix}right_outer_knuckle_joint</mimicJoint>
@@ -11,11 +11,5 @@
             <plugin filename="libroboticsgroup_gazebo_mimic_joint_plugin.so" name="${prefix}mimic_robotiq_140_2">
                 <joint>${prefix}finger_joint</joint>
-                <mimicJoint>${prefix}left_inner_finger_joint</mimicJoint>
-                <multiplier>-1.0</multiplier>
-                <offset>0.0</offset>
-            </plugin>
-            <plugin filename="libroboticsgroup_gazebo_mimic_joint_plugin.so" name="${prefix}mimic_robotiq_140_1">
-                <joint>${prefix}finger_joint</joint>
-                <mimicJoint>${prefix}right_inner_finger_joint</mimicJoint>
+                <mimicJoint>${prefix}left_inner_knuckle_joint</mimicJoint>
                 <multiplier>-1.0</multiplier>
                 <offset>0.0</offset>
@@ -23,12 +17,18 @@
             <plugin filename="libroboticsgroup_gazebo_mimic_joint_plugin.so" name="${prefix}mimic_robotiq_140_3">
                 <joint>${prefix}finger_joint</joint>
-                <mimicJoint>${prefix}left_inner_knuckle_joint</mimicJoint>
+                <mimicJoint>${prefix}right_inner_knuckle_joint</mimicJoint>
                 <multiplier>-1.0</multiplier>
+                <offset>0.0</offset>
+            </plugin>
+            <plugin filename="libroboticsgroup_gazebo_mimic_joint_plugin.so" name="${prefix}mimic_robotiq_140_4">
+                <joint>${prefix}finger_joint</joint>
+                <mimicJoint>${prefix}left_inner_finger_joint</mimicJoint>
+                <multiplier>1.0</multiplier>
                 <offset>0.0</offset>
             </plugin>
             <plugin filename="libroboticsgroup_gazebo_mimic_joint_plugin.so" name="${prefix}mimic_robotiq_140_5">
                 <joint>${prefix}finger_joint</joint>
-                <mimicJoint>${prefix}right_inner_knuckle_joint</mimicJoint>
-                <multiplier>-1.0</multiplier>
+                <mimicJoint>${prefix}right_inner_finger_joint</mimicJoint>
+                <multiplier>1.0</multiplier>
                 <offset>0.0</offset>
             </plugin>

File: urdf/Danfoa_140_2f_robotiq/robotiq_arg2f_140_model_macro.xacro (robot description, xacro)
@@ -161,6 +161,6 @@
       <child link="${prefix}${fingerprefix}_inner_knuckle" />
       <axis xyz="1 0 0" />
-      <limit lower="0" upper="0.8757" velocity="2.0" effort="1000" />
-      <mimic joint="${prefix}finger_joint" multiplier="1" offset="0" />
+      <limit lower="-0.857" upper="0" velocity="2.0" effort="1000" />
+      <mimic joint="${prefix}finger_joint" multiplier="-1" offset="0" />
     </joint>
   </xacro:macro>
@@ -200,5 +200,5 @@
       <child link="${prefix}right_outer_knuckle" />
       <axis xyz="1 0 0" />
-      <limit lower="0" upper="0.725" velocity="2.0" effort="1000" />
+      <limit lower="0" upper="-0.725" velocity="2.0" effort="1000" />
     <mimic joint="${prefix}finger_joint" multiplier="-1" offset="0" />
     </joint>
@@ -212,6 +212,5 @@
     <xacro:finger_joint prefix="${prefix}"/>
     <xacro:right_outer_knuckle_joint prefix="${prefix}"/>
-    <xacro:robotiq_arg2f_transmission0 prefix="${prefix}"/>
-    <xacro:robotiq_arg2f_transmission1 prefix="${prefix}"/>
+    <xacro:robotiq_arg2f_transmission prefix="${prefix}"/>
     <xacro:robotiq_arg2f_gazebo prefix="${prefix}"/>
   </xacro:macro>

File: urdf/Danfoa_140_2f_robotiq/robotiq_arg2f_transmission.xacro (robot description, xacro)
@@ -1,10 +1,10 @@
 <?xml version="1.0"?>
 <robot xmlns:xacro="http://ros.org/wiki/xacro">
-  <xacro:macro name="robotiq_arg2f_transmission0" params="prefix">
+  <xacro:macro name="robotiq_arg2f_transmission" params="prefix">
     <transmission name="${prefix}finger_joint_trans">
       <type>transmission_interface/SimpleTransmission</type>
       <joint name="${prefix}finger_joint">
-        <!--hardwareInterface>hardware_interface/PositionJointInterface</hardwareInterface-->
-        <hardwareInterface>hardware_interface/EffortJointInterface</hardwareInterface>
+        <!--hardwareInterface>PositionJointInterface</hardwareInterface-->
+        <hardwareInterface>EffortJointInterface</hardwareInterface>
       </joint>
       <actuator name="${prefix}finger_joint_motor">
@@ -13,14 +13,3 @@
     </transmission>
   </xacro:macro>
-  <xacro:macro name="robotiq_arg2f_transmission1" params="prefix">
-    <transmission name="${prefix}right_inner_finger_joint_trans">
-      <type>transmission_interface/SimpleTransmission</type>
-      <joint name="${prefix}right_inner_finger_joint">
-        <hardwareInterface>hardware_interface/EffortJointInterface</hardwareInterface>
-      </joint>
-      <actuator name="${prefix}right_inner_finger_joint_motor">
-        <mechanicalReduction>1</mechanicalReduction>
-      </actuator>
-    </transmission>
-  </xacro:macro>
 </robot>
