Commit message: added grasp fix plugin from https://github.com/JenniferBuehler/gazebo-pkgs/wiki/The-Gazebo-grasp-fix-plugin . See installation requirements

File: urdf/gripper/schunk_egp40.urdf.xacro (robot description, xacro)
@@ -61,4 +61,7 @@
          <limit effort="10" lower="0.001" upper="0.015" velocity="0.041"/>
       </joint>
+      <gazebo reference="${prefix}left_finger_base_joint">
+        <implicitSpringDamper>1</implicitSpringDamper>
+      </gazebo>
       <link name="${prefix}left_finger_base_link">
          <inertial>
@@ -110,4 +113,11 @@
          </collision>
       </link>
+      <gazebo reference="${prefix}left_finger_link">
+        <kp>1000000.0</kp>
+        <kd>1.0</kd>
+        <mu1>1.0</mu1>
+        <mu2>1.0</mu2>
+        <minDepth>0.001</minDepth>
+      </gazebo>
       <!-- GRIPPER FINGER RIGHT -->
       <joint name="${prefix}right_finger_base_joint" type="prismatic">
@@ -118,4 +128,7 @@
          <limit effort="10" lower="0.001" upper="0.015" velocity="0.041"/>
       </joint>
+      <gazebo reference="${prefix}left_finger_base_joint">
+        <implicitSpringDamper>1</implicitSpringDamper>
+      </gazebo>
       <link name="${prefix}right_finger_base_link">
          <inertial>
@@ -158,13 +171,51 @@
             <material name="grey">
                <color rgba="0.5 0.5 0.5 1"/>
-            </material>
-         </visual>
-         <collision>
-            <origin xyz="0.0 0 0" rpy="0 0 0" />
-            <geometry>
-               <mesh filename="package://icclab_turtlebot/meshes/gripper/schunk_epg40/schunk_epg40_finger.stl" scale="1 1 1"/>
-            </geometry>
-         </collision>
-      </link>
+            </material>${prefix}right_finger_base_joint
+         </visual>
+         <collision>
+            <origin xyz="0.0 0 0" rpy="0 0 0" />
+            <geometry>
+               <mesh filename="package://icclab_turtlebot/meshes/gripper/schunk_epg40/schunk_epg40_finger.stl" scale="1 1 1"/>
+            </geometry>
+         </collision>
+      </link>
+      <gazebo reference="${prefix}right_finger_link">
+        <kp>1000000.0</kp>
+        <kd>1.0</kd>
+        <mu1>1.0</mu1>
+        <mu2>1.0</mu2>
+        <minDepth>0.001</minDepth>
+      </gazebo>
+    <gazebo>
+    <plugin name='ft_sensor_l' filename='libgazebo_ros_ft_sensor.so'>
+      <updateRate>100.0</updateRate>
+      <topicName>ft_sensor_left_finger</topicName>
+      <jointName>${prefix}left_finger_base_joint</jointName>
+    </plugin>
+    <static>0</static>
+    <plugin name='ft_sensor_r' filename='libgazebo_ros_ft_sensor.so'>
+      <updateRate>100.0</updateRate>
+      <topicName>ft_sensor_right_finger</topicName>
+      <jointName>${prefix}right_finger_base_joint</jointName>
+    </plugin>
+    </gazebo>
+    <!-- hack from here: https://github.com/JenniferBuehler/gazebo-pkgs/wiki/The-Gazebo-grasp-fix-plugin -->
+    <gazebo>
+       <plugin name="gazebo_grasp_fix" filename="libgazebo_grasp_fix.so">
+            <arm>
+               <arm_name>ur5-arm</arm_name>
+               <palm_link>arm_wrist_3_link</palm_link>
+               <gripper_link>${prefix}left_finger_base_link</gripper_link>
+               <gripper_link>${prefix}right_finger_base_link</gripper_link>
+            </arm>
+           <forces_angle_tolerance>100</forces_angle_tolerance>
+           <update_rate>4</update_rate>
+           <grip_count_threshold>4</grip_count_threshold>
+           <max_grip_count>8</max_grip_count>
+           <release_tolerance>0.005</release_tolerance>
+           <disable_collisions_on_attach>false</disable_collisions_on_attach>
+           <contact_topic>__default_topic__</contact_topic>
+        </plugin>
+    </gazebo>
     <xacro:default_transmission jname="${prefix}left_finger_base"/>
     <xacro:default_transmission jname="${prefix}right_finger_base"/>

Commit message: made simulated gripper wider

File: urdf/gripper/schunk_egp40.urdf.xacro (robot description, xacro)
@@ -59,5 +59,5 @@
          <origin xyz="-0.012 0 0.08915" rpy="0 0 0" />
          <axis xyz="-1 0 0" />
-         <limit effort="10" lower="0.001" upper="0.015" velocity="0.041"/>
+         <limit effort="10" lower="0.001" upper="0.035" velocity="0.041"/>
       </joint>
       <gazebo reference="${prefix}left_finger_base_joint">
@@ -126,5 +126,5 @@
          <origin xyz="0.012 0 0.08915" rpy="0 0 3.14" />
          <axis xyz="-1 0 0" />
-         <limit effort="10" lower="0.001" upper="0.015" velocity="0.041"/>
+         <limit effort="10" lower="0.001" upper="0.035" velocity="0.041"/>
       </joint>
       <gazebo reference="${prefix}left_finger_base_joint">

Commit message: arm fine tuning

File: urdf/gripper/schunk_egp40.urdf.xacro (robot description, xacro)
@@ -57,5 +57,5 @@
          <parent link="${prefix}base_link"/>
          <child link="${prefix}left_finger_base_link"/>
-         <origin xyz="-0.012 0 0.08915" rpy="0 0 0" />
+         <origin xyz="-0.031 0 0.08915" rpy="0 0 0" />
          <axis xyz="-1 0 0" />
          <limit effort="10" lower="0.001" upper="0.015" velocity="0.041"/>
@@ -124,5 +124,5 @@
          <parent link="${prefix}base_link"/>
          <child link="${prefix}right_finger_base_link"/>
-         <origin xyz="0.012 0 0.08915" rpy="0 0 3.14" />
+         <origin xyz="0.022 0 0.08915" rpy="0 0 3.14" />
          <axis xyz="-1 0 0" />
          <limit effort="10" lower="0.001" upper="0.015" velocity="0.041"/>
