Commit message: added _mimic to gripper joints in sim so move_it stops complaining. See https://github.com/ros-controls/gazebo_ros2_control/issues/173

File: icclab_summit_xl/urdf/robotiq_gripper/robotiq_gripper.ros2_control.xacro (robot description, xacro)
@@ -8,5 +8,6 @@
         use_fake_hardware:=false
         fake_sensor_commands:=false
-        com_port:=/dev/ttyUSB0">
+        com_port:=/dev/ttyUSB0
+        suffix:=_mimic">
         <ros2_control name="${name}" type="system">
             <!-- Plugins -->
@@ -44,5 +45,5 @@
             <!-- When simulating we need to include the rest of the gripper joints -->
             <xacro:if value="${use_fake_hardware or sim_isaac or sim_ignition}">
-                <joint name="${prefix}robotiq_85_right_knuckle_joint">
+                <joint name="${prefix}robotiq_85_right_knuckle_joint${suffix}">
                     <param name="mimic">${prefix}robotiq_85_left_knuckle_joint</param>
                     <param name="multiplier">-1</param>
@@ -53,5 +54,5 @@
                     </xacro:unless>
                 </joint>
-                <joint name="${prefix}robotiq_85_left_inner_knuckle_joint">
+                <joint name="${prefix}robotiq_85_left_inner_knuckle_joint${suffix}">
                     <param name="mimic">${prefix}robotiq_85_left_knuckle_joint</param>
                     <param name="multiplier">1</param>
@@ -62,5 +63,5 @@
                     </xacro:unless>
                 </joint>
-                <joint name="${prefix}robotiq_85_right_inner_knuckle_joint">
+                <joint name="${prefix}robotiq_85_right_inner_knuckle_joint${suffix}">
                     <param name="mimic">${prefix}robotiq_85_left_knuckle_joint</param>
                     <param name="multiplier">-1</param>
@@ -71,5 +72,5 @@
                     </xacro:unless>
                 </joint>
-                <joint name="${prefix}robotiq_85_left_finger_tip_joint">
+                <joint name="${prefix}robotiq_85_left_finger_tip_joint${suffix}">
                     <param name="mimic">${prefix}robotiq_85_left_knuckle_joint</param>
                     <param name="multiplier">-1</param>
@@ -80,5 +81,5 @@
                     </xacro:unless>
                 </joint>
-                <joint name="${prefix}robotiq_85_right_finger_tip_joint">
+                <joint name="${prefix}robotiq_85_right_finger_tip_joint${suffix}">
                     <param name="mimic">${prefix}robotiq_85_left_knuckle_joint</param>
                     <param name="multiplier">1</param>

File: icclab_summit_xl_move_it_config/config/summit_xl.ros2_control.xacro (robot description, xacro)
@@ -50,4 +50,11 @@
                 <state_interface name="velocity"/>
             </joint>
+            <joint name="robotiq_85_left_knuckle_joint">
+                <command_interface name="position"/>
+                <state_interface name="position">
+                  <param name="initial_value">${initial_positions['robotiq_85_left_knuckle_joint']}</param>
+                </state_interface>
+                <state_interface name="velocity"/>
+            </joint>
         </ros2_control>
     </xacro:macro>
