Commit message: use find to get camera mount mesh

File: icclab_summit_xl/urdf/sensors/intel_camera_mount.urdf.xacro (robot description, xacro)
@@ -12,5 +12,5 @@
       <origin xyz="0 0 0" rpy="0 0 0"/>
         <geometry>
-          <mesh filename="package://icclab_summit_xl/meshes/camera_mount/RealSense_D435_UR5_camera_mount.stl" scale="0.00095 0.00095 0.00095"/>
+          <mesh filename="$(find icclab_summit_xl)/meshes/camera_mount/RealSense_D435_UR5_camera_mount.stl" scale="0.00095 0.00095 0.00095"/>
         </geometry>
         <material name="white">

Commit message: fixed rviz2 error in importing arm camera mount

File: icclab_summit_xl/urdf/sensors/intel_camera_mount.urdf.xacro (robot description, xacro)
@@ -12,5 +12,5 @@
       <origin xyz="0 0 0" rpy="0 0 0"/>
         <geometry>
-          <mesh filename="$(find icclab_summit_xl)/meshes/camera_mount/RealSense_D435_UR5_camera_mount.stl" scale="0.00095 0.00095 0.00095"/>
+          <mesh filename="file://$(find icclab_summit_xl)/meshes/camera_mount/RealSense_D435_UR5_camera_mount.stl" scale="0.00095 0.00095 0.00095"/>
         </geometry>
         <material name="white">
