Commit message: updated back box vis

File: icclab_summit_xl/urdf/sensors/back_box.urdf.xacro (robot description, xacro)
@@ -11,5 +11,5 @@
     </material>
     <link name="back_box_link">
-      <visual>
+      <!-- <visual>
       <origin xyz="0 0 0" rpy="0 0 0"/>
         <geometry>
@@ -17,5 +17,5 @@
         </geometry>
         <material name="black"/>
-      </visual>
+      </visual> -->
       <collision>
         <origin xyz="0.0 0.0 0.0" rpy="0 0 0"/>
@@ -27,5 +27,5 @@
         <mass value="1.0"/>
         <origin xyz="0 0 0"/>
-        <inertia ixx="0.0167" ixy="0" ixz="0" iyy="0.0202" iyz="0" izz="0.0302"/>
+        <inertia ixx="0.0167" ixy="0" ixz="0" iyy="0.0085" iyz="0" izz="0.0185"/>
       </inertial>
     </link>
