Commit message: changed oak camera frame name to be consistent with the camera driver

File: icclab_summit_xl/urdf/sensors/luxonis_oak_d_pro.urdf.xacro (robot description, xacro)
@@ -7,5 +7,6 @@
 	  <xacro:insert_block name="origin" />
 	</xacro:luxonis>
-	<xacro:luxonis_camera_gazebo ns="${ns}" prefix="${prefix}" frame="${prefix}_color_optical_frame"/>
+	<!-- <xacro:luxonis_camera_gazebo ns="${ns}" prefix="${prefix}" frame="${prefix}_color_optical_frame"/> -->
+	<xacro:luxonis_camera_gazebo ns="${ns}" prefix="${prefix}" frame="oak_rgb_camera_optical_frame"/>
 </xacro:macro>
 </robot>

File: icclab_summit_xl/urdf/sensors/luxonis_oak_d_pro_model.urdf.xacro (robot description, xacro)
@@ -62,11 +62,11 @@
 		  	<origin xyz="0 0 0" rpy="0 0 0" />
 		</joint>
-		<!-- <link name="oak_rgb_camera_optical_frame" /> -->
-    <link name="arm_camera_color_optical_frame" />
+		<link name="oak_rgb_camera_optical_frame" />
+    <!-- <link name="arm_camera_color_optical_frame" /> -->
 		<joint name="oak_rgb_camera_optical_joint" type="fixed">
 				<origin xyz="0 0 0" rpy="-${M_PI/2} 0.0 -${M_PI/2}" />
 				<parent link="oak_rgb_camera_frame" />
-				<!-- <child link="oak_rgb_camera_optical_frame" /> -->
-        		<child link="arm_camera_color_optical_frame" />
+				<child link="oak_rgb_camera_optical_frame" />
+        		<!-- <child link="arm_camera_color_optical_frame" /> -->
 		</joint>
     <!-- Left Camera -->

Commit message: fixed controller startup sequence, gazebo now starts unpaused

File: icclab_summit_xl/urdf/sensors/luxonis_oak_d_pro.urdf.xacro (robot description, xacro)
@@ -9,5 +9,5 @@
 	<link name="oak-d_frame_rotated"/>
 	<joint name="oak-d_frame_rotated_joint" type="fixed">
-	  <origin xyz="0 0 0" rpy="${PI} 0 0" />
+	  <origin xyz="0.02 0 0" rpy="${PI} 0 0" />
 	  <parent link="oak-d_frame"/>
 	  <child link="oak-d_frame_rotated"/>
