Commit message: added new ur5 calib file

File: icclab_summit_xl/urdf/arm/ur.urdf.xacro (robot description, xacro)
@@ -14,6 +14,8 @@
     <xacro:property name="joint_limit_params"
       default="$(find ur_description)/config/${ur_type}/joint_limits.yaml" />
+    <!-- <xacro:property name="kinematics_params"
+      default="$(find icclab_summit_xl)/config/ur5_calibrated_kinematics.yaml" /> -->
     <xacro:property name="kinematics_params"
-      default="$(find icclab_summit_xl)/config/ur5_calibrated_kinematics.yaml" />
+      default="$(find icclab_summit_xl)/config/ur5_calibrated_kinematics_01042025.yaml" />
     <xacro:property name="physical_params"
       default="$(find ur_description)/config/${ur_type}/physical_parameters.yaml" />
