Commit message: added robotiq 2f_85 griper (waiting for 2f_140 here https://github.com/PickNikRobotics/ros2_robotiq_gripper/pull/18), cleaned up old files

File: icclab_summit_xl/robots/summit_xls_icclab.urdf.xacro (robot description, xacro)
@@ -15,6 +15,8 @@
 	<!-- Import our modified sensor -->
 	<xacro:include filename="$(find summit_xl_description)/urdf/sensors/hokuyo_ust20lx_no_frame_prefix.urdf.xacro" />
-	<!-- import arm -->
+	<!-- Import arm -->
 	<xacro:include filename="$(find icclab_summit_xl)/urdf/arm/ur.urdf.xacro" />
+	<!-- Import gripper -->
+    <xacro:include filename="$(find icclab_summit_xl)/urdf/robotiq_gripper/robotiq_2f_85_macro.urdf.xacro" />
 	<xacro:property name="PI" value="3.1415926535897931"/>
 	<!-- Wheel parameters -->
@@ -93,4 +95,7 @@
 			<origin xyz="${gps_offset_x} ${gps_offset_y} ${gps_offset_z}" rpy="0 0 0"/>
 		</xacro:sensor_gps-->
+		<xacro:robotiq_gripper name="RobotiqGripperHardwareInterface" prefix="" parent="arm_flange" use_fake_hardware="true">
+        	<origin xyz="0 0 0" rpy="${-1/2*PI} 0 ${-1/2*PI}" />
+    	</xacro:robotiq_gripper>
    </xacro:macro>
    <xacro:if value="$(arg ros_planar_move_plugin)">

Commit message: added correct lidar model

File: icclab_summit_xl/robots/summit_xls_icclab.urdf.xacro (robot description, xacro)
@@ -14,7 +14,7 @@
 	<xacro:include filename="$(find robotnik_sensors)/urdf/all_sensors.urdf.xacro" />
 	<!-- Import our modified sensor -->
-	<xacro:include filename="$(find summit_xl_description)/urdf/sensors/hokuyo_ust20lx_no_frame_prefix.urdf.xacro" />
+	<xacro:include filename="$(find icclab_summit_xl)/urdf/sensors/hokuyo_utm30lx_no_frame_prefix.urdf.xacro" />
 	<xacro:include filename="$(find icclab_summit_xl)/urdf/sensors/orbbec_astra.urdf.xacro" />
-	<!-- Import arm -->
+	<!-- Import and create arm -->
 	<xacro:include filename="$(find icclab_summit_xl)/urdf/arm/ur.urdf.xacro" />
 	<!-- Import gripper -->
@@ -78,10 +78,10 @@
 		</xacro:sensor_imu_hector>
 		<!-- SENSORS -->
-		<xacro:sensor_hokuyo_ust20lx_no_frame_prefix ns="$(arg robot_ns)" prefix="front_laser" parent="base_link">
-			<origin xyz="${front_laser_offset_x} ${front_laser_offset_y} ${front_laser_offset_z}" rpy="0 ${-PI} ${3/4*PI}" />
-  		</xacro:sensor_hokuyo_ust20lx_no_frame_prefix>
-        <xacro:sensor_hokuyo_ust20lx_no_frame_prefix ns="$(arg robot_ns)" prefix="rear_laser" parent="base_link">
-			<origin xyz="${rear_laser_offset_x} ${rear_laser_offset_y} ${rear_laser_offset_z}" rpy="0 ${-PI} ${-1/4*PI}" />
-  		</xacro:sensor_hokuyo_ust20lx_no_frame_prefix>
+		<xacro:sensor_hokuyo_utm30lx_no_frame_prefix ns="$(arg robot_ns)" prefix="front_laser" parent="base_link" min_angle="${-3/4*PI}" max_angle="${3/4*PI}" gpu="false">
+			<origin xyz="${front_laser_offset_x} ${front_laser_offset_y} ${front_laser_offset_z}" rpy="0 0 ${-1/4*PI}" />
+  		</xacro:sensor_hokuyo_utm30lx_no_frame_prefix>
+        <xacro:sensor_hokuyo_utm30lx_no_frame_prefix ns="$(arg robot_ns)" prefix="rear_laser" parent="base_link" min_angle="${-3/4*PI}" max_angle="${3/4*PI}" gpu="false">
+			<origin xyz="${rear_laser_offset_x} ${rear_laser_offset_y} ${rear_laser_offset_z}" rpy="0 0 ${3/4*PI}" />
+  		</xacro:sensor_hokuyo_utm30lx_no_frame_prefix>
 		<!--xacro:sensor_axis_m5013 prefix="$(arg prefix)front_ptz_camera" parent="$(arg prefix)base_link">
 			<origin xyz="${front_ptz_camera_offset_x} ${front_ptz_camera_offset_y} ${front_ptz_camera_offset_z}" rpy="${-PI/2} 0 0"/>

Commit message: Moved front camera, added arm camera. Missing gazebo sensor WIP

File: icclab_summit_xl/robots/summit_xls_icclab.urdf.xacro (robot description, xacro)
@@ -16,4 +16,6 @@
 	<xacro:include filename="$(find icclab_summit_xl)/urdf/sensors/hokuyo_utm30lx_no_frame_prefix.urdf.xacro" />
 	<xacro:include filename="$(find icclab_summit_xl)/urdf/sensors/orbbec_astra.urdf.xacro" />
+	<xacro:include filename="$(find icclab_summit_xl)/urdf/sensors/intel_d435.urdf.xacro" />
+	<xacro:include filename="$(find icclab_summit_xl)/urdf/sensors/intel_camera_mount.urdf.xacro" />
 	<!-- Import and create arm -->
 	<xacro:include filename="$(find icclab_summit_xl)/urdf/arm/ur.urdf.xacro" />
@@ -43,5 +45,5 @@
 	<xacro:property name="front_rgbd_camera_offset_x" value="0.35850"/>
 	<xacro:property name="front_rgbd_camera_offset_y" value="0.0"/>
-	<xacro:property name="front_rgbd_camera_offset_z" value="0.25062"/>
+	<xacro:property name="front_rgbd_camera_offset_z" value="0.22062"/>
 	<xacro:property name="gps_offset_x" value="-0.365"/>
 	<xacro:property name="gps_offset_y" value="-0.167"/>
@@ -99,4 +101,13 @@
         	<origin xyz="0 0 0" rpy="${-1/2*PI} 0 ${-1/2*PI}" />
     	</xacro:robotiq_gripper>
+		<!-- Camera mount -->
+		<xacro:camera_mount prefix="arm" parent="arm_flange">
+			<origin xyz="0 0 0" rpy="${-PI/2} 0 ${-PI/2}" />
+		</xacro:camera_mount>
+		<!-- Camera on gripper  -->
+		<!-- had to copy and modidy camera to avoid name clash with robotnik defined sensors -->
+		<xacro:sensor_d435_icclab prefix="arm" prefix_topic="summit_xl/arm_camera" parent="arm_camera_mount_link">
+     		  <origin xyz="0.0 0.06 0.01" rpy="${PI} ${-PI/2} ${PI/2}"/> <!-- camera on gripper -->
+   		</xacro:sensor_d435_icclab>
    </xacro:macro>
    <xacro:if value="$(arg ros_planar_move_plugin)">

File: icclab_summit_xl/urdf/sensors/intel_d435.urdf.xacro (robot description, xacro)
@@ -2,13 +2,12 @@
 <robot xmlns:xacro="http://www.ros.org/wiki/xacro" name="realsense">
 <xacro:include filename="$(find realsense2_description)/urdf/_d435.urdf.xacro" />
-<xacro:include filename="$(find icclab_grasping_niryo)/urdf/_d435.gazebo.kinect.xacro"/>
-<xacro:macro name="sensor_d435_icclab" params="parent *origin prefix:=arm prefix_topic:=arm_camera use_nominal_extrinsics:=true add_plug:=false use_mesh:=true">
+<!-- <xacro:include filename="$(find icclab_grasping_niryo)/urdf/_d435.gazebo.kinect.xacro"/> -->
+<xacro:macro name="sensor_d435_icclab" params="parent *origin prefix:=arm prefix_topic:=arm_camera use_nominal_extrinsics:=true add_plug:=true use_mesh:=true">
 	<xacro:sensor_d435 parent="${parent}" name="${prefix}_camera" use_nominal_extrinsics="${use_nominal_extrinsics}" add_plug="${add_plug}" use_mesh="${use_mesh}">
 	  <xacro:insert_block name="origin" />
 	</xacro:sensor_d435>
-	<xacro:gazebo_d435 camera_name="${prefix}_camera"/>
+	<!-- <xacro:gazebo_d435 camera_name="${prefix}_camera"/> -->
 	<!-- Realsense Gazebo Plugin -->
-	<!--
-	<xacro:include filename="$(find icclab_grasping_niryo)/urdf/_d435.gazebo.xacro"/>
+	<!-- <xacro:include filename="$(find icclab_grasping_niryo)/urdf/_d435.gazebo.xacro"/>
 	<xacro:gazebo_d435 camera_name="${prefix}_camera_" reference_link="${prefix}_camera_link" topics_ns="${prefix_topic}"
 	depth_optical_frame="${prefix}_camera_depth_optical_frame" color_optical_frame="${prefix}_camera_color_optical_frame"

File: icclab_summit_xl/urdf/sensors/orbbec_astra.urdf.xacro (robot description, xacro)
@@ -57,6 +57,6 @@
       <sensor name="${prefix}" type="depth">
         <pose>0 0 0 0 0 0</pose>
-        <visualize>false</visualize>
-        <update_rate>5</update_rate>
+        <visualize>true</visualize>
+        <update_rate>15</update_rate>
         <camera>
           <horizontal_fov>1,04719755</horizontal_fov>
@@ -80,6 +80,6 @@
           </ros>
           <frame_name>${prefix}_rgb_optical_frame</frame_name>
-          <min_depth>0.2</min_depth>
-          <max_depth>6.5</max_depth>
+          <min_depth>0.05</min_depth>
+          <max_depth>20.0</max_depth>
         </plugin>
       </sensor>

Commit message: Added robotiq 2f_140 gripper, including controller, updated move_it_config

File: icclab_summit_xl/robots/summit_xls_icclab.urdf.xacro (robot description, xacro)
@@ -21,5 +21,5 @@
 	<xacro:include filename="$(find icclab_summit_xl)/urdf/arm/ur.urdf.xacro" />
 	<!-- Import gripper -->
-    <xacro:include filename="$(find icclab_summit_xl)/urdf/robotiq_gripper/robotiq_2f_85_macro.urdf.xacro" />
+    <xacro:include filename="$(find robotiq_description)/urdf/robotiq_2f_140_macro.urdf.xacro" />
 	<xacro:property name="PI" value="3.1415926535897931"/>
 	<!-- Wheel parameters -->
@@ -98,6 +98,6 @@
 			<origin xyz="${gps_offset_x} ${gps_offset_y} ${gps_offset_z}" rpy="0 0 0"/>
 		</xacro:sensor_gps-->
-		<xacro:robotiq_gripper name="RobotiqGripperHardwareInterface" prefix="" parent="arm_flange" use_fake_hardware="true">
-        	<origin xyz="0 0 0" rpy="${-1/2*PI} 0 ${-1/2*PI}" />
+		<xacro:robotiq_gripper name="RobotiqGripperHardwareInterface" prefix="" parent="arm_tool0" use_fake_hardware="true">
+        	<origin xyz="0 0 0" rpy="0 0 0" />
     	</xacro:robotiq_gripper>
 		<!-- Camera mount -->

File: icclab_summit_xl/urdf/robotiq_gripper/2f_140.ros2_control.xacro (robot description, xacro)
@@ -1,20 +1,22 @@
 <?xml version="1.0"?>
+<!-- Taken from https://github.com/PickNikRobotics/ros2_robotiq_gripper and updated to work on Gazebo 11 / humble-->
 <robot xmlns:xacro="http://www.ros.org/wiki/xacro">
-    <xacro:macro name="robotiq_gripper_ros2_control_icclab" params="
+    <xacro:macro name="robotiq_gripper_ros2_control" params="
         name
         prefix
         sim_ignition:=false
         sim_isaac:=false
+        isaac_joint_commands:=/isaac_joint_commands
+        isaac_joint_states:=/isaac_joint_states
         use_fake_hardware:=false
         fake_sensor_commands:=false
-        com_port:=/dev/ttyUSB0
-        suffix:=_mimic">
+        com_port:=/dev/ttyUSB0">
         <ros2_control name="${name}" type="system">
             <!-- Plugins -->
             <hardware>
                 <xacro:if value="${sim_isaac}">
-                    <plugin>isaac_ros2_control/IsaacSystem</plugin>
-                    <param name="joint_commands_topic">/isaac_joint_commands</param>
-                    <param name="joint_states_topic">/isaac_joint_states</param>
+                    <plugin>topic_based_ros2_control/TopicBasedSystem</plugin>
+                    <param name="joint_commands_topic">${isaac_joint_commands}</param>
+                    <param name="joint_states_topic">${isaac_joint_states}</param>
                 </xacro:if>
                 <xacro:if value="${sim_ignition}">
@@ -28,5 +30,5 @@
                 <xacro:unless value="${use_fake_hardware or sim_ignition or sim_isaac}">
                     <plugin>robotiq_driver/RobotiqGripperHardwareInterface</plugin>
-                    <param name="gripper_closed_position">0.7929</param>
+                    <param name="gripper_closed_position">0.695</param>
                     <param name="COM_port">${com_port}</param>
                     <param name="gripper_speed_multiplier">1.0</param>
@@ -36,8 +38,8 @@
             <!-- Joint interfaces -->
             <!-- With Ignition or Hardware, they handle mimic joints, so we only need this command interface activated -->
-            <joint name="${prefix}robotiq_85_left_knuckle_joint">
+            <joint name="${prefix}finger_joint">
                 <command_interface name="position" />
                 <state_interface name="position">
-                    <param name="initial_value">0.7929</param>
+                    <param name="initial_value">0.695</param>
                 </state_interface>
                 <state_interface name="velocity"/>
@@ -45,6 +47,6 @@
             <!-- When simulating we need to include the rest of the gripper joints -->
             <xacro:if value="${use_fake_hardware or sim_isaac or sim_ignition}">
-                <joint name="${prefix}robotiq_85_right_knuckle_joint${suffix}">
-                    <param name="mimic">${prefix}robotiq_85_left_knuckle_joint</param>
+                <joint name="${prefix}left_inner_knuckle_joint">
+                    <param name="mimic">${prefix}finger_joint</param>
                     <param name="multiplier">-1</param>
                     <xacro:unless value="${sim_ignition}">
@@ -54,6 +56,6 @@
                     </xacro:unless>
                 </joint>
-                <joint name="${prefix}robotiq_85_left_inner_knuckle_joint${suffix}">
-                    <param name="mimic">${prefix}robotiq_85_left_knuckle_joint</param>
+                <joint name="${prefix}left_inner_finger_joint">
+                    <param name="mimic">${prefix}finger_joint</param>
                     <param name="multiplier">1</param>
                     <xacro:unless value="${sim_ignition}">
@@ -63,6 +65,6 @@
                     </xacro:unless>
                 </joint>
-                <joint name="${prefix}robotiq_85_right_inner_knuckle_joint${suffix}">
-                    <param name="mimic">${prefix}robotiq_85_left_knuckle_joint</param>
+                <joint name="${prefix}right_outer_knuckle_joint">
+                    <param name="mimic">${prefix}finger_joint</param>
                     <param name="multiplier">-1</param>
                     <xacro:unless value="${sim_ignition}">
@@ -72,6 +74,6 @@
                     </xacro:unless>
                 </joint>
-                <joint name="${prefix}robotiq_85_left_finger_tip_joint${suffix}">
-                    <param name="mimic">${prefix}robotiq_85_left_knuckle_joint</param>
+                <joint name="${prefix}right_inner_knuckle_joint">
+                    <param name="mimic">${prefix}finger_joint</param>
                     <param name="multiplier">-1</param>
                     <xacro:unless value="${sim_ignition}">
@@ -81,6 +83,6 @@
                     </xacro:unless>
                 </joint>
-                <joint name="${prefix}robotiq_85_right_finger_tip_joint${suffix}">
-                    <param name="mimic">${prefix}robotiq_85_left_knuckle_joint</param>
+                <joint name="${prefix}right_inner_finger_joint">
+                    <param name="mimic">${prefix}finger_joint</param>
                     <param name="multiplier">1</param>
                     <xacro:unless value="${sim_ignition}">

File: icclab_summit_xl_move_it_config/config/summit_xl.ros2_control.xacro (robot description, xacro)
@@ -50,8 +50,8 @@
                 <state_interface name="velocity"/>
             </joint>
-            <joint name="robotiq_85_left_knuckle_joint">
+            <joint name="finger_joint">
                 <command_interface name="position"/>
                 <state_interface name="position">
-                  <param name="initial_value">${initial_positions['robotiq_85_left_knuckle_joint']}</param>
+                  <param name="initial_value">${initial_positions['finger_joint']}</param>
                 </state_interface>
                 <state_interface name="velocity"/>

Commit message: added arm camera in gazebo

File: icclab_summit_xl/robots/summit_xls_icclab.urdf.xacro (robot description, xacro)
@@ -107,5 +107,5 @@
 		<!-- Camera on gripper  -->
 		<!-- had to copy and modidy camera to avoid name clash with robotnik defined sensors -->
-		<xacro:sensor_d435_icclab prefix="arm" prefix_topic="summit_xl/arm_camera" parent="arm_camera_mount_link">
+		<xacro:sensor_d435_icclab prefix="arm_camera" ns="$(arg robot_ns)" parent="arm_camera_mount_link">
      		  <origin xyz="0.0 0.06 0.01" rpy="${PI} ${-PI/2} ${PI/2}"/> <!-- camera on gripper -->
    		</xacro:sensor_d435_icclab>

File: icclab_summit_xl/urdf/sensors/intel_d435.urdf.xacro (robot description, xacro)
@@ -2,15 +2,11 @@
 <robot xmlns:xacro="http://www.ros.org/wiki/xacro" name="realsense">
 <xacro:include filename="$(find realsense2_description)/urdf/_d435.urdf.xacro" />
-<!-- <xacro:include filename="$(find icclab_grasping_niryo)/urdf/_d435.gazebo.kinect.xacro"/> -->
-<xacro:macro name="sensor_d435_icclab" params="parent *origin prefix:=arm prefix_topic:=arm_camera use_nominal_extrinsics:=true add_plug:=true use_mesh:=true">
-	<xacro:sensor_d435 parent="${parent}" name="${prefix}_camera" use_nominal_extrinsics="${use_nominal_extrinsics}" add_plug="${add_plug}" use_mesh="${use_mesh}">
+<xacro:include filename="$(find icclab_summit_xl)/urdf/sensors/orbbec_astra.urdf.xacro"/>
+<xacro:macro name="sensor_d435_icclab" params="parent *origin prefix:=arm_camera use_nominal_extrinsics:=true add_plug:=true use_mesh:=true ns:=summit">
+	<xacro:sensor_d435 parent="${parent}" name="${prefix}" use_nominal_extrinsics="${use_nominal_extrinsics}" add_plug="${add_plug}" use_mesh="${use_mesh}">
 	  <xacro:insert_block name="origin" />
 	</xacro:sensor_d435>
-	<!-- <xacro:gazebo_d435 camera_name="${prefix}_camera"/> -->
-	<!-- Realsense Gazebo Plugin -->
-	<!-- <xacro:include filename="$(find icclab_grasping_niryo)/urdf/_d435.gazebo.xacro"/>
-	<xacro:gazebo_d435 camera_name="${prefix}_camera_" reference_link="${prefix}_camera_link" topics_ns="${prefix_topic}"
-	depth_optical_frame="${prefix}_camera_depth_optical_frame" color_optical_frame="${prefix}_camera_color_optical_frame"
-infrared1_optical_frame="${prefix}_camera_left_ir_optical_frame" infrared2_optical_frame="${prefix}_camera_right_ir_optical_frame"/>-->
+	<!-- reuse gazebo camera for orbec -->
+	<xacro:sensor_orbbec_astra_gazebo_icclab ns="${ns}" prefix="${prefix}" frame="${prefix}_color_optical_frame"/>
 </xacro:macro>
 </robot>

File: icclab_summit_xl/urdf/sensors/orbbec_astra.urdf.xacro (robot description, xacro)
@@ -50,7 +50,7 @@
     </joint>
     <link name="${prefix}_depth_optical_frame"/>
-    <xacro:sensor_orbbec_astra_gazebo_icclab ns="${ns}" prefix="${prefix}"/>
+    <xacro:sensor_orbbec_astra_gazebo_icclab ns="${ns}" prefix="${prefix}" frame="${prefix}_rgb_optical_frame"/>
   </xacro:macro>
-  <xacro:macro name="sensor_orbbec_astra_gazebo_icclab" params="ns prefix">
+  <xacro:macro name="sensor_orbbec_astra_gazebo_icclab" params="ns prefix frame">
     <xacro:property name="deg_to_rad" value="0.01745329251994329577"/>
     <gazebo reference="${prefix}_link">
@@ -72,4 +72,5 @@
           </clip>
         </camera>
+        <!-- plugin https://docs.ros.org/en/ros2_packages/rolling/api/gazebo_plugins/generated/classgazebo__plugins_1_1GazeboRosCamera.html -->
         <plugin name="${prefix}" filename="libgazebo_ros_camera.so">
           <ros>
@@ -78,6 +79,9 @@
             <remapping>~/camera_info:=~/color/camera_info</remapping>
             <remapping>~/image_raw/compressed:=~/color/image_raw/compressed</remapping>
+            <remapping>~/image_raw/compressedDepth:=~/color/image_raw/compressedDepth</remapping>
+            <remapping>~/image_raw/theora:=~/color/image_raw/theora</remapping>
           </ros>
-          <frame_name>${prefix}_rgb_optical_frame</frame_name>
+          <camera_name>${prefix}</camera_name>
+          <frame_name>${frame}</frame_name>
           <min_depth>0.05</min_depth>
           <max_depth>20.0</max_depth>
