Commit message: Extracted arm macro, restored working gripper in sim

File: icclab_summit_xl/robots/summit_xls_icclab.urdf.xacro (robot description, xacro)
@@ -18,6 +18,6 @@
 	<xacro:include filename="$(find icclab_summit_xl)/urdf/sensors/intel_d435.urdf.xacro" />
 	<xacro:include filename="$(find icclab_summit_xl)/urdf/sensors/intel_camera_mount.urdf.xacro" />
-	<!-- Import and create arm -->
-	<xacro:include filename="$(find icclab_summit_xl)/urdf/arm/ur.urdf.xacro" />
+	<!-- Import arm macros -->
+	<xacro:include filename="$(find icclab_summit_xl)/urdf/arm/ur.urdf.xacro"/>
 	<!-- Import gripper -->
     <xacro:include filename="$(find icclab_summit_xl)/urdf/robotiq_gripper/robotiq_2f_140_macro.urdf.xacro" />
@@ -52,9 +52,9 @@
 	<xacro:property name="hq" value="true" />
 	<xacro:arg name="prefix" default=""/> <!-- was: summit_xl_-->
+	<xacro:arg name="use_fake_hardware" default="true"/>
 	<xacro:arg name="ros_planar_move_plugin" default="true"/>
 	<xacro:arg name="gpu" default="false"/>
 	<xacro:arg name="robot_id" default="summit"/>
 	<xacro:arg name="robot_ns" default="$(arg robot_id)"/>
-	<xacro:arg name="use_fake_hardware" default="true"/>
     <xacro:macro name="summit_xl" params="prefix publish_bf hq">
 		<!-- *************** -->
@@ -99,4 +99,8 @@
 			<origin xyz="${gps_offset_x} ${gps_offset_y} ${gps_offset_z}" rpy="0 0 0"/>
 		</xacro:sensor_gps-->
+		<!-- Add arm -->
+		<xacro:icclab_summit_arm simulation="$(arg use_fake_hardware)">
+			<origin xyz="0.255 0 0.275" rpy="0 0 ${pi}" />
+		</xacro:icclab_summit_arm>
 		<xacro:robotiq_gripper name="RobotiqGripperHardwareInterface" prefix="" parent="arm_tool0" use_fake_hardware="$(arg use_fake_hardware)">
         	<origin xyz="0 0 0" rpy="0 0 0" />

File: icclab_summit_xl/urdf/arm/ur.urdf.xacro (robot description, xacro)
@@ -1,89 +1,56 @@
 <?xml version="1.0"?>
 <robot xmlns:xacro="http://wiki.ros.org/xacro" name="arm">
-   <!-- robot name parameter -->
-   <xacro:arg name="name" default="ur"/>
-   <!-- import main macro -->
-   <xacro:include filename="$(find ur_description)/urdf/ur_macro.xacro"/>
-   <!-- possible 'ur_type' values: ur3, ur3e, ur5, ur5e, ur10, ur10e, ur16e -->
-   <!-- the default value should raise an error in case this was called without defining the type -->
-   <xacro:arg name="ur_type" default="ur5"/>
-   <xacro:arg name="parent" default="base_link"/>
-   <!-- parameters -->
-   <xacro:arg name="tf_prefix" default="arm_" />
-   <xacro:arg name="joint_limit_params" default="$(find ur_description)/config/$(arg ur_type)/joint_limits.yaml"/>
-   <xacro:arg name="kinematics_params" default="$(find icclab_summit_xl)/config/ur5_calibrated_kinematics.yaml"/>
-   <xacro:arg name="physical_params" default="$(find ur_description)/config/$(arg ur_type)/physical_parameters.yaml"/>
-   <xacro:arg name="visual_params" default="$(find ur_description)/config/$(arg ur_type)/visual_parameters.yaml"/>
-   <xacro:arg name="transmission_hw_interface" default=""/>
-   <xacro:arg name="safety_limits" default="false"/>
-   <xacro:arg name="safety_pos_margin" default="0.15"/>
-   <xacro:arg name="safety_k_position" default="20"/>
-   <!-- ros2_control related parameters -->
-   <xacro:arg name="headless_mode" default="false" />
-   <xacro:arg name="robot_ip" default="0.0.0.0" />
-   <xacro:arg name="script_filename" default=""/>
-   <xacro:arg name="output_recipe_filename" default=""/>
-   <xacro:arg name="input_recipe_filename" default=""/>
-   <xacro:arg name="reverse_ip" default="0.0.0.0"/>
-   <xacro:arg name="script_command_port" default="50004"/>
-   <!--   tool communication related parameters-->
-   <xacro:arg name="use_tool_communication" default="false" />
-   <xacro:arg name="tool_voltage" default="0" />
-   <xacro:arg name="tool_parity" default="0" />
-   <xacro:arg name="tool_baud_rate" default="115200" />
-   <xacro:arg name="tool_stop_bits" default="1" />
-   <xacro:arg name="tool_rx_idle_chars" default="1.5" />
-   <xacro:arg name="tool_tx_idle_chars" default="3.5" />
-   <xacro:arg name="tool_device_name" default="/tmp/ttyUR" />
-   <xacro:arg name="tool_tcp_port" default="54321" />
-     <!-- Simulation parameters -->
-   <xacro:arg name="use_fake_hardware" default="false" />
-   <xacro:arg name="fake_sensor_commands" default="false" />
-   <xacro:arg name="sim_gazebo" default="true" />
-   <xacro:arg name="sim_ignition" default="false" />
-   <xacro:arg name="simulation_controllers" default="$(find icclab_summit_xl)/config/ur_controllers.yaml" />
-   <!-- initial position for simulations (Fake Hardware, Gazebo, Ignition) -->
-   <xacro:arg name="initial_positions_file" default="$(find ur_description)/config/initial_positions.yaml"/>
-   <!-- convert to property to use substitution in function -->
-   <xacro:property name="initial_positions_file" default="$(arg initial_positions_file)"/>
-   <!-- arm -->
-   <xacro:ur_robot
-     name="$(arg name)"
-     tf_prefix="$(arg tf_prefix)"
-     parent="$(arg parent)"
-     joint_limits_parameters_file="$(arg joint_limit_params)"
-     kinematics_parameters_file="$(arg kinematics_params)"
-     physical_parameters_file="$(arg physical_params)"
-     visual_parameters_file="$(arg visual_params)"
-     transmission_hw_interface="$(arg transmission_hw_interface)"
-     safety_limits="$(arg safety_limits)"
-     safety_pos_margin="$(arg safety_pos_margin)"
-     safety_k_position="$(arg safety_k_position)"
-     use_fake_hardware="$(arg use_fake_hardware)"
-     fake_sensor_commands="$(arg fake_sensor_commands)"
-     sim_gazebo="$(arg sim_gazebo)"
-     sim_ignition="$(arg sim_ignition)"
-     headless_mode="$(arg headless_mode)"
-     initial_positions="${xacro.load_yaml(initial_positions_file)}"
-     use_tool_communication="$(arg use_tool_communication)"
-     tool_voltage="$(arg tool_voltage)"
-     tool_parity="$(arg tool_parity)"
-     tool_baud_rate="$(arg tool_baud_rate)"
-     tool_stop_bits="$(arg tool_stop_bits)"
-     tool_rx_idle_chars="$(arg tool_rx_idle_chars)"
-     tool_tx_idle_chars="$(arg tool_tx_idle_chars)"
-     tool_device_name="$(arg tool_device_name)"
-     tool_tcp_port="$(arg tool_tcp_port)"
-     robot_ip="$(arg robot_ip)"
-     script_filename="$(arg script_filename)"
-     output_recipe_filename="$(arg output_recipe_filename)"
-     input_recipe_filename="$(arg input_recipe_filename)"
-     reverse_ip="$(arg reverse_ip)"
-     script_command_port="$(arg script_command_port)"
-     >
-     <origin xyz="0.255 0 0.275" rpy="0 0 ${PI}" />  <!-- position robot in the world -->
-   </xacro:ur_robot>
-   <!-- Commented: we use a single controller manager and it's included by the robot base-->
-   <!-- <xacro:if value="$(arg sim_gazebo)">
+  <xacro:macro name="icclab_summit_arm" params="*origin
+    tf_prefix:=arm_
+    parent:=base_link
+    simulation:=true
+    sim_ignition:=false"
+    >
+    <!-- arm name  -->
+    <xacro:property name="name" default="icclab_ur5" />
+    <xacro:property name="ur_type" default="ur5" />
+    <xacro:property name="headless_mode" default="true" />
+    <!-- parameters -->
+    <xacro:property name="joint_limit_params"
+      default="$(find ur_description)/config/${ur_type}/joint_limits.yaml" />
+    <xacro:property name="kinematics_params"
+      default="$(find icclab_summit_xl)/config/ur5_calibrated_kinematics.yaml" />
+    <xacro:property name="physical_params"
+      default="$(find ur_description)/config/${ur_type}/physical_parameters.yaml" />
+    <xacro:property name="visual_params" default="$(find ur_description)/config/${ur_type}/visual_parameters.yaml"/>
+    <xacro:if value="${simulation}">
+      <!-- Simulation parameters -->
+      <xacro:property name="fake_sensor_commands" default="false" />
+      <xacro:property name="sim_gazebo" default="${not sim_ignition}" />
+      <xacro:property name="sim_ignition" default="${sim_ignition}" />
+      <xacro:property name="simulation_controllers"
+        default="$(find icclab_summit_xl)/config/ur_controllers.yaml" />
+        <xacro:property name="robot_ip" default="0.0.0.0" />
+    </xacro:if>
+    <xacro:unless value="${simulation}">
+      <xacro:property name="robot_ip" default="192.168.0.210" />
+    </xacro:unless>
+    <!-- import ur macro -->
+    <xacro:include filename="$(find ur_description)/urdf/ur_macro.xacro" />
+    <!-- call the actual ur macro -->
+    <!-- NOTE: we pass use_fake_hardware="false" to avoid generation of unneeded ros2 control plugins, i.e., mock_components/GenericSystem -->
+    <xacro:ur_robot
+      name="${name}"
+      tf_prefix="${tf_prefix}"
+      parent="${parent}"
+      joint_limits_parameters_file="${joint_limit_params}"
+      kinematics_parameters_file="${kinematics_params}"
+      physical_parameters_file="${physical_params}"
+      visual_parameters_file="${visual_params}"
+      use_fake_hardware="false"
+      sim_gazebo="${sim_gazebo}"
+      sim_ignition="${sim_ignition}"
+      headless_mode="${headless_mode}"
+      robot_ip="${robot_ip}"
+    >
+      <xacro:insert_block name="origin" />  <!-- position robot in the world -->
+    </xacro:ur_robot>
+    <!-- Commented: we use a single controller manager and it's included by the robot base-->
+    <!-- <xacro:if value="$(arg sim_gazebo)">
     <gazebo reference="$(arg tf_prefix)base_link">
     </gazebo>
@@ -95,14 +62,19 @@
     </gazebo>
   </xacro:if> -->
-  <xacro:if value="$(arg sim_ignition)">
-    <!-- Gazebo plugins -->
+    <!-- TODO: FIXME for Ignition
+  <xacro:if value="${sim_ignition}">
     <gazebo reference="$(arg tf_prefix)base_link">
     </gazebo>
     <gazebo>
-      <plugin filename="libign_ros2_control-system.so" name="ign_ros2_control::IgnitionROS2ControlPlugin">
+      <plugin filename="libign_ros2_control-system.so"
+    name="ign_ros2_control::IgnitionROS2ControlPlugin">
         <parameters>$(arg simulation_controllers)</parameters>
         <controller_manager_node_name>$(arg tf_prefix)controller_manager</controller_manager_node_name>
       </plugin>
     </gazebo>
-  </xacro:if>
+  </xacro:if> -->
+  </xacro:macro>
+  <!-- <xacro:icclab_summit_arm simulation="true">
+			<origin xyz="0.255 0 0.275" rpy="0 0 ${pi}" />
+	</xacro:icclab_summit_arm> -->
 </robot>

Commit message: lidars workkksing

File: icclab_summit_xl/robots/summit_xls_icclab.urdf.xacro (robot description, xacro)
@@ -117,5 +117,5 @@
    </xacro:macro>
    <xacro:if value="$(arg ros_planar_move_plugin)">
-	   <xacro:omni_steering namespace="$(arg robot_ns)" publish_tf="true"/>
+	   <xacro:omni_steering prefix="$(arg prefix)" publish_tf="true"/>
    </xacro:if>
    <xacro:summit_xl prefix="$(arg prefix)" publish_bf="true" hq="true"/>

File: icclab_summit_xl/urdf/arm/ur.urdf.xacro (robot description, xacro)
@@ -5,5 +5,5 @@
     parent:=base_link
     simulation:=true
-    sim_ignition:=false"
+    sim_ignition:=true"
     >
     <!-- arm name  -->
@@ -43,5 +43,5 @@
       physical_parameters_file="${physical_params}"
       visual_parameters_file="${visual_params}"
-      use_fake_hardware="false"
+      use_fake_hardware="true"
       sim_gazebo="${sim_gazebo}"
       sim_ignition="${sim_ignition}"

File: icclab_summit_xl/urdf/robotiq_gripper/2f_140.ros2_control.xacro (robot description, xacro)
@@ -5,9 +5,9 @@
         name
         prefix
-        sim_ignition:=false
+        sim_ignition:=true
         sim_isaac:=false
         isaac_joint_commands:=/isaac_joint_commands
         isaac_joint_states:=/isaac_joint_states
-        use_fake_hardware:=false
+        use_fake_hardware:=true
         fake_sensor_commands:=false
         com_port:=/dev/ttyUSB_gripper">

File: icclab_summit_xl/urdf/robotiq_gripper/robotiq_2f_140_macro.urdf.xacro (robot description, xacro)
@@ -7,10 +7,10 @@
         parent
         *origin
-        sim_ignition:=false
+        sim_ignition:=true
         sim_isaac:=false
         isaac_joint_commands:=/isaac_joint_commands
         isaac_joint_states:=/isaac_joint_states
-        use_fake_hardware:=false
-        fake_sensor_commands:=false
+        use_fake_hardware:=true
+        fake_sensor_commands:=true
         include_ros2_control:=true
         com_port:=/dev/ttyUSB_gripper">

File: icclab_summit_xl/urdf/sensors/hokuyo_utm30lx_no_frame_prefix.urdf.xacro (robot description, xacro)
@@ -39,15 +39,16 @@
 			<xacro:if value="${gpu}">
         <xacro:property name="ray_type" value="gpu_ray" />
-        <xacro:property name="plugin_lib" value="libgazebo_ros_gpu_laser.so" />
+        <xacro:property name="plugin_lib" value="libignition-gazebo-sensors-system.so" />
       </xacro:if>
       <xacro:unless value="${gpu}">
         <xacro:property name="ray_type" value="ray" />
-        <xacro:property name="plugin_lib" value="libgazebo_ros_ray_sensor.so" />
+        <xacro:property name="plugin_lib" value="libignition-gazebo-sensors-system.so" />
       </xacro:unless>
-			<sensor type="${ray_type}" name="${prefix}_sensor">
+			<sensor type="gpu_lidar" name="${prefix}_sensor">
 				<pose>0 0 0 0 0 0</pose>
-				<visualize>false</visualize>
-				<update_rate>30</update_rate>
-				<ray>
+        <topic>${ns}/${prefix}/scan</topic>
+				<update_rate>5</update_rate>
+				<lidar>
+        <!-- <ray> -->
 					<scan>
 						<horizontal>
@@ -68,13 +69,17 @@
 						<stddev>0.01</stddev>
 					</noise>
-				</ray>
-				<plugin name="${prefix}" filename="${plugin_lib}">
-          <ros>
+        <!-- </ray> -->
+				</lidar>
+        <always_on>true</always_on>
+        <visualize>true</visualize>
+				<!-- <plugin name="${prefix}" filename="${plugin_lib}"> -->
+          <!-- <ros>
             <namespace>${ns}</namespace>
             <remapping>~/out:=~/scan</remapping>
           </ros>
-          <output_type>sensor_msgs/LaserScan</output_type>
-					<frame_name>${prefix}_link</frame_name>
-				</plugin>
+          <output_type>sensor_msgs/LaserScan</output_type> -->
+					<gz_frame_id>${prefix}_link</gz_frame_id>
+          <render_engine>ogre2</render_engine>
+			  <!-- </plugin> -->
 			</sensor>
 		</gazebo>

Commit message: Fixed controllers startup on real robot for arm and gripper

File: icclab_summit_xl/robots/summit_xls_icclab.urdf.xacro (robot description, xacro)
@@ -122,5 +122,7 @@
    <!-- Gazebo ros control plugins -->
   <xacro:arg name="config_controllers" default=""/>
-  <xacro:include filename="$(find summit_xl_description)/urdf/ros2_control.urdf.xacro"/>
-  <xacro:ros2_control/>
+  <xacro:if value="$(arg use_fake_hardware)">
+    <xacro:include filename="$(find summit_xl_description)/urdf/ros2_control.urdf.xacro"/>
+    <xacro:ros2_control/>
+  </xacro:if>
 </robot>

File: icclab_summit_xl/urdf/arm/ur.urdf.xacro (robot description, xacro)
@@ -29,5 +29,7 @@
     </xacro:if>
     <xacro:unless value="${simulation}">
-      <xacro:property name="robot_ip" default="192.168.0.210" />
+	<xacro:property name="robot_ip" default="192.168.0.210" />
+        <xacro:property name="sim_gazebo" default="false" />
+	<xacro:property name="sim_ignition" default="false" />
     </xacro:unless>
     <!-- import ur macro -->
@@ -48,4 +50,7 @@
       headless_mode="${headless_mode}"
       robot_ip="${robot_ip}"
+      script_filename="/opt/ros/humble/share/ur_client_library/resources/external_control.urscript"
+      output_recipe_filename="/opt/ros/humble/share/ur_robot_driver/resources/rtde_output_recipe.txt"
+      input_recipe_filename="/opt/ros/humble/share/ur_robot_driver/resources/rtde_input_recipe.txt"
     >
       <xacro:insert_block name="origin" />  <!-- position robot in the world -->

Commit message: nav2 working now

File: icclab_summit_xl/robots/summit_xls_icclab.urdf.xacro (robot description, xacro)
@@ -54,4 +54,5 @@
 	<xacro:arg name="use_fake_hardware" default="true"/>
 	<xacro:arg name="ros_planar_move_plugin" default="true"/>
+	<!-- <xacro:arg name="ros_planar_move_plugin" default="false"/> -->
 	<xacro:arg name="gpu" default="false"/>
 	<xacro:arg name="robot_id" default="summit"/>
@@ -76,4 +77,16 @@
 			<origin xyz="-${wheel_offset_x} -${wheel_offset_y} ${wheel_offset_z}" rpy="0 0 0"/>
 		</xacro:omni_wheel>
+            <!-- <xacro:rubber_wheel prefix="$(arg prefix)front_right" parent="$(arg prefix)base_link" reflect="false" hq="${hq}">
+                <origin xyz="${wheel_offset_x} -${wheel_offset_y} ${wheel_offset_z}" rpy="0 0 0"/>
+            </xacro:rubber_wheel>
+            <xacro:rubber_wheel prefix="$(arg prefix)front_left" parent="$(arg prefix)base_link" reflect="true" hq="${hq}">
+                <origin xyz="${wheel_offset_x} ${wheel_offset_y} ${wheel_offset_z}" rpy="0 0 0"/>
+            </xacro:rubber_wheel>
+            <xacro:rubber_wheel prefix="$(arg prefix)rear_left" parent="$(arg prefix)base_link" reflect="true" hq="${hq}">
+                <origin xyz="-${wheel_offset_x} ${wheel_offset_y} ${wheel_offset_z}" rpy="0 0 0"/>
+            </xacro:rubber_wheel>
+            <xacro:rubber_wheel prefix="$(arg prefix)rear_right" parent="$(arg prefix)base_link" reflect="false" hq="${hq}">
+                <origin xyz="-${wheel_offset_x} -${wheel_offset_y} ${wheel_offset_z}" rpy="0 0 0"/>
+            </xacro:rubber_wheel> -->
         <!-- IMU -->
 		<xacro:sensor_imu_hector prefix="$(arg prefix)imu" ns="$(arg robot_ns)" parent="$(arg prefix)base_link">
@@ -113,10 +126,16 @@
 		<!-- had to copy and modidy camera to avoid name clash with robotnik defined sensors -->
 		<xacro:sensor_d435_icclab prefix="arm_camera" ns="$(arg robot_ns)" parent="arm_camera_mount_link">
-     		  <origin xyz="0.0 0.06 0.01" rpy="${PI} ${-PI/2} ${PI/2}"/> <!-- camera on gripper -->
+     		  <origin xyz="0.0 0.06 0.01" rpy="${PI} ${-PI/2} ${PI/2}"/>
+			  camera on gripper
    		</xacro:sensor_d435_icclab>
    </xacro:macro>
    <xacro:if value="$(arg ros_planar_move_plugin)">
-	   <xacro:omni_steering prefix="$(arg prefix)" publish_tf="true"/>
+	   <xacro:omni_steering prefix="$(arg prefix)" ns="$(arg robot_ns)"/>
+	   	<!-- <xacro:joint_state_publisher prefix="$(arg prefix)"/> -->
    </xacro:if>
+    <xacro:unless value="$(arg ros_planar_move_plugin)">
+	   <xacro:skid_steering prefix="$(arg prefix)" ns="$(arg robot_ns)"/>
+	    <!-- <xacro:joint_state_publisher prefix="$(arg prefix)"/> -->
+   </xacro:unless>
    <xacro:summit_xl prefix="$(arg prefix)" publish_bf="true" hq="true"/>
    <!-- Gazebo ros control plugins -->

Commit message: added luxonis camera in GZ IGN but orientation is wrong

File: icclab_summit_xl/robots/summit_xls_icclab.urdf.xacro (robot description, xacro)
@@ -19,4 +19,6 @@
 	<xacro:include filename="$(find icclab_summit_xl)/urdf/sensors/intel_d435.urdf.xacro" />
 	<xacro:include filename="$(find icclab_summit_xl)/urdf/sensors/intel_camera_mount.urdf.xacro" />
+	<xacro:include filename="$(find icclab_summit_xl)/urdf/sensors/luxonis_oak_d_pro.urdf.xacro" />
+	<xacro:include filename="$(find icclab_summit_xl)/urdf/sensors/luxonis_camera_mount.urdf.xacro" />
 	<!-- Import arm macros -->
 	<xacro:include filename="$(find icclab_summit_xl)/urdf/arm/ur.urdf.xacro"/>
@@ -121,13 +123,21 @@
     	</xacro:robotiq_gripper>
 		<!-- Camera mount -->
-		<xacro:camera_mount prefix="arm" parent="arm_flange">
-			<origin xyz="0 0 0" rpy="${-PI/2} 0 ${-PI/2}" />
-		</xacro:camera_mount>
+		<!-- <xacro:camera_mount prefix="arm" parent="arm_flange"> -->
+			<!-- <origin xyz="0 0 0" rpy="${-PI/2} 0 ${-PI/2}" /> -->
+		<!-- </xacro:camera_mount> -->
+		<!-- Luxonis Camera mount -->
+		<xacro:luxonis_camera_mount prefix="arm" parent="arm_flange">
+			<origin xyz="0 -0.04 0" rpy="${-PI/2} 0 ${-PI/2}" />
+		</xacro:luxonis_camera_mount>
 		<!-- Camera on gripper  -->
 		<!-- had to copy and modidy camera to avoid name clash with robotnik defined sensors -->
-		<xacro:sensor_d435_icclab prefix="arm_camera" ns="$(arg robot_ns)" parent="arm_camera_mount_link">
-     		  <origin xyz="0.0 0.06 0.01" rpy="${PI} ${-PI/2} ${PI/2}"/>
-			  camera on gripper
-   		</xacro:sensor_d435_icclab>
+		<!-- <xacro:sensor_d435_icclab prefix="arm_camera" ns="$(arg robot_ns)" parent="arm_camera_mount_link"> -->
+     		  <!-- <origin xyz="0.0 0.06 0.01" rpy="${PI} ${-PI/2} ${PI/2}"/>  -->
+			  <!-- camera on gripper -->
+   		<!-- </xacro:sensor_d435_icclab>  -->
+		<!-- Luxonis OAK_D_PRO -->
+		<xacro:luxonis_oak_icclab prefix="arm_camera" ns="$(arg robot_ns)" parent="arm_camera_mount_link">
+			   <origin xyz="-0.05 0.08 0.02" rpy="${PI} ${-PI/2} ${PI/2}"/>
+		</xacro:luxonis_oak_icclab>
    </xacro:macro>
    <xacro:if value="$(arg ros_planar_move_plugin)">

Commit message: added Luxonis camera

File: icclab_summit_xl/robots/summit_xls_icclab.urdf.xacro (robot description, xacro)
@@ -18,4 +18,6 @@
 	<xacro:include filename="$(find icclab_summit_xl)/urdf/sensors/intel_d435.urdf.xacro" />
 	<xacro:include filename="$(find icclab_summit_xl)/urdf/sensors/intel_camera_mount.urdf.xacro" />
+	<xacro:include filename="$(find icclab_summit_xl)/urdf/sensors/luxonis_oak_d_pro.urdf.xacro" />
+	<xacro:include filename="$(find icclab_summit_xl)/urdf/sensors/luxonis_camera_mount.urdf.xacro" />
 	<!-- Import arm macros -->
 	<xacro:include filename="$(find icclab_summit_xl)/urdf/arm/ur.urdf.xacro"/>
@@ -107,12 +109,21 @@
     	</xacro:robotiq_gripper>
 		<!-- Camera mount -->
-		<xacro:camera_mount prefix="arm" parent="arm_flange">
-			<origin xyz="0 0 0" rpy="${-PI/2} 0 ${-PI/2}" />
-		</xacro:camera_mount>
+		<!-- <xacro:camera_mount prefix="arm" parent="arm_flange"> -->
+			<!-- <origin xyz="0 0 0" rpy="${-PI/2} 0 ${-PI/2}" /> -->
+		<!-- </xacro:camera_mount> -->
+		<!-- Luxonis Camera mount -->
+		<xacro:luxonis_camera_mount prefix="arm" parent="arm_flange">
+			<origin xyz="0 -0.04 0" rpy="${-PI/2} 0 ${-PI/2}" />
+		</xacro:luxonis_camera_mount>
 		<!-- Camera on gripper  -->
 		<!-- had to copy and modidy camera to avoid name clash with robotnik defined sensors -->
-		<xacro:sensor_d435_icclab prefix="arm_camera" ns="$(arg robot_ns)" parent="arm_camera_mount_link">
-     		  <origin xyz="0.0 0.06 0.01" rpy="${PI} ${-PI/2} ${PI/2}"/> <!-- camera on gripper -->
-   		</xacro:sensor_d435_icclab>
+		<!-- <xacro:sensor_d435_icclab prefix="arm_camera" ns="$(arg robot_ns)" parent="arm_camera_mount_link"> -->
+     		  <!-- <origin xyz="0.0 0.06 0.01" rpy="${PI} ${-PI/2} ${PI/2}"/>  -->
+			  <!-- camera on gripper -->
+   		<!-- </xacro:sensor_d435_icclab>  -->
+		<!-- Luxonis OAK_D_PRO -->
+		<xacro:luxonis_oak_icclab prefix="arm_camera" ns="$(arg robot_ns)" parent="arm_camera_mount_link">
+			   <origin xyz="-0.05 0.08 0.02" rpy="${PI} ${-PI/2} ${PI/2}"/>
+		</xacro:luxonis_oak_icclab>
    </xacro:macro>
    <xacro:if value="$(arg ros_planar_move_plugin)">

File: icclab_summit_xl/urdf/sensors/orbbec_astra.urdf.xacro (robot description, xacro)
@@ -60,5 +60,5 @@
         <update_rate>15</update_rate>
         <camera>
-          <horizontal_fov>1,04719755</horizontal_fov>
+          <horizontal_fov>1.04719755</horizontal_fov>
           <vertical_fov>0.86393798</vertical_fov>
           <image>
