Commit message: removed dependency from robotnik_sensors, WIP: UR arm still to be fixed

File: icclab_summit_xl/robots/summit_xls_icclab.urdf.xacro (robot description, xacro)
@@ -11,6 +11,4 @@
 	<xacro:include filename="$(find summit_xl_description)/urdf/wheels/rubber_wheel.urdf.xacro" />
 	<xacro:include filename="$(find summit_xl_description)/urdf/structures/structure_hokuyo.urdf.xacro" />
-	<!-- Import all available sensors -->
-	<xacro:include filename="$(find robotnik_sensors)/urdf/all_sensors.urdf.xacro" />
 	<!-- Import our modified sensor -->
 	<xacro:include filename="$(find icclab_summit_xl)/urdf/sensors/hokuyo_utm30lx_no_frame_prefix.urdf.xacro" />
@@ -20,4 +18,5 @@
 	<xacro:include filename="$(find icclab_summit_xl)/urdf/sensors/luxonis_oak_d_pro.urdf.xacro" />
 	<xacro:include filename="$(find icclab_summit_xl)/urdf/sensors/luxonis_camera_mount.urdf.xacro" />
+	<xacro:include filename="$(find icclab_summit_xl)/urdf/sensors/imu_hector_plugin.urdf.xacro"/>
 	<!-- Import arm macros -->
 	<xacro:include filename="$(find icclab_summit_xl)/urdf/arm/ur.urdf.xacro"/>

File: icclab_summit_xl/urdf/sensors/hokuyo_utm30lx_no_frame_prefix.urdf.xacro (robot description, xacro)
@@ -16,5 +16,5 @@
         <origin xyz="0 0 0.055" rpy="0 0 0"/>
         <geometry>
-            <mesh filename="package://robotnik_sensors/meshes/hokuyo_utm_30lx.dae"/>
+            <mesh filename="package://icclab_summit_xl/meshes/hokuyo_utm_30lx.dae"/>
         </geometry>
       </visual>

File: icclab_summit_xl/urdf/sensors/orbbec_astra.urdf.xacro (robot description, xacro)
@@ -11,5 +11,5 @@
         <origin xyz="0 0 0" rpy="0 0 0"/>
         <geometry>
-          <mesh filename="package://robotnik_sensors/meshes/orbbec_astra.dae"/>
+          <mesh filename="package://icclab_summit_xl/meshes/orbbec_astra.dae"/>
         </geometry>
       </visual>

Commit message: WIP porting to Jazzy. Nav2 and slam work with laserscan merger jazzy. Still missing arm and gripper

File: icclab_summit_xl/robots/summit_xls_icclab.urdf.xacro (robot description, xacro)
@@ -6,5 +6,6 @@
 	<!-- First we import all posible elements defined in the urdf.xacro files. All these elements are defined as macro:xacros -->
 	<!-- Import summit XL base elements -->
-	<xacro:include filename="$(find summit_xl_description)/urdf/bases/summit_xl_hls_base.urdf.xacro" />
+	<!-- <xacro:include filename="$(find summit_xl_description)/urdf/bases/summit_xl_hls_base.urdf.xacro" /> -->
+	<xacro:include filename="$(find icclab_summit_xl)/urdf/bases/summit_xl_hls_base.urdf.xacro" />
 	<!-- Import summit XL wheels -->
 	<xacro:include filename="$(find summit_xl_description)/urdf/wheels/omni_wheel.urdf.xacro" />
@@ -55,4 +56,5 @@
 	<xacro:arg name="use_fake_hardware" default="true"/>
 	<xacro:arg name="ros_planar_move_plugin" default="true"/>
+	<!-- <xacro:arg name="ros_planar_move_plugin" default="false"/> -->
 	<xacro:arg name="gpu" default="false"/>
 	<xacro:arg name="robot_id" default="summit"/>
@@ -101,10 +103,10 @@
 		</xacro:sensor_gps-->
 		<!-- Add arm -->
-		<xacro:icclab_summit_arm simulation="$(arg use_fake_hardware)">
+		<!-- <xacro:icclab_summit_arm simulation="$(arg use_fake_hardware)">
 			<origin xyz="0.255 0 0.275" rpy="0 0 ${pi}" />
-		</xacro:icclab_summit_arm>
-		<xacro:robotiq_gripper name="RobotiqGripperHardwareInterface" prefix="" parent="arm_tool0" use_fake_hardware="$(arg use_fake_hardware)">
+		</xacro:icclab_summit_arm> -->
+		<!-- <xacro:robotiq_gripper name="RobotiqGripperHardwareInterface" prefix="" parent="arm_tool0" use_fake_hardware="$(arg use_fake_hardware)">
         	<origin xyz="0 0 0" rpy="0 0 0" />
-    	</xacro:robotiq_gripper>
+    	</xacro:robotiq_gripper> -->
 		<!-- Camera mount -->
 		<!-- <xacro:camera_mount prefix="arm" parent="arm_flange"> -->
@@ -112,7 +114,7 @@
 		<!-- </xacro:camera_mount> -->
 		<!-- Luxonis Camera mount -->
-		<xacro:luxonis_camera_mount prefix="arm" parent="arm_flange">
+		<!-- <xacro:luxonis_camera_mount prefix="arm" parent="arm_flange">
 			<origin xyz="0 -0.04 0" rpy="${-PI/2} 0 ${-PI/2}" />
-		</xacro:luxonis_camera_mount>
+		</xacro:luxonis_camera_mount> -->
 		<!-- Camera on gripper  -->
 		<!-- had to copy and modidy camera to avoid name clash with robotnik defined sensors -->
@@ -122,11 +124,16 @@
    		<!-- </xacro:sensor_d435_icclab>  -->
 		<!-- Luxonis OAK_D_PRO -->
-		<xacro:luxonis_oak_icclab prefix="arm_camera" ns="$(arg robot_ns)" parent="arm_camera_mount_link">
+		<!-- <xacro:luxonis_oak_icclab prefix="arm_camera" ns="$(arg robot_ns)" parent="arm_camera_mount_link">
 			   <origin xyz="-0.05 0.08 0.02" rpy="${PI} ${-PI/2} ${PI/2}"/>
-		</xacro:luxonis_oak_icclab>
+		</xacro:luxonis_oak_icclab>  -->
    </xacro:macro>
    <xacro:if value="$(arg ros_planar_move_plugin)">
-	   <xacro:omni_steering namespace="$(arg robot_ns)" publish_tf="true"/>
+	   <xacro:omni_steering prefix="$(arg prefix)" ns="$(arg robot_ns)"/>
+	   	<!-- <xacro:joint_state_publisher prefix="$(arg prefix)"/> -->
    </xacro:if>
+    <xacro:unless value="$(arg ros_planar_move_plugin)">
+	   <xacro:skid_steering prefix="$(arg prefix)" ns="$(arg robot_ns)"/>
+	    <!-- <xacro:joint_state_publisher prefix="$(arg prefix)"/> -->
+   </xacro:unless>
    <xacro:summit_xl prefix="$(arg prefix)" publish_bf="true" hq="true"/>
    <!-- Gazebo ros control plugins -->

File: icclab_summit_xl/urdf/sensors/hokuyo_utm30lx_no_frame_prefix.urdf.xacro (robot description, xacro)
@@ -39,15 +39,16 @@
 			<xacro:if value="${gpu}">
         <xacro:property name="ray_type" value="gpu_ray" />
-        <xacro:property name="plugin_lib" value="libgazebo_ros_gpu_laser.so" />
+        <xacro:property name="plugin_lib" value="libignition-gazebo-sensors-system.so" />
       </xacro:if>
       <xacro:unless value="${gpu}">
         <xacro:property name="ray_type" value="ray" />
-        <xacro:property name="plugin_lib" value="libgazebo_ros_ray_sensor.so" />
+        <xacro:property name="plugin_lib" value="libignition-gazebo-sensors-system.so" />
       </xacro:unless>
-			<sensor type="${ray_type}" name="${prefix}_sensor">
+			<sensor type="gpu_lidar" name="${prefix}_sensor">
 				<pose>0 0 0 0 0 0</pose>
+				<topic>${ns}/${prefix}/scan</topic>
 				<visualize>false</visualize>
 				<update_rate>30</update_rate>
-				<ray>
+				<lidar>
 					<scan>
 						<horizontal>
@@ -68,13 +69,17 @@
 						<stddev>0.01</stddev>
 					</noise>
-				</ray>
-				<plugin name="${prefix}" filename="${plugin_lib}">
-          <ros>
+        <!-- </ray> -->
+				</lidar>
+        <always_on>true</always_on>
+        <visualize>true</visualize>
+				<!-- <plugin name="${prefix}" filename="${plugin_lib}"> -->
+          <!-- <ros>
             <namespace>${ns}</namespace>
             <remapping>~/out:=~/scan</remapping>
           </ros>
-          <output_type>sensor_msgs/LaserScan</output_type>
-					<frame_name>${prefix}_link</frame_name>
-				</plugin>
+          <output_type>sensor_msgs/LaserScan</output_type> -->
+					<gz_frame_id>${prefix}_link</gz_frame_id>
+          <render_engine>ogre2</render_engine>
+			  <!-- </plugin> -->
 			</sensor>
 		</gazebo>

File: icclab_summit_xl/urdf/sensors/luxonis_camera_gazebo.urdf.xacro (robot description, xacro)
@@ -1,12 +1,15 @@
 <?xml version="1.0"?>
 <robot name="luxonis_camera_gazebo" xmlns:xacro="http://wiki.ros.org/Sensors/OrbbecAstra">
-  <xacro:property name="deg_to_rad" value="0.01745329251994329577"/>
   <xacro:macro name="luxonis_camera_gazebo" params="ns prefix frame">
+    <xacro:property name="M_PI" value="3.1415926535897931" />
     <gazebo reference="${prefix}_link">
-      <sensor name="${prefix}" type="depth">
-        <pose>0 0 0 0 0 0</pose>
-        <!-- <visualize>true</visualize> -->
+      <sensor name="${prefix}" type="camera">
+        <pose>0 0 0 0 -1.5707963267948966 -1.5707963267948966</pose>
+        <visualize>true</visualize>
+        <always_on>true</always_on>
         <update_rate>15</update_rate>
-        <camera>
+        <!-- <camera name="orbbec"> -->
+        <camera name="${prefix}">
+          <camera_info_topic>${ns}/${prefix}/color/camera_info</camera_info_topic>
           <horizontal_fov>1.04719755</horizontal_fov>
           <vertical_fov>0.86393798</vertical_fov>
@@ -22,5 +25,5 @@
         </camera>
         <!-- plugin https://docs.ros.org/en/ros2_packages/rolling/api/gazebo_plugins/generated/classgazebo__plugins_1_1GazeboRosCamera.html -->
-        <plugin name="${prefix}" filename="libgazebo_ros_camera.so">
+        <!-- <plugin name="${prefix}" filename="libignition-gazebo-sensors-system.so"> -->
           <ros>
             <namespace>${ns}</namespace>
@@ -31,9 +34,10 @@
             <remapping>~/image_raw/theora:=~/color/image_raw/theora</remapping>
           </ros>
-          <camera_name>${prefix}</camera_name>
-          <frame_name>${frame}</frame_name>
+          <!-- <camera name="${prefix}"/> -->
+          <gz_frame_id>${frame}</gz_frame_id>
           <min_depth>0.05</min_depth>
           <max_depth>20.0</max_depth>
-        </plugin>
+        <!-- </plugin>  -->
+        <topic>${ns}/${prefix}/color/image_raw</topic>
       </sensor>
     </gazebo>

File: icclab_summit_xl/urdf/sensors/luxonis_oak_d_pro.urdf.xacro (robot description, xacro)
@@ -7,6 +7,5 @@
 	  <xacro:insert_block name="origin" />
 	</xacro:luxonis>
-	<!-- <xacro:luxonis_camera_gazebo ns="${ns}" prefix="${prefix}" frame="${prefix}_color_optical_frame"/> -->
-	<xacro:luxonis_camera_gazebo ns="${ns}" prefix="${prefix}" frame="oak_rgb_camera_optical_frame"/>
+	<xacro:luxonis_camera_gazebo ns="${ns}" prefix="${prefix}" frame="${prefix}_color_optical_frame"/>
 </xacro:macro>
 </robot>

File: icclab_summit_xl/urdf/sensors/luxonis_oak_d_pro_model.urdf.xacro (robot description, xacro)
@@ -19,15 +19,15 @@
     <!-- <link name="oak_model_origin"> -->
     <link name="arm_camera_link">
-		<visual>
-			<origin xyz="0 0 0" rpy="${M_PI/2} 0 ${M_PI/2}" />
-			<geometry>
-				<mesh filename="file://$(find icclab_summit_xl)/meshes/sensors/OAK-D-PRO.stl" />
-			</geometry>
-			<material name="mat">
-				<color rgba="0.8 0.8 0.8 0.8" />
-			</material>
-		</visual>
+				<visual>
+					<origin xyz="0 0 0" rpy="0 0 0" />
+					<geometry>
+						<mesh filename="file://$(find icclab_summit_xl)/meshes/sensors/OAK-D-PRO.stl" />
+					</geometry>
+					<material name="mat">
+						<color rgba="0.8 0.8 0.8 0.8" />
+					</material>
+				</visual>
         <collision>
-          <origin xyz="0 0 0" rpy="${M_PI/2} 0 ${M_PI/2}" />
+          <origin xyz="0 0 0" rpy="0 0 0"/>
           <geometry>
             <box size="0.097 0.0295 0.0229"/>
@@ -37,5 +37,5 @@
           <mass value="0.072" />
           <!-- <mass value="0.091" /> -->
-		  <origin xyz="0 0 0" rpy="0 0 0" />
+          <origin xyz="0 0 0" />
           <inertia ixx="0.003881243" ixy="0.0" ixz="0.0" iyy="0.000498940" iyz="0.0" izz="0.003879257" />
           <!-- <inertia ixx="0.000010576" ixy="0.0" ixz="0.0" iyy="0.000075328" iyz="0.0" izz="0.000077951" /> -->
@@ -45,7 +45,6 @@
 			<parent link="oak-d_frame" />
 			<!-- <child link="oak_model_origin" /> -->
-      		<child link="arm_camera_link" />
-			<!-- <origin xyz="0 0 0" rpy="1.5708 0 1.5708" /> -->
-			<origin xyz="0 0 0" rpy="0.0 0.0 0.0" />
+      <child link="arm_camera_link" />
+			<origin xyz="0 0 0" rpy="1.5708 0 1.5708" />
 		</joint>
     <link name="oak_imu_frame" />
@@ -62,11 +61,11 @@
 		  	<origin xyz="0 0 0" rpy="0 0 0" />
 		</joint>
-		<link name="oak_rgb_camera_optical_frame" />
-    <!-- <link name="arm_camera_color_optical_frame" /> -->
+		<!-- <link name="oak_rgb_camera_optical_frame" /> -->
+    <link name="arm_camera_color_optical_frame" />
 		<joint name="oak_rgb_camera_optical_joint" type="fixed">
 				<origin xyz="0 0 0" rpy="-${M_PI/2} 0.0 -${M_PI/2}" />
 				<parent link="oak_rgb_camera_frame" />
-				<child link="oak_rgb_camera_optical_frame" />
-        		<!-- <child link="arm_camera_color_optical_frame" /> -->
+				<!-- <child link="oak_rgb_camera_optical_frame" /> -->
+        <child link="arm_camera_color_optical_frame" />
 		</joint>
     <!-- Left Camera -->
@@ -98,6 +97,5 @@
     <joint name="arm_camera_usb_plug_joint" type="fixed">
       <!-- <origin xyz="0.0 -0.05 0" rpy="0 0 0"/> -->
-      <!-- <origin xyz="0.0 0.01 -0.01" rpy="0 ${M_PI/2} ${M_PI}"/> -->
-	  <origin xyz="-0.01 0.01 0.0" rpy="${M_PI/2} ${M_PI} 0.0"/>
+      <origin xyz="0.0 0.01 -0.01" rpy="0 ${M_PI/2} ${M_PI}"/>
       <parent link="arm_camera_link" />
       <child link="arm_camera_usb_plug_link" />

File: icclab_summit_xl/urdf/sensors/orbbec_astra.urdf.xacro (robot description, xacro)
@@ -55,9 +55,12 @@
     <xacro:property name="deg_to_rad" value="0.01745329251994329577"/>
     <gazebo reference="${prefix}_link">
-      <sensor name="${prefix}" type="depth">
+      <sensor name="${prefix}" type="camera">
         <pose>0 0 0 0 0 0</pose>
         <visualize>true</visualize>
+        <always_on>true</always_on>
         <update_rate>15</update_rate>
-        <camera>
+        <!-- <camera name="orbbec"> -->
+        <camera name="${prefix}">
+          <camera_info_topic>${ns}/${prefix}/color/camera_info</camera_info_topic>
           <horizontal_fov>1.04719755</horizontal_fov>
           <vertical_fov>0.86393798</vertical_fov>
@@ -73,5 +76,5 @@
         </camera>
         <!-- plugin https://docs.ros.org/en/ros2_packages/rolling/api/gazebo_plugins/generated/classgazebo__plugins_1_1GazeboRosCamera.html -->
-        <plugin name="${prefix}" filename="libgazebo_ros_camera.so">
+        <!-- <plugin name="${prefix}" filename="libignition-gazebo-sensors-system.so"> -->
           <ros>
             <namespace>${ns}</namespace>
@@ -82,9 +85,10 @@
             <remapping>~/image_raw/theora:=~/color/image_raw/theora</remapping>
           </ros>
-          <camera_name>${prefix}</camera_name>
-          <frame_name>${frame}</frame_name>
+          <!-- <camera name="${prefix}"/> -->
+          <gz_frame_id>${frame}</gz_frame_id>
           <min_depth>0.05</min_depth>
           <max_depth>20.0</max_depth>
-        </plugin>
+        <!-- </plugin>  -->
+        <topic>${ns}/${prefix}/color/image_raw</topic>
       </sensor>
     </gazebo>

Commit message: WIP: jazzy porting. Added arm and controllers

File: icclab_summit_xl/robots/summit_xls_icclab.urdf.xacro (robot description, xacro)
@@ -138,8 +138,19 @@
    <xacro:summit_xl prefix="$(arg prefix)" publish_bf="true" hq="true"/>
    <!-- Gazebo ros control plugins -->
-  <xacro:arg name="config_controllers" default=""/>
+   <xacro:arg name="config_controllers" default=""/>
+   <gazebo reference="$(arg robot_id)"></gazebo>
+   <gazebo>
+		<plugin filename="gz_ros2_control-system" name="gz_ros2_control::GazeboSimROS2ControlPlugin">
+			<parameters>$(arg config_controllers)</parameters>
+			<ros>
+			<namespace>$(arg robot_id)</namespace>
+			<remapping>/robot_description:=robot_description</remapping>
+			</ros>
+		</plugin>
+   </gazebo>
+  <!-- <xacro:arg name="config_controllers" default=""/>
   <xacro:if value="$(arg use_fake_hardware)">
     <xacro:include filename="$(find summit_xl_description)/urdf/ros2_control.urdf.xacro"/>
     <xacro:ros2_control/>
-  </xacro:if>
+  </xacro:if> -->
 </robot>

File: icclab_summit_xl/urdf/arm/ur.urdf.xacro (robot description, xacro)
@@ -35,7 +35,6 @@
     <!-- import ur macros -->
     <xacro:include filename="$(find ur_description)/urdf/ur_macro.xacro" />
-    <xacro:include filename="$(find ur_description)/urdf/ros2_control_mock_hardware.xacro" />
+    <xacro:include filename="$(find ur_simulation_gz)/urdf/ur_gz.ros2_control.xacro" />
     <!-- call the actual ur macro -->
-    <!-- NOTE: we pass use_fake_hardware="false" to avoid generation of unneeded ros2 control plugins, i.e., mock_components/GenericSystem -->
     <xacro:ur_robot
      name="${name}"
@@ -52,32 +51,5 @@
       name="${name}"
       tf_prefix="${tf_prefix}"
-      mock_sensor_commands="false"
     />
-    <!-- Commented: we use a single controller manager and it's included by the robot base-->
-    <!-- <xacro:if value="$(arg sim_gazebo)">
-    <gazebo reference="$(arg tf_prefix)base_link">
-    </gazebo>
-    <gazebo>
-      <plugin filename="libgazebo_ros2_control.so" name="gazebo_ros2_control_arm">
-        <namespace>$(arg robot_id)</namespace>
-        <parameters>$(arg simulation_controllers)</parameters>
-      </plugin>
-    </gazebo>
-  </xacro:if> -->
-    <!-- TODO: FIXME for Ignition
-  <xacro:if value="${sim_ignition}">
-    <gazebo reference="$(arg tf_prefix)base_link">
-    </gazebo>
-    <gazebo>
-      <plugin filename="libign_ros2_control-system.so"
-    name="ign_ros2_control::IgnitionROS2ControlPlugin">
-        <parameters>$(arg simulation_controllers)</parameters>
-        <controller_manager_node_name>$(arg tf_prefix)controller_manager</controller_manager_node_name>
-      </plugin>
-    </gazebo>
-  </xacro:if> -->
   </xacro:macro>
-  <!-- <xacro:icclab_summit_arm simulation="true">
-			<origin xyz="0.255 0 0.275" rpy="0 0 ${pi}" />
-	</xacro:icclab_summit_arm> -->
 </robot>

Commit message: WIP Jazzy porting. Arm motion planning and execution now work

File: icclab_summit_xl/robots/summit_xls_icclab.urdf.xacro (robot description, xacro)
@@ -128,12 +128,4 @@
 		</xacro:luxonis_oak_icclab>  -->
    </xacro:macro>
-   <xacro:if value="$(arg ros_planar_move_plugin)">
-	   <xacro:omni_steering prefix="$(arg prefix)" ns="$(arg robot_ns)"/>
-	   	<!-- <xacro:joint_state_publisher prefix="$(arg prefix)"/> -->
-   </xacro:if>
-    <xacro:unless value="$(arg ros_planar_move_plugin)">
-	   <xacro:skid_steering prefix="$(arg prefix)" ns="$(arg robot_ns)"/>
-	    <!-- <xacro:joint_state_publisher prefix="$(arg prefix)"/> -->
-   </xacro:unless>
    <xacro:summit_xl prefix="$(arg prefix)" publish_bf="true" hq="true"/>
    <!-- Gazebo ros control plugins -->
@@ -149,4 +141,12 @@
 		</plugin>
    </gazebo>
+	<xacro:if value="$(arg ros_planar_move_plugin)">
+	   <xacro:omni_steering prefix="$(arg prefix)" ns="$(arg robot_ns)"/>
+	   	<!-- <xacro:joint_state_publisher prefix="$(arg prefix)"/> -->
+   </xacro:if>
+    <xacro:unless value="$(arg ros_planar_move_plugin)">
+	   <xacro:skid_steering prefix="$(arg prefix)" ns="$(arg robot_ns)"/>
+   </xacro:unless>
+   <xacro:joint_state_publisher prefix="$(arg robot_id)"/>
   <!-- Macro for robot wheels. TODO: For gz ign is now managed by gz, we might want to FIX this  -->
   <!-- <xacro:if value="$(arg use_fake_hardware)">

File: icclab_summit_xl/urdf/bases/summit_xl_base.gazebo.xacro (robot description, xacro)
@@ -12,21 +12,21 @@
     </gazebo>
 	</xacro:macro> -->
-	<!-- <xacro:macro name="joint_state_publisher" params="prefix"> -->
-    <!-- <gazebo> -->
-		<!-- <plugin filename="ignition-gazebo-joint-state-publisher-system" -->
-		<!-- name="ignition::gazebo::systems::JointStatePublisher"> -->
-		<!-- <topic>${prefix}joint_states</topic> -->
-		<!-- <update_rate>30</update_rate> -->
-		<!-- <joint_name>${prefix}front_left_wheel_joint</joint_name> -->
-		<!-- <joint_name>${prefix}front_right_wheel_joint</joint_name> -->
-		<!-- <joint_name>${prefix}rear_left_wheel_joint</joint_name> -->
-		<!-- <joint_name>${prefix}rear_right_wheel_joint</joint_name> -->
-		<!-- </plugin>     -->
-	<!-- </gazebo> -->
-  	<!-- </xacro:macro> -->
+	<xacro:macro name="joint_state_publisher" params="prefix">
+    <gazebo>
+		<plugin filename="gz-sim-joint-state-publisher-system"
+		name="gz::sim::systems::JointStatePublisher">
+		<topic>${prefix}/joint_states</topic>
+		<update_rate>30</update_rate>
+		<joint_name>front_left_wheel_joint</joint_name>
+		<joint_name>front_right_wheel_joint</joint_name>
+		<joint_name>rear_left_wheel_joint</joint_name>
+		<joint_name>rear_right_wheel_joint</joint_name>
+		</plugin>
+	 </gazebo>
+  	 </xacro:macro>
 	<!-- skid steering plugin -->
 	<xacro:macro name="skid_steering" params="ns prefix">
     <gazebo>
-	  <plugin filename="libignition-gazebo-diff-drive-system.so" name="ignition::gazebo::systems::DiffDrive">
+	  <plugin filename="libgz-diff-drive-system.so" name="gz::sim::systems::DiffDrive">
 		    <odom_publish_frequency>50</odom_publish_frequency>
 		    <left_joint>${prefix}front_left_wheel_joint</left_joint>
@@ -47,5 +47,5 @@
   <xacro:macro name="omni_steering" params="ns prefix">
 		<gazebo>
-		<!-- <plugin filename="ignition-gazebo-mecanum-drive-system" name="ignition::gazebo::systems::MecanumDrive"> -->
+		<!-- <plugin filename="gz-sim-mecanum-drive-system" name="gz::sim::systems::MecanumDrive"> -->
 			<!-- <odom_publish_frequency>50.0</odom_publish_frequency> -->
 			<!-- <front_left_joint>${prefix}front_left_wheel_joint</front_left_joint> -->
@@ -64,10 +64,10 @@
       <!-- </plugin> -->
 	    <plugin
-        filename="ignition-gazebo-velocity-control-system"
-        name="ignition::gazebo::systems::VelocityControl">
+        filename="gz-sim-velocity-control-system"
+        name="gz::sim::systems::VelocityControl">
       	</plugin>
 		<plugin
-        filename="ignition-gazebo-odometry-publisher-system"
-        name="ignition::gazebo::systems::OdometryPublisher">
+        filename="gz-sim-odometry-publisher-system"
+        name="gz::sim::systems::OdometryPublisher">
 		<odom_frame>${prefix}odom</odom_frame>
 		<robot_base_frame>${prefix}base_footprint</robot_base_frame>

Commit message: disabled collisions with the back of the robot

File: icclab_summit_xl/robots/summit_xls_icclab.urdf.xacro (robot description, xacro)
@@ -20,4 +20,5 @@
 	<xacro:include filename="$(find icclab_summit_xl)/urdf/sensors/luxonis_oak_d_pro.urdf.xacro" />
 	<xacro:include filename="$(find icclab_summit_xl)/urdf/sensors/luxonis_camera_mount.urdf.xacro" />
+	<xacro:include filename="$(find icclab_summit_xl)/urdf/sensors/back_box.urdf.xacro" />
 	<!-- Import arm macros -->
 	<xacro:include filename="$(find icclab_summit_xl)/urdf/arm/ur.urdf.xacro"/>
@@ -126,4 +127,8 @@
 			   <origin xyz="-0.05 0.08 0.02" rpy="${PI} ${-PI/2} ${PI/2}"/>
 		</xacro:luxonis_oak_icclab>
+		<!-- Back Box -->
+		<xacro:back_box prefix="$(arg prefix)" parent="$(arg prefix)base_link">
+			<origin xyz="-0.08 0 0.4" rpy="0 0 0" />
+		</xacro:back_box>
    </xacro:macro>
    <xacro:if value="$(arg ros_planar_move_plugin)">
