Commit message: updated back box

File: icclab_summit_xl/robots/summit_xls_icclab.urdf.xacro (robot description, xacro)
@@ -20,5 +20,5 @@
 	<xacro:include filename="$(find icclab_summit_xl)/urdf/sensors/luxonis_oak_d_pro.urdf.xacro" />
 	<xacro:include filename="$(find icclab_summit_xl)/urdf/sensors/luxonis_camera_mount.urdf.xacro" />
-	<!-- <xacro:include filename="$(find icclab_summit_xl)/urdf/sensors/back_box.urdf.xacro" /> -->
+	<xacro:include filename="$(find icclab_summit_xl)/urdf/sensors/back_box.urdf.xacro" />
 	<!-- Import arm macros -->
 	<xacro:include filename="$(find icclab_summit_xl)/urdf/arm/ur.urdf.xacro"/>
@@ -128,7 +128,7 @@
 		</xacro:luxonis_oak_icclab>
 		<!-- Back Box -->
-		<!-- <xacro:back_box prefix="$(arg prefix)" parent="$(arg prefix)base_link">
-			<origin xyz="-0.08 0 0.4" rpy="0 0 0" />
-		</xacro:back_box> -->
+		<xacro:back_box prefix="$(arg prefix)" parent="$(arg prefix)base_link">
+			<origin xyz="-0.2 0 0.4" rpy="0 0 0" />
+		</xacro:back_box>
    </xacro:macro>
    <xacro:if value="$(arg ros_planar_move_plugin)">

File: icclab_summit_xl/urdf/sensors/back_box.urdf.xacro (robot description, xacro)
@@ -11,15 +11,15 @@
     </material>
     <link name="back_box_link">
-      <!-- <visual>
+      <visual>
       <origin xyz="0 0 0" rpy="0 0 0"/>
         <geometry>
-          <box size="0.45 0.4 0.2" />
+          <box size="0.25 0.4 0.20" />
         </geometry>
         <material name="black"/>
-      </visual> -->
+      </visual>
       <collision>
         <origin xyz="0.0 0.0 0.0" rpy="0 0 0"/>
         <geometry>
-          <box size="0.45 0.4 0.2" />
+          <box size="0.25 0.4 0.20" />
         </geometry>
       </collision>

Commit message: Fixed unaligned image and pointcloud using depth_camera https://github.com/gazebosim/gz-sensors/issues/545

File: icclab_summit_xl/robots/summit_xls_icclab.urdf.xacro (robot description, xacro)
@@ -123,6 +123,6 @@
    		<!-- </xacro:sensor_d435_icclab>  -->
 		<!-- Luxonis OAK_D_PRO -->
-		<xacro:luxonis_oak_icclab prefix="arm_camera" ns="$(arg robot_ns)" parent="arm_camera_mount_link">
-			   <origin xyz="-0.05 0.08 0.02" rpy="${PI} ${-PI/2} ${PI/2}"/>
+		<xacro:luxonis_oak_icclab prefix="arm_camera" ns="$(arg robot_ns)" parent="arm_flange">
+			   <origin xyz="0.027 0 -0.08" rpy="0 0 0"/>
 		</xacro:luxonis_oak_icclab>
    </xacro:macro>

File: icclab_summit_xl/urdf/sensors/luxonis_camera_gazebo.urdf.xacro (robot description, xacro)
@@ -3,7 +3,8 @@
   <xacro:macro name="luxonis_camera_gazebo" params="ns prefix frame">
     <xacro:property name="M_PI" value="3.1415926535897931" />
-    <gazebo reference="${prefix}_link">
+    <gazebo reference="${frame}">
       <sensor name="${prefix}" type="rgbd_camera">
-        <pose>0 0 0 0 -1.5707963267948966 -1.5707963267948966</pose>
+        <gz_frame_id>${frame}</gz_frame_id>
+        <!-- <pose>0 0 0 0 -1.5707963267948966 -1.5707963267948966</pose> -->
         <visualize>true</visualize>
         <always_on>true</always_on>
@@ -11,5 +12,5 @@
         <!-- <camera name="orbbec"> -->
         <camera name="${prefix}">
-          <optical_frame_id>${prefix}_color_optical_frame</optical_frame_id>
+          <!-- <optical_frame_id>${prefix}_color_optical_frame</optical_frame_id> -->
           <!-- <camera_info_topic>${ns}/${prefix}/color/camera_info</camera_info_topic> -->
           <horizontal_fov>1.04719755</horizontal_fov>
@@ -25,11 +26,6 @@
           </clip>
         </camera>
-        <!-- plugin https://docs.ros.org/en/ros2_packages/rolling/api/gazebo_plugins/generated/classgazebo__plugins_1_1GazeboRosCamera.html -->
-        <!-- <plugin name="${prefix}" filename="libignition-gazebo-sensors-system.so"> -->
-          <!-- <camera name="${prefix}"/> -->
-          <gz_frame_id>${frame}</gz_frame_id>
           <min_depth>0.05</min_depth>
           <max_depth>20.0</max_depth>
-        <!-- </plugin>  -->
         <topic>${ns}/${prefix}</topic>
       </sensor>

File: icclab_summit_xl/urdf/sensors/luxonis_oak_d_pro.urdf.xacro (robot description, xacro)
@@ -7,5 +7,11 @@
 	  <xacro:insert_block name="origin" />
 	</xacro:luxonis>
-	<xacro:luxonis_camera_gazebo ns="${ns}" prefix="${prefix}" frame="oak-d_frame"/>
+	<link name="oak-d_frame_rotated"/>
+	<joint name="oak-d_frame_rotated_joint" type="fixed">
+	  <origin xyz="0 0 0" rpy="${PI} 0 0" />
+	  <parent link="oak-d_frame"/>
+	  <child link="oak-d_frame_rotated"/>
+	</joint>
+	<xacro:luxonis_camera_gazebo ns="${ns}" prefix="${prefix}" frame="oak-d_frame_rotated"/>
 </xacro:macro>
 </robot>

File: icclab_summit_xl/urdf/sensors/luxonis_oak_d_pro_model.urdf.xacro (robot description, xacro)
@@ -45,5 +45,5 @@
 			<parent link="oak-d_frame" />
 			<!-- <child link="oak_model_origin" /> -->
-      <child link="arm_camera_link" />
+      		<child link="arm_camera_link" />
 			<origin xyz="0 0 0" rpy="1.5708 0 1.5708" />
 		</joint>

File: icclab_summit_xl/urdf/sensors/orbbec_astra.urdf.xacro (robot description, xacro)
@@ -55,6 +55,6 @@
     <xacro:property name="deg_to_rad" value="0.01745329251994329577"/>
     <gazebo reference="${prefix}_link">
-      <sensor name="${prefix}_color" type="rgbd_camera">
-        <pose>0 0 0 0 0 0</pose>
+      <sensor name="${prefix}" type="rgbd_camera">
+        <gz_frame_id>${prefix}_link</gz_frame_id>
         <visualize>true</visualize>
         <always_on>true</always_on>
@@ -62,5 +62,5 @@
         <camera name="${prefix}">
           <!-- <camera_info_topic>${ns}/${prefix}/color/camera_info</camera_info_topic> -->
-          <optical_frame_id>${prefix}_rgb_optical_frame</optical_frame_id>
+          <!-- <optical_frame_id>${prefix}_rgb_optical_frame</optical_frame_id> -->
           <horizontal_fov>1.04719755</horizontal_fov>
           <vertical_fov>0.86393798</vertical_fov>
@@ -75,5 +75,4 @@
           </clip>
         </camera>
-        <gz_frame_id>${frame}</gz_frame_id>
         <min_depth>0.05</min_depth>
         <max_depth>40.0</max_depth>

Commit message: Fix rgbd_camera optical frame: use depth_image_proc for pointcloud
Gazebo Harmonic's rgbd_camera sensor publishes pointcloud XYZ data in
Gazebo convention (X-fwd) but optical_frame_id only relabels the header
without rotating the data (confirmed in gz-sensors source). This causes
misaligned pointclouds for any ROS tool expecting optical frame data
(MoveIt octomaps, AprilTag detection, etc).

Solution: skip bridging Gazebo's broken pointcloud and regenerate it on
the ROS side using depth_image_proc/point_cloud_xyzrgb from depth+color
images, which correctly produces optical-frame pointclouds.

- Add depth_image variant sensor xacros with optical_frame_id for images
- Add bridge config without arm_camera pointcloud topic
- Add depth_image_proc node to launch for arm_camera pointcloud
- Move PI rotation from rotated frame hack into oak_rgb_camera_joint
- Keep Option A files (camera frame) as fallback alternative
- Add depth_image_proc to package.xml exec_depend

Co-Authored-By: Claude Opus 4.6 <noreply@anthropic.com>

File: icclab_summit_xl/robots/summit_xls_icclab.urdf.xacro (robot description, xacro)
@@ -17,5 +17,5 @@
 	<xacro:include filename="$(find icclab_summit_xl)/urdf/sensors/intel_d435.urdf.xacro" />
 	<xacro:include filename="$(find icclab_summit_xl)/urdf/sensors/intel_camera_mount.urdf.xacro" />
-	<xacro:include filename="$(find icclab_summit_xl)/urdf/sensors/luxonis_oak_d_pro.urdf.xacro" />
+	<xacro:include filename="$(find icclab_summit_xl)/urdf/sensors/luxonis_oak_d_pro_depth_image.urdf.xacro" />
 	<xacro:include filename="$(find icclab_summit_xl)/urdf/sensors/luxonis_camera_mount.urdf.xacro" />
 	<xacro:include filename="$(find icclab_summit_xl)/urdf/sensors/imu_hector_plugin.urdf.xacro"/>

File: icclab_summit_xl/urdf/sensors/luxonis_camera_gazebo_depth_image.urdf.xacro (robot description, xacro)
@@ -1,9 +1,9 @@
 <?xml version="1.0"?>
 <robot name="luxonis_camera_gazebo" xmlns:xacro="http://wiki.ros.org/Sensors/OrbbecAstra">
-  <!-- Option A: All data published with camera frame (Gazebo convention: X-fwd, Y-left, Z-up).
-       Pointcloud + images + camera_info all use the camera frame as frame_id.
-       Data is consistent with frame_id. RViz/TF handles transforms to optical frame.
-       Note: ROS tools expecting optical frame data may need config adjustments. -->
-  <xacro:macro name="luxonis_camera_gazebo" params="ns prefix frame">
+  <!-- Option B: Images/depth published with optical_frame_id for correct ROS convention.
+       Pointcloud NOT bridged from Gazebo (it's in wrong convention anyway).
+       Use depth_image_proc/point_cloud_xyzrgb on ROS side to generate a proper
+       optical-frame pointcloud from depth + color + camera_info. -->
+  <xacro:macro name="luxonis_camera_gazebo" params="ns prefix frame optical_frame">
     <xacro:property name="M_PI" value="3.1415926535897931" />
     <gazebo reference="${frame}">
@@ -15,4 +15,5 @@
         <update_rate>15</update_rate>
         <camera name="${prefix}">
+          <optical_frame_id>${optical_frame}</optical_frame_id>
           <horizontal_fov>1.04719755</horizontal_fov>
           <vertical_fov>0.86393798</vertical_fov>

File: icclab_summit_xl/urdf/sensors/luxonis_oak_d_pro_depth_image.urdf.xacro (robot description, xacro)
@@ -1,5 +1,5 @@
 <?xml version="1.0"?>
 <robot xmlns:xacro="http://www.ros.org/wiki/xacro" name="luxonis">
-<xacro:include filename="$(find icclab_summit_xl)/urdf/sensors/luxonis_camera_gazebo.urdf.xacro"/>
+<xacro:include filename="$(find icclab_summit_xl)/urdf/sensors/luxonis_camera_gazebo_depth_image.urdf.xacro"/>
 <xacro:include filename="$(find icclab_summit_xl)/urdf/sensors/luxonis_oak_d_pro_model.urdf.xacro" />
 <xacro:macro name="luxonis_oak_icclab" params="parent *origin prefix:=arm_camera ns:=summit">
@@ -7,5 +7,5 @@
 	  <xacro:insert_block name="origin" />
 	</xacro:luxonis>
-	<xacro:luxonis_camera_gazebo ns="${ns}" prefix="${prefix}" frame="oak_rgb_camera_frame"/>
+	<xacro:luxonis_camera_gazebo ns="${ns}" prefix="${prefix}" frame="oak_rgb_camera_frame" optical_frame="arm_camera_color_optical_frame"/>
 </xacro:macro>
 </robot>

File: icclab_summit_xl/urdf/sensors/luxonis_oak_d_pro_model.urdf.xacro (robot description, xacro)
@@ -19,13 +19,13 @@
     <!-- <link name="oak_model_origin"> -->
     <link name="arm_camera_link">
-				<visual>
-					<origin xyz="0 0 0" rpy="0 0 0" />
-					<geometry>
-						<mesh filename="file://$(find icclab_summit_xl)/meshes/sensors/OAK-D-PRO.stl" />
-					</geometry>
-					<material name="mat">
-						<color rgba="0.8 0.8 0.8 0.8" />
-					</material>
-				</visual>
+		<visual>
+			<origin xyz="0 0 0" rpy="0 0 0" />
+			<geometry>
+				<mesh filename="file://$(find icclab_summit_xl)/meshes/sensors/OAK-D-PRO.stl" />
+			</geometry>
+			<material name="mat">
+				<color rgba="0.8 0.8 0.8 0.8" />
+			</material>
+		</visual>
         <collision>
           <origin xyz="0 0 0" rpy="0 0 0"/>
@@ -46,5 +46,5 @@
 			<!-- <child link="oak_model_origin" /> -->
       		<child link="arm_camera_link" />
-			<origin xyz="0 0 0" rpy="1.5708 0 1.5708" />
+			<origin xyz="0 0 0" rpy="${M_PI/2} 0 ${M_PI/2}" />
 		</joint>
     <link name="oak_imu_frame" />
@@ -59,5 +59,5 @@
 		  	<parent link="oak-d_frame" />
 		  	<child link="oak_rgb_camera_frame" />
-		  	<origin xyz="0 0 0" rpy="0 0 0" />
+		  	<origin xyz="0 0 0" rpy="${M_PI} 0 0" />
 		</joint>
 		<!-- <link name="oak_rgb_camera_optical_frame" /> -->

Commit message: Robot model without summit_xl_common

File: icclab_summit_xl/robots/summit_xls_icclab.urdf.xacro (robot description, xacro)
@@ -6,10 +6,10 @@
 	<!-- First we import all posible elements defined in the urdf.xacro files. All these elements are defined as macro:xacros -->
 	<!-- Import summit XL base elements -->
-	<!-- <xacro:include filename="$(find summit_xl_description)/urdf/bases/summit_xl_hls_base.urdf.xacro" /> -->
+	<!-- <xacro:include filename="$(find icclab_summit_xl)/urdf/bases/summit_xl_hls_base.urdf.xacro" /> -->
 	<xacro:include filename="$(find icclab_summit_xl)/urdf/bases/summit_xl_hls_base.urdf.xacro" />
 	<!-- Import summit XL wheels -->
-	<xacro:include filename="$(find summit_xl_description)/urdf/wheels/omni_wheel.urdf.xacro" />
-	<xacro:include filename="$(find summit_xl_description)/urdf/wheels/rubber_wheel.urdf.xacro" />
-	<xacro:include filename="$(find summit_xl_description)/urdf/structures/structure_hokuyo.urdf.xacro" />
+	<xacro:include filename="$(find icclab_summit_xl)/urdf/wheels/omni_wheel.urdf.xacro" />
+	<xacro:include filename="$(find icclab_summit_xl)/urdf/wheels/rubber_wheel.urdf.xacro" />
+	<xacro:include filename="$(find icclab_summit_xl)/urdf/structures/structure_hokuyo.urdf.xacro" />
 	<!-- Import our modified sensor -->
 	<xacro:include filename="$(find icclab_summit_xl)/urdf/sensors/hokuyo_utm30lx_no_frame_prefix.urdf.xacro" />

File: icclab_summit_xl/urdf/bases/summit_xl_hls_base.urdf.xacro (robot description, xacro)
@@ -1,5 +1,5 @@
 <?xml version="1.0"?>
 <robot name="summit_xl" xmlns:xacro="http://wiki.ros.org/xacro">
-  <!-- <xacro:include filename="$(find summit_xl_description)/urdf/bases/summit_xl_base.gazebo.xacro" /> -->
+  <!-- <xacro:include filename="$(find icclab_summit_xl)/urdf/bases/summit_xl_base.gazebo.xacro" /> -->
   <xacro:include filename="$(find icclab_summit_xl)/urdf/bases/summit_xl_base.gazebo.xacro" />
   <xacro:macro name="summit_xl_hls_base" params="prefix publish_bf hq">
@@ -35,10 +35,10 @@
        <xacro:if value="${hq}">
        <geometry>
-	     <mesh filename="file://$(find summit_xl_description)/meshes/bases/hls/summit_xl_hls.stl"/>
+	     <mesh filename="file://$(find icclab_summit_xl)/meshes/bases/hls/summit_xl_hls.stl"/>
        </geometry>
        </xacro:if>
        <xacro:unless value="${hq}">
        <geometry>
-	     <mesh filename="file://$(find summit_xl_description)/meshes/bases/hls/summit_xl_hls.dae"/>
+	     <mesh filename="file://$(find icclab_summit_xl)/meshes/bases/hls/summit_xl_hls.dae"/>
        </geometry>
        </xacro:unless>
@@ -50,5 +50,5 @@
        <origin xyz="0 0 0" rpy="0 0 0 " />
        <geometry>
-         <mesh filename="file://$(find summit_xl_description)/meshes/bases/hls/summit_xl_hls.dae"/>
+         <mesh filename="file://$(find icclab_summit_xl)/meshes/bases/hls/summit_xl_hls.dae"/>
        </geometry>
     </collision>
